File: PCB/PIC64-Final/64Pin-2.brd (EAGLE design)
At the start: 100 x 80 mm, 163 parts, among them IC1 , IC2 , IC3 , IC4 , Q1 , X1 , X10 , X2 , X3 , X4 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

Commit message: t
Parts:
- moved X1 20.6 mm to (78.4, 38.4)
Changed lines of the file:
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@@
 <element name="C8" library="rcl" package="C0603" value=" " x="47.73" y="33.405"/>
 <element name="R3" library="rcl" package="RTRIM3296W" value=" " x="2.54" y="19.33" rot="R180"/>
-<element name="X1" library="con-molex" package="22-23-2021" value=" " x="92.4725" y="23.365" rot="R270">
-<attribute name="OC_NEWARK" value="25C3832" x="92.4725" y="23.365" size="1.778" layer="27" rot="R270" display="off"/>
-<attribute name="MPN" value="22-23-2021" x="92.4725" y="23.365" size="1.778" layer="27" rot="R270" display="off"/>
-<attribute name="MF" value="MOLEX" x="92.4725" y="23.365" size="1.778" layer="27" rot="R270" display="off"/>
-<attribute name="OC_FARNELL" value="1462926" x="92.4725" y="23.365" size="1.778" layer="27" rot="R270" display="off"/>
+<element name="X1" library="con-molex" package="22-23-2021" value=" " x="78.3725" y="38.365" rot="R270">
+<attribute name="OC_NEWARK" value="25C3832" x="78.3725" y="38.365" size="1.778" layer="27" rot="R270" display="off"/>
+<attribute name="MPN" value="22-23-2021" x="78.3725" y="38.365" size="1.778" layer="27" rot="R270" display="off"/>
+<attribute name="MF" value="MOLEX" x="78.3725" y="38.365" size="1.778" layer="27" rot="R270" display="off"/>
+<attribute name="OC_FARNELL" value="1462926" x="78.3725" y="38.365" size="1.778" layer="27" rot="R270" display="off"/>
 </element>
 <element name="X2" library="con-molex" package="22-23-2101" value=" " x="79" y="76.5">

Commit message: n
Parts:
- moved X1 19.1 mm to (92.0, 25.0)
Changed lines of the file:
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@@
 <element name="C8" library="rcl" package="C0603" value=" " x="47.73" y="33.405"/>
 <element name="R3" library="rcl" package="RTRIM3296W" value=" " x="2.54" y="19.33" rot="R180"/>
-<element name="X1" library="con-molex" package="22-23-2021" value=" " x="78.3725" y="38.365" rot="R270">
-<attribute name="OC_NEWARK" value="25C3832" x="78.3725" y="38.365" size="1.778" layer="27" rot="R270" display="off"/>
-<attribute name="MPN" value="22-23-2021" x="78.3725" y="38.365" size="1.778" layer="27" rot="R270" display="off"/>
-<attribute name="MF" value="MOLEX" x="78.3725" y="38.365" size="1.778" layer="27" rot="R270" display="off"/>
-<attribute name="OC_FARNELL" value="1462926" x="78.3725" y="38.365" size="1.778" layer="27" rot="R270" display="off"/>
+<element name="X1" library="con-molex" package="22-23-2021" value=" " x="91.9725" y="24.965" rot="R270">
+<attribute name="OC_NEWARK" value="25C3832" x="91.9725" y="24.965" size="1.778" layer="27" rot="R270" display="off"/>
+<attribute name="MPN" value="22-23-2021" x="91.9725" y="24.965" size="1.778" layer="27" rot="R270" display="off"/>
+<attribute name="MF" value="MOLEX" x="91.9725" y="24.965" size="1.778" layer="27" rot="R270" display="off"/>
+<attribute name="OC_FARNELL" value="1462926" x="91.9725" y="24.965" size="1.778" layer="27" rot="R270" display="off"/>
 </element>
 <element name="X2" library="con-molex" package="22-23-2101" value=" " x="79" y="76.5">

Commit message: u
Parts:
- removed X10: (no value), con-molex:22-23-2041
- added J1: 84952-4, ZIF-4:CON4_SMT-RA_FCC-FPC2
- added X8: (no value), con-molex:22-23-2101
- X4: device con-molex:22-23-2101 -> con-molex:22-23-2041
- moved X4 7.40 mm to (35.4, 76.5)
- moved R48 4.30 mm to (12.6, 58.8)
- moved IC4 3.90 mm to (8.89, 49.4)
- moved R50 3.82 mm to (15.8, 44.1)
- moved C24 3.81 mm to (6.50, 43.0)
- moved C25 3.81 mm to (11.8, 43.2)
- moved R49 3.81 mm to (9.13, 42.3)
- moved R51 3.79 mm to (7.64, 57.5), turned to 90 degrees
- turned R46 to 180 degrees
- renumbered D1 to SILVIA-ESPRESSO-MACHINE..DAVE-ZIEGL.R1.0
Connections:
- removed net N$74: R51.2, X10.1
- removed net N$76: IC4.3, X10.2
- removed net N$77: IC4.4, R51.1
- removed net N$79: IC4.2, R48.1
- removed net N$80: R48.2, X10.3
- removed net N$81: IC4.1, X10.4
- removed net N$82: D15.10, X4.1
- removed net N$83: R43.2, X4.2
- removed net N$85: D15.8, X4.3
- removed net N$86: R42.2, X4.4
- removed net N$88: D15.6, X4.5
- removed net N$89: R41.2, X4.6
- removed net N$91: D15.4, X4.7
- removed net N$92: R40.2, X4.8
- removed net N$94: D15.2, X4.9
- removed net N$97: R39.2, X4.10
- new net N$1: IC4.4, X8.1
- new net N$11: R48.2, X8.4
- new net N$17: D15.10, X8.5
- new net N$19: IC4.1, J1.3, R48.1
- new net N$21: IC4.3, J1.2, R51.1
- new net N$23: R43.2, X8.6
- new net N$24: D15.8, X8.7
- new net N$25: R42.2, X8.8
- new net N$26: D15.6, X8.9
- new net N$28: R41.2, X8.10
- new net N$29: D15.4, X4.1
- new net N$30: R40.2, X4.2
- new net N$31: D15.2, X4.3
- new net N$32: R39.2, X4.4
- new net N$5: R51.2, X8.2
- new net N$7: IC4.2, X8.3
- net N$84: now also J1.1
- net N$87: now also J1.4
Routing:
- net N$21: track 0.00 -> 37.0 mm
- net N$19: track 0.00 -> 34.8 mm
- net N$28: track 0.00 -> 34.1 mm
- net N$26: track 0.00 -> 32.6 mm
- net N$25: track 0.00 -> 28.4 mm
- net N$24: track 0.00 -> 22.2 mm
- net N$23: track 0.00 -> 20.8 mm, vias 0 -> 1
- net N$81: track 16.4 -> 0.00 mm
- net N$17: track 0.00 -> 14.2 mm
- net N$7: track 0.00 -> 13.8 mm
- net N$11: track 0.00 -> 12.3 mm
- net VSS: track 589.0 -> 600.6 mm
- net N$76: track 9.22 -> 0.00 mm
- net N$29: track 0.00 -> 7.99 mm
- net N$31: track 0.00 -> 7.99 mm
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- added copper zone on layer 16, net VSS
