File: PCB/PIC64-Final/64Pin-2.brd (EAGLE design)
At the start: 100 x 80 mm, 164 parts, among them IC1 , IC2 , IC3 , IC4 , J1 84952-4, Q1 , X1 , X2 , X3 , X4 , X5 , X6 , X7 , X8 , X9 

Commit message: nd
Parts:
- added Q2, Q3, Q4: IRF540, transistor-power:TO220BV
- added R55, R56, R57, R58, R59, R60, R61, R62, R63: (no value), resistor:R0603
- added U1, U2, U3: LM5114BMFX/S7003094SOT26-GATEDRIVER, SOT26:MF06A
- added X10, X11: (no value), con-molex:KK-156-2
- X1: device con-molex:22-23-2021 -> con-molex:KK-156-2
- moved X1 10.0 mm to (88.9, 34.5)
Connections:
- new net N$33: R57.1, U2.4
- new net N$34: R58.1, U2.6
- new net N$35: R55.1, U1.4
- new net N$41: R56.1, U1.6
- new net N$48: Q2.G, R55.2, R56.2
- new net N$50: Q3.G, R57.2, R58.2
- new net N$52: R59.1, U3.4
- new net N$59: R60.1, U3.6
- new net N$61: Q4.G, R59.2, R60.2
- new net N$63: Q4.D, X1.1
- new net N$65: Q4.S, X1.2
- new net N$67: Q3.D, X10.1
- new net N$74: Q3.S, X10.2
- new net N$75: Q2.D, X11.1
- new net N$76: Q2.S, X11.2
- new net N$77: R61.2, U1.2
- new net N$78: R62.2, U2.2
- new net N$79: R63.2, U3.2
- new net N$80: P.55, R62.1
- new net N$81: P.58, R63.1
- net PIN54: now also R61.1
- net VDD: now also U1.1, U2.1, U3.1
- net VSS: now also U1.3, U2.3, U3.3
Routing:
- net N$46: track 36.5 -> 0.00 mm
- net PIN54: track 43.8 -> 45.5 mm

Commit message: nf
Parts:
- moved R63 147.3 mm to (60.7, 36.8)
- moved R62 146.4 mm to (59.9, 41.0)
- moved R60 141.4 mm to (71.2, 38.9)
- moved R58 137.3 mm to (71.2, 43.6)
- moved R59 135.5 mm to (71.2, 36.8)
- moved R61 134.0 mm to (60.5, 31.6)
- moved R57 131.5 mm to (71.2, 41.5)
- moved U3 119.7 mm to (65.6, 36.7)
- moved Q4 119.6 mm to (79.2, 43.2)
- moved U2 119.6 mm to (65.5, 40.9)
- moved X10 115.2 mm to (91.0, 49.6), turned to 270 degrees
- moved X11 111.2 mm to (91.0, 33.3), turned to 270 degrees
- moved Q2 107.4 mm to (79.0, 35.2)
- moved Q3 16.3 mm to (79.2, 50.8)
- moved U1 16.2 mm to (65.5, 31.2)
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Routing:
- net PIN54: track 45.5 -> 43.8 mm

Commit message: nd
Parts:
- removed R52, R53: (no value), resistor:R0603
- removed X1, X10, X11: (no value), con-molex:KK-156-2
- moved Q3 7.77 mm to (79.7, 43.0)
- moved Q4 7.57 mm to (79.8, 50.8)
- moved R57 5.80 mm to (71.0, 35.8)
- moved R58 5.65 mm to (71.0, 38.0)
- moved R62 4.74 mm to (60.5, 36.2)
- moved U2 4.65 mm to (65.5, 36.2)
- moved R60 4.60 mm to (71.0, 43.5)
- moved R59 4.50 mm to (71.0, 41.2)
- moved U3 3.30 mm to (65.5, 40.0)
- moved R63 3.26 mm to (60.5, 40.0)
- moved U1 1.25 mm to (65.5, 32.5)
- moved R55 1.08 mm to (71.0, 30.2)
- moved R56 0.92 mm to (71.0, 32.5)
- moved R61 0.90 mm to (60.5, 32.5)
- moved Q2 0.84 mm to (79.8, 35.5)
Connections:
- removed net N$46: R52.1, R53.1
- removed net N$65: Q4.S, X1.2
- removed net N$74: Q3.S, X10.2
- removed net N$76: Q2.S, X11.2
- net N$63: no longer X1.1
- net N$67: no longer X10.1
- net N$75: no longer X11.1
- net VSS: now also Q2.S, Q3.S, Q4.S; no longer R52.2, R53.2
Routing:
- net VDD: track 482.5 -> 520.9 mm, vias 5 -> 7
- net VSS: track 600.6 -> 625.3 mm, vias 5 -> 6
- net N$80: track 0.00 -> 16.9 mm
- net N$81: track 0.00 -> 16.1 mm
- net N$61: track 0.00 -> 9.56 mm
- net N$50: track 0.00 -> 8.56 mm
- net N$48: track 0.00 -> 7.80 mm
- net N$59: track 0.00 -> 4.49 mm
- net N$52: track 0.00 -> 4.34 mm
- net N$35: track 0.00 -> 4.00 mm
- net N$41: track 0.00 -> 3.83 mm
- net N$34: track 0.00 -> 3.76 mm
- net N$33: track 0.00 -> 3.62 mm
- net PIN54: track 43.8 -> 47.3 mm
- net N$79: track 0.00 -> 2.93 mm
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
Commit message: D!!
Parts:
- added R52: (no value), rcl:RTRIM3296W
- added R53, R64: (no value), resistor:R0603
- added U4, U5: 282837-3, 3-Pin-5.08:282837-3
- moved LED3 2.20 mm to (83.0, 26.4)
- moved R67 2.20 mm to (84.8, 24.2)
- moved R68 1.75 mm to (82.7, 24.2)
- moved R69 1.60 mm to (80.3, 24.2)
- moved R54 1.21 mm to (79.7, 27.9)
- moved LED4 1.20 mm to (78.9, 26.4)
- moved R70 1.20 mm to (78.2, 24.2)
- moved R71 1.00 mm to (75.8, 24.2)
- moved LED5 0.70 mm to (74.4, 26.4)
- moved R72 0.60 mm to (73.7, 24.2)
- moved R73 0.40 mm to (71.4, 24.2)
Connections:
- new net N$46: Q4.D, U4.1
- new net N$65: Q3.D, U4.3
- new net N$74: Q2.D, U5.2
- net N$63: now also LCDHEADER.20, R53.1; no longer Q4.D
- net N$67: now also R52.1, R64.1; no longer Q3.D
- net N$75: now also LCDHEADER.19, R64.2; no longer Q2.D
- net VDD: now also R52.2, R52.3
- net VSS: now also R53.2, U4.2, U5.1, U5.3
Routing:
- net N$67: track 0.00 -> 75.0 mm
- net N$46: track 0.00 -> 16.0 mm
- net N$65: track 0.00 -> 14.7 mm
- net VDD: track 520.9 -> 534.9 mm
- net N$74: track 0.00 -> 13.2 mm
- net VSS: track 625.3 -> 622.4 mm
- net N$63: track 0.00 -> 2.42 mm
- net N$75: track 0.00 -> 2.05 mm
- net PIN43: track 28.9 -> 27.6 mm
- net OUT: track 7.68 -> 6.54 mm
- net PIN42: track 27.8 -> 26.7 mm
- net N$68: track 2.53 -> 3.44 mm
- net PIN59: track 102.6 -> 103.4 mm
- net PIN54: track 47.3 -> 46.5 mm
- net N$66: track 2.53 -> 3.19 mm
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
Commit message: f?
Parts:
- removed R53, R64: (no value), resistor:R0603
- removed X6: (no value), con-molex:22-23-2021
- added POWER: (no value), con-molex:22-23-2041
- renumbered R3 to CONTRAST, SILVIA-ESPRESSO-MACHINE..DAVE-ZIEGL.R1.0 to D1
Connections:
- removed net N$67: R52.1, R64.1
- new net N$76: POWER.1, R52.2, R52.3
- net N$63: now also POWER.2; no longer R53.1
- net N$75: now also R52.1; no longer R64.2
- net VDD: now also POWER.3; no longer R52.2, R52.3, X6.1
- net VSS: now also POWER.4; no longer R53.2, X6.2
Routing:
- net N$75: track 2.05 -> 80.1 mm
- net N$67: track 75.0 -> 0.00 mm
- net N$76: track 0.00 -> 70.8 mm
- net VDD: track 534.9 -> 520.8 mm
- net N$63: track 2.42 -> 12.5 mm, vias 0 -> 1

Commit message: ND
Parts:
- D10, D11, D12, D13, D14, D16, D17, D3, D4, D5, D6, D7, D8, D9: device zetex:SOD323 -> 0603ZenerDiode:CZRU-M
- moved D10 0.80 mm to (49.0, 58.0)
- moved D17 0.63 mm to (16.6, 57.9)
- moved D5 0.59 mm to (73.7, 58.0)
- moved D14 0.55 mm to (26.4, 58.0)
- moved D3 0.52 mm to (84.4, 58.0)
- moved D6 0.52 mm to (68.3, 58.0)
- moved D12 0.52 mm to (37.6, 58.0)
- moved D16 0.51 mm to (22.2, 58.0)
- moved D7 0.51 mm to (63.6, 58.0)
- moved D8 0.51 mm to (58.4, 58.0)
- moved D11 0.50 mm to (43.4, 58.0)
- moved D9 0.50 mm to (53.4, 58.0)
- moved D4 0.47 mm to (78.9, 58.0)
- moved D13 0.43 mm to (31.6, 58.1)
- renumbered R52 to BRIGHTNESS
Routing:
- net VSS: track 622.4 -> 610.5 mm

Commit message: F?
Parts:
- removed Q4: IRF540, transistor-power:TO220BV
- added OSC: (no value), crystal:TC26H
- DR1, DR2, DR3: value LM5114BMFX/S7003094SOT26-GATEDRIVER -> (none)
- Q1: device crystal:TC26H -> transistor-power:TO220BV
- Q2: value IRF540 -> Dave Ziegl
- Q3: value IRF540 -> R1.0 Aug/2017
- TERM1, TERM2: value 282837-3 -> (none)
- moved Q1 35.4 mm to (79.8, 35.5), flipped to the top, turned to 0 degrees
- moved Q3 7.73 mm to (79.8, 50.8)
- moved Q2 7.52 mm to (79.7, 43.0)
- renumbered J1 to ZIF1, U1 to DR1, U2 to DR2, U3 to DR3, U4 to TERM2, U5 to TERM1, X2 to INPUTS-4, X3 to INPUTS-3, X4 to INPUTS-2, X5 to OUTPUTS-2, X7 to OUTPUTS-1, X8 to INPUTS-1, X9 to OUTPUTS-3
Connections:
- net N$46: now also Q3.D; no longer Q4.D
- net N$48: now also Q1.G; no longer Q2.G
- net N$50: now also Q2.G; no longer Q3.G
- net N$61: now also Q3.G; no longer Q4.G
- net N$65: now also Q2.D; no longer Q3.D
- net N$74: now also Q1.D; no longer Q2.D
- net SOSCI: now also OSC.1; no longer Q1.1
- net SOSCO: now also OSC.2; no longer Q1.2
- net VSS: now also Q1.S; no longer Q4.S

Commit message: DONE!
Parts:
- removed D16, D17: (no value), 0603ZenerDiode:CZRU-M
- removed R61, R62, R63: (no value), resistor:R0603
- added R3, R52, R53: (no value), resistor:R0603
- added SOC1, SOC2: (no value), ic-package:DIL20
- D1, D2: device ic-package:DIL20 -> 0603ZenerDiode:CZRU-M
- moved R50 75.1 mm to (90.0, 55.8), flipped to the bottom, turned to 0 degrees
- moved R51 68.1 mm to (71.0, 32.5), turned to 0 degrees
- moved R20 29.3 mm to (44.0, 71.5)
- moved D2 26.4 mm to (78.9, 58.0), flipped to the bottom, turned to 0 degrees
- moved R35 24.1 mm to (19.1, 71.6), turned to 0 degrees
- moved R19 22.9 mm to (49.5, 71.5)
- moved R18 22.5 mm to (55.0, 71.5), flipped to the top, turned to 0 degrees
- moved R34 22.5 mm to (24.1, 71.6)
- moved R33 21.8 mm to (29.2, 71.6), turned to 0 degrees
- moved R25 20.8 mm to (55.0, 51.4)
- moved R42 20.8 mm to (26.9, 51.0), turned to 270 degrees
- moved R37 20.3 mm to (7.64, 57.5), turned to 90 degrees
- moved R32 20.3 mm to (34.3, 71.6)
- moved R17 20.3 mm to (60.0, 71.5), flipped to the top, turned to 0 degrees
- moved R26 20.2 mm to (53.5, 53.6)
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- renumbered D15 to SOC3, IC1 to SOC7, IC2 to SOC6, IC3 to SOC5, IC4 to SOC4, R67 to R129, R68 to R128, R69 to R127, R70 to R126, R71 to R125, R72 to R124, R73 to R123, R74 to R122, R75 to R121, R76 to R120, R77 to R119, R78 to R118, R79 to R117, R80 to R116, R81 to R115, R82 to R114, R83 to R113, R84 to R112, R85 to R111, R86 to R110, R87 to R109, R88 to R108, R89 to R107, R90 to R106, R91 to R105, R92 to R104, R93 to R103, R94 to R102, R95 to R101, R96 to R100
Connections:
- net N$100: now also R20.2; no longer R26.2
- net N$101: now also R19.2; no longer R25.2
- net N$102: now also SOC2.6; no longer D2.6
- net N$103: now also R19.1, SOC2.7; no longer D2.7, R25.1
- net N$104: now also SOC2.4; no longer D2.4
- net N$105: now also R17.1, SOC2.3; no longer D2.3, R23.1
- net N$106: now also R17.2; no longer R23.2
- net N$107: now also SOC2.2; no longer D2.2
- net N$108: now also SOC2.1; no longer D2.1
- net N$11: now also R36.2; no longer R48.2
- net N$110: now also SOC1.10; no longer D1.10
- net N$111: now also R7.2; no longer R13.2
- net N$112: now also R7.1, SOC1.9; no longer D1.9, R13.1
- net N$113: now also SOC1.8; no longer D1.8
- net N$114: now also R18.1, SOC2.5; no longer D2.5, R24.1
- net N$115: now also R18.2; no longer R24.2
- net N$116: now also R5.2; no longer R7.2
- net N$117: now also R5.1, SOC1.5; no longer D1.5, R7.1
- net N$118: now also SOC1.4; no longer D1.4
- net N$119: now also R4.2; no longer R6.2
- net N$120: now also R4.1, SOC1.3; no longer D1.3, R6.1
- net N$121: now also SOC1.2; no longer D1.2
- net N$122: now also R3.2; no longer R4.2
- net N$123: now also R3.1, SOC1.1; no longer D1.1, R4.1
- net N$19: now also R36.1; no longer R48.1
- net N$21: now also R37.1; no longer R51.1
- net N$23: now also R35.2; no longer R43.2
- net N$25: now also R34.2; no longer R42.2
- net N$28: now also R33.2; no longer R41.2
- net N$30: now also R32.2; no longer R40.2
- net N$32: now also R31.2; no longer R39.2
- net N$33: now also R54.1; no longer R57.1
- net N$34: now also R53.1; no longer R58.1
- net N$35: now also R52.1; no longer R55.1
- net N$41: now also R51.1; no longer R56.1
- net N$44: now also SOC1.6; no longer D1.6
- net N$45: now also R6.2; no longer R10.2
- net N$48: now also R51.2, R52.2; no longer R55.2, R56.2
- net N$5: now also R37.2; no longer R51.2
- net N$50: now also R53.2, R54.2; no longer R57.2, R58.2
- net N$52: now also R56.1; no longer R59.1
- net N$54: now also R6.1, SOC1.7; no longer D1.7, R10.1
- net N$59: now also R55.1; no longer R60.1
- net N$61: now also R55.2, R56.2; no longer R59.2, R60.2
- net N$77: now also R57.2; no longer R61.2
- net N$78: now also R58.2; no longer R62.2
- net N$79: now also R59.2; no longer R63.2
- net N$80: now also R58.1; no longer R62.1
- net N$81: now also R59.1; no longer R63.1
- net N$84: now also R35.1; no longer R43.1
- net N$87: now also R34.1; no longer R42.1
- net N$90: now also R33.1; no longer R41.1
- net N$93: now also R32.1; no longer R40.1
- net N$95: now also R31.1; no longer R39.1
- net N$96: now also SOC2.10; no longer D2.10
- net N$98: now also R20.1, SOC2.9; no longer D2.9, R26.1
- net N$99: now also SOC2.8; no longer D2.8
- net OUT: now also R60.2; no longer R54.2
- net PIN11: now also D1.1, SOC1.18; no longer D1.18, D3.1
- net PIN12: now also D2.1, R10.1, R11.2, SOC1.16; no longer D1.16, D4.1, R11.1, R12.2
- net PIN13: now also D3.1, R12.1, R13.2, SOC1.14; no longer D1.14, D5.1, R14.1, R15.2
- net PIN14: now also D4.1, R14.1, R15.2, SOC1.12; no longer D1.12, D6.1, R17.1, R18.2
- net PIN17: now also D5.1, R21.1, R22.2, SOC2.20; no longer D2.20, D7.1, R20.1, R21.2
- net PIN18: now also D6.1, R23.1, R24.2, SOC2.18; no longer D2.18, D8.1, R19.1, R22.2
- net PIN21: now also D7.1, R25.1, R26.2, SOC2.16; no longer D2.16, D9.1, R27.1, R28.2
- net PIN22: now also D8.1, R27.1, R28.2, SOC2.14; no longer D10.1, D2.14, R29.1, R30.2
- net PIN23: now also D9.1, R29.1, R30.2, SOC2.12; no longer D11.1, D2.12, R31.1, R32.2
- net PIN24: now also D10.1, R38.1, R39.2; no longer D12.1, R33.1, R34.2
- net PIN27: now also D11.1, R40.1, R41.2; no longer D13.1, R35.1, R36.2
- net PIN28: now also D12.1, R42.1, R43.2; no longer D14.1, R37.1, R38.2
- net PIN29: now also D13.1; no longer D16.1
- net PIN30: now also D14.1; no longer D17.1
- net PIN31: now also R49.1; no longer R50.1
- net PIN32: now also R48.1; no longer R49.1
- net PIN54: now also R57.1, R60.1; no longer R54.1, R61.1
- net PIN8: now also R50.1, SOC1.20; no longer D1.20, R5.1
- net VDD: now also R10.2, R12.2, R21.2, R23.2, R25.2, R38.2, R40.2, R42.2, R48.2; no longer R11.2, R17.2, R19.2, R20.2, R31.2, R33.2, R35.2, R37.2, R5.2
- net VSS: now also D1.2, D2.2, R11.1, R13.1, R24.1, R26.1, R39.1, R41.1, R43.1, SOC1.11, SOC1.13, SOC1.15, SOC1.17, SOC1.19, SOC2.11, SOC2.13, SOC2.15, SOC2.17, SOC2.19; no longer D1.11, D1.13, D1.15, D1.17, D1.19, D16.2, D17.2, D2.11, D2.13, D2.15, D2.17, D2.19, R12.1, R18.1, R21.1, R32.1, R34.1, R36.1, R38.1
