File: PCB/PIC64-Final/64Pin-2.brd (EAGLE design)
At the start: 100 x 80 mm, 179 parts, among them Q1 , Q2 Dave Ziegl, Q3 R1.0 Aug/2017

Commit message: AtOrd
Routing:
- net VSS: track 610.5 -> 604.3 mm
Other:
- board text added: "Dave Zieglgansberger Aug 2017, Rev 1.0"
Changed lines of the file:
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@@
 <wire x1="100" y1="80" x2="0" y2="80" width="0" layer="20"/>
 <wire x1="0" y1="80" x2="0" y2="0" width="0" layer="20"/>
+<text x="6.3" y="29.7" size="1.4224" layer="1" font="vector" ratio="12">Dave Zieglgansberger
+Aug 2017, Rev 1.0</text>
 </plain>
 <attributes>
@@
 <wire x1="5" y1="32.6425" x2="5" y2="24.205" width="0.6096" layer="16"/>
 <wire x1="2.54" y1="21.87" x2="5" y2="24.205" width="0.6096" layer="16"/>
-<wire x1="41.9" y1="7.25" x2="37.875" y2="7.25" width="0.6096" layer="16"/>
 <wire x1="37.25" y1="10.25" x2="37.25" y2="15.75" width="0.6096" layer="16"/>
 <wire x1="37.25" y1="15.75" x2="34.25" y2="18.75" width="0.6096" layer="16"/>
@@
 <wire x1="25.525" y1="53.625" x2="25.525" y2="56.125" width="0.3048" layer="1"/>
 <wire x1="30.775" y1="53.625" x2="30.775" y2="56.125" width="0.3048" layer="1"/>
-<wire x1="37.875" y1="7.25" x2="37.875" y2="9.495" width="0.6096" layer="16"/>
 <wire x1="37.875" y1="9.495" x2="37.87" y2="9.5" width="0.254" layer="16"/>
 <wire x1="37.25" y1="10.25" x2="37.25" y2="10.12" width="0.254" layer="16"/>
@@
 </board>
 </drawing>
+<compatibility>
+<note version="6.3" minversion="6.2.2" severity="warning">
+Since Version 6.2.2 text objects can contain more than one line,
+which will not be processed correctly with this version.
+</note>
+</compatibility>
 </eagle>
