File: PCB/PIC64-Final/64Pin-2.sch (EAGLE design)
At the start: 158 parts, among them IC1 , IC2 , IC3 , IC4 , Q1 , X10 , X2 , X3 , X4 , X5 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

Commit message: u
Parts:
- removed X10: (no value), con-molex:22-23-2041
- added J1: 84952-4, ZIF-4:84952-4
- added X8: (no value), con-molex:22-23-2101
- X4: device con-molex:22-23-2101 -> con-molex:22-23-2041
- renumbered D1 to SILVIA-ESPRESSO-MACHINE..DAVE-ZIEGL.R1.0
Connections:
- removed net N$74: R51.2, X10-1.S
- removed net N$76: IC4.3, X10-2.S
- removed net N$77: IC4.4, R51.1
- removed net N$79: IC4.2, R48.1
- removed net N$80: R48.2, X10-3.S
- removed net N$81: IC4.1, X10-4.S
- removed net N$82: D15.10, X4-1.S
- removed net N$83: R43.2, X4-2.S
- removed net N$85: D15.8, X4-3.S
- removed net N$86: R42.2, X4-4.S
- removed net N$88: D15.6, X4-5.S
- removed net N$89: R41.2, X4-6.S
- removed net N$91: D15.4, X4-7.S
- removed net N$92: R40.2, X4-8.S
- removed net N$94: D15.2, X4-9.S
- removed net N$97: R39.2, X4-10.S
- new net N$1: IC4.4, X8-1.S
- new net N$11: R48.2, X8-4.S
- new net N$17: D15.10, X8-5.S
- new net N$19: IC4.1, J1.3, R48.1
- new net N$21: IC4.3, J1.2, R51.1
- new net N$23: R43.2, X8-6.S
- new net N$24: D15.8, X8-7.S
- new net N$25: R42.2, X8-8.S
- new net N$26: D15.6, X8-9.S
- new net N$28: R41.2, X8-10.S
- new net N$29: D15.4, X4-1.S
- new net N$30: R40.2, X4-2.S
- new net N$31: D15.2, X4-3.S
- new net N$32: R39.2, X4-4.S
- new net N$5: R51.2, X8-2.S
- new net N$7: IC4.2, X8-3.S
- net N$84: now also J1.1
- net N$87: now also J1.4
Other:
- moved on the sheet: D15, R39, R40, R41, R42, R43, R48, R51, X4-1, X4-2, X4-3, X4-4
