File: PCB/PIC64-Final/64Pin-2.sch (EAGLE design)
At the start: 159 parts, among them IC1 , IC2 , IC3 , IC4 , J1 84952-4, Q1 , X2 , X3 , X4 , X5 , X6 , X7 , X8 , X9 

Commit message: nd
Parts:
- added Q2, Q3, Q4: IRF540, transistor-power:IRF540
- added R55, R56, R57, R58, R59, R60, R61, R62, R63: (no value), resistor:R-US_R0603
- added U1, U2, U3: LM5114BMFX/S7003094SOT26-GATEDRIVER, SOT26:LM5114BMFX/S7003094SOT26-GATEDRIVER
- added X1, X10, X11: (no value), con-molex:KK-156-2
Connections:
- new net N$33: R57.1, U2.N_OUT
- new net N$34: R58.1, U2.P_OUT
- new net N$35: R55.1, U1.N_OUT
- new net N$41: R56.1, U1.P_OUT
- new net N$48: Q2.G, R55.2, R56.2
- new net N$50: Q3.G, R57.2, R58.2
- new net N$52: R59.1, U3.N_OUT
- new net N$59: R60.1, U3.P_OUT
- new net N$61: Q4.G, R59.2, R60.2
- new net N$63: Q4.D, X1-1.S
- new net N$65: Q4.S, X1-2.S
- new net N$67: Q3.D, X10-1.S
- new net N$74: Q3.S, X10-2.S
- new net N$75: Q2.D, X11-1.S
- new net N$76: Q2.S, X11-2.S
- new net N$77: R61.2, U1.IN
- new net N$78: R62.2, U2.IN
- new net N$79: R63.2, U3.IN
- new net N$80: P.C3INA/*U5RTS/U5BCLK/OC5/RD7, R62.1
- new net N$81: P.*U5CTS/OC6/RF0, R63.1
- net PIN54: now also R61.1
- net VDD: now also U1.VDD, U2.VDD, U3.VDD
- net VSS: now also U1.VSS, U2.VSS, U3.VSS

Commit message: nd
Parts:
- removed R52, R53: (no value), resistor:R-US_R0603
- removed X1, X10, X11: (no value), con-molex:KK-156-2
Connections:
- removed net N$46: R52.1, R53.1
- removed net N$65: Q4.S, X1-2.S
- removed net N$74: Q3.S, X10-2.S
- removed net N$76: Q2.S, X11-2.S
- net N$63: no longer X1-1.S
- net N$67: no longer X10-1.S
- net N$75: no longer X11-1.S
- net VSS: now also Q2.S, Q3.S, Q4.S; no longer R52.2, R53.2
Changed lines of the file:
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@@
 <part name="R24" library="resistor" deviceset="R-US_" device="R0603" value=" "/>
 <part name="X5" library="con-molex" deviceset="22-23-2101" device="" value=" "/>
-<part name="R52" library="resistor" deviceset="R-US_" device="R0603" value=" "/>
-<part name="R53" library="resistor" deviceset="R-US_" device="R0603" value=" "/>
 <part name="R54" library="resistor" deviceset="R-US_" device="R0603" value=" "/>
 <part name="VSS3" library="supply1" deviceset="VSS" device=""/>
@@
 <part name="R55" library="resistor" deviceset="R-US_" device="R0603" value=" "/>
 <part name="R56" library="resistor" deviceset="R-US_" device="R0603" value=" "/>
-<part name="X1" library="con-molex" deviceset="KK-156-2" device="" value=" "/>
-<part name="X10" library="con-molex" deviceset="KK-156-2" device="" value=" "/>
-<part name="X11" library="con-molex" deviceset="KK-156-2" device="" value=" "/>
 <part name="Q3" library="transistor-power" deviceset="IRF540" device=""/>
 <part name="Q2" library="transistor-power" deviceset="IRF540" device=""/>
@@
 <instance part="X5" gate="-9" x="15.24" y="-243.84" rot="R270"/>
 <instance part="X5" gate="-10" x="12.7" y="-243.84" rot="R270"/>
-<instance part="R52" gate="G$1" x="111.76" y="-246.38" rot="R90"/>
-<instance part="R53" gate="G$1" x="95.25" y="-251.46" rot="R180"/>
 <instance part="R54" gate="G$1" x="55.88" y="-173.99"/>
 <instance part="VSS3" gate="G$1" x="76.2" y="208.28"/>
@@
 <instance part="R55" gate="G$1" x="259.08" y="-135.89"/>
 <instance part="R56" gate="G$1" x="259.08" y="-138.43"/>
-<instance part="X1" gate="-1" x="289.56" y="-71.12"/>
-<instance part="X1" gate="-2" x="289.56" y="-81.28"/>
-<instance part="X10" gate="-1" x="289.56" y="-100.33"/>
-<instance part="X10" gate="-2" x="289.56" y="-110.49"/>
-<instance part="X11" gate="-1" x="289.56" y="-128.27"/>
-<instance part="X11" gate="-2" x="289.56" y="-138.43"/>
 <instance part="Q3" gate="G$1" x="266.7" y="-105.41"/>
 <instance part="Q2" gate="G$1" x="266.7" y="-133.35"/>
@@
 <wire x1="78.74" y1="-251.46" x2="78.74" y2="-241.3" width="0.1524" layer="91"/>
 <junction x="78.74" y="-251.46"/>
-<pinref part="R53" gate="G$1" pin="2"/>
-<wire x1="90.17" y1="-251.46" x2="86.36" y2="-251.46" width="0.1524" layer="91"/>
 <wire x1="86.36" y1="-251.46" x2="78.74" y2="-251.46" width="0.1524" layer="91"/>
 <wire x1="78.74" y1="-251.46" x2="73.66" y2="-251.46" width="0.1524" layer="91"/>
@@
 <wire x1="186.69" y1="-78.74" x2="186.69" y2="-107.95" width="0.1524" layer="91"/>
 <junction x="186.69" y="-107.95"/>
-</segment>
-<segment>
+<wire x1="86.36" y1="-251.46" x2="88.9" y2="-251.46" width="0.1524" layer="91"/>
+<wire x1="88.9" y1="-251.46" x2="88.9" y2="-241.3" width="0.1524" layer="91"/>
 <pinref part="P" gate="A" pin="VSS_3"/>
 <wire x1="-2.54" y1="83.82" x2="-2.54" y2="38.1" width="0.1524" layer="91"/>
@@
 <junction x="7.62" y="33.02"/>
 <pinref part="VSS1" gate="G$1" pin="VSS"/>
-<pinref part="R52" gate="G$1" pin="2"/>
 <pinref part="R3" gate="G$1" pin="A"/>
 <wire x1="111.76" y1="-241.3" x2="111.76" y2="-233.68" width="0.1524" layer="91"/>
@@
 <wire x1="91.44" y1="-68.58" x2="91.44" y2="101.6" width="0.1524" layer="91"/>
 <junction x="91.44" y="101.6"/>
+<wire x1="88.9" y1="-241.3" x2="111.76" y2="-241.3" width="0.1524" layer="91"/>
+<junction x="88.9" y="-251.46"/>
 </segment>
 <segment>
@@
 <junction x="-35.56" y="209.55"/>
 </segment>
+<segment>
+<pinref part="Q3" gate="G$1" pin="S"/>
+<wire x1="269.24" y1="-110.49" x2="287.02" y2="-110.49" width="0.1524" layer="91"/>
+</segment>
+<segment>
+<pinref part="Q2" gate="G$1" pin="S"/>
+<wire x1="269.24" y1="-138.43" x2="287.02" y2="-138.43" width="0.1524" layer="91"/>
+</segment>
+<segment>
+<pinref part="Q4" gate="G$1" pin="S"/>
+<wire x1="287.02" y1="-81.28" x2="269.24" y2="-81.28" width="0.1524" layer="91"/>
+</segment>
 </net>
 <net name="VDD" class="1">
@@
 </segment>
 </net>
-<net name="N$46" class="0">
-<segment>
-<pinref part="R52" gate="G$1" pin="1"/>
-<pinref part="R53" gate="G$1" pin="1"/>
-<wire x1="100.33" y1="-251.46" x2="111.76" y2="-251.46" width="0.1524" layer="91"/>
-</segment>
-</net>
 <net name="N$33" class="0">
 <segment>
@@
 <segment>
 <pinref part="Q4" gate="G$1" pin="D"/>
-<pinref part="X1" gate="-1" pin="S"/>
 <wire x1="269.24" y1="-71.12" x2="287.02" y2="-71.12" width="0.1524" layer="91"/>
 </segment>
 </net>
-<net name="N$65" class="0">
-<segment>
-<pinref part="X1" gate="-2" pin="S"/>
-<pinref part="Q4" gate="G$1" pin="S"/>
-<wire x1="287.02" y1="-81.28" x2="269.24" y2="-81.28" width="0.1524" layer="91"/>
-</segment>
-</net>
 <net name="N$67" class="0">
 <segment>
 <pinref part="Q3" gate="G$1" pin="D"/>
-<pinref part="X10" gate="-1" pin="S"/>
 <wire x1="269.24" y1="-100.33" x2="287.02" y2="-100.33" width="0.1524" layer="91"/>
 </segment>
 </net>
-<net name="N$74" class="0">
-<segment>
-<pinref part="Q3" gate="G$1" pin="S"/>
-<pinref part="X10" gate="-2" pin="S"/>
-<wire x1="269.24" y1="-110.49" x2="287.02" y2="-110.49" width="0.1524" layer="91"/>
-</segment>
-</net>
 <net name="N$75" class="0">
 <segment>
 <pinref part="Q2" gate="G$1" pin="D"/>
-<pinref part="X11" gate="-1" pin="S"/>
 <wire x1="269.24" y1="-128.27" x2="287.02" y2="-128.27" width="0.1524" layer="91"/>
 </segment>
 </net>
-<net name="N$76" class="0">
-<segment>
-<pinref part="Q2" gate="G$1" pin="S"/>
-<pinref part="X11" gate="-2" pin="S"/>
-<wire x1="269.24" y1="-138.43" x2="287.02" y2="-138.43" width="0.1524" layer="91"/>
-</segment>
-</net>

Commit message: D!!
Parts:
- added R52: (no value), rcl:R-TRIMM3296W
- added R53, R64: (no value), resistor:R-US_R0603
- added U4, U5: 282837-3, 3-Pin-5.08:282837-3
Connections:
- new net N$46: Q4.D, U4.1
- new net N$65: Q3.D, U4.3
- new net N$74: Q2.D, U5.2
- net N$63: now also LCDHEADER.20, R53.1; no longer Q4.D
- net N$67: now also R52.A, R64.1; no longer Q3.D
- net N$75: now also LCDHEADER.19, R64.2; no longer Q2.D
- net VDD: now also R52.E, R52.S
- net VSS: now also R53.2, U4.2, U5.1, U5.3

Commit message: f?
Parts:
- removed R53, R64: (no value), resistor:R-US_R0603
- removed X6: (no value), con-molex:22-23-2021
- added POWER: (no value), con-molex:22-23-2041
- renumbered R3 to CONTRAST, SILVIA-ESPRESSO-MACHINE..DAVE-ZIEGL.R1.0 to D1
Connections:
- removed net N$67: R52.A, R64.1
- new net N$76: POWER-1.S, R52.E, R52.S
- net N$63: now also POWER-2.S; no longer R53.1
- net N$75: now also R52.A; no longer R64.2
- net VDD: now also POWER-3.S; no longer R52.E, R52.S, X6-1.S
- net VSS: now also POWER-4.S; no longer R53.2, X6-2.S

Commit message: ND
Parts:
- D10, D11, D12, D13, D14, D16, D17, D3, D4, D5, D6, D7, D8, D9: device zetex:DSOD323 -> 0603ZenerDiode:CZRU52C3V3CZRU-M
- renumbered R52 to BRIGHTNESS
Connections:
- net PIN11: now also D3.11; no longer D3.C
- net PIN12: now also D4.11; no longer D4.C
- net PIN13: now also D5.11; no longer D5.C
- net PIN14: now also D6.11; no longer D6.C
- net PIN17: now also D7.11; no longer D7.C
- net PIN18: now also D8.11; no longer D8.C
- net PIN21: now also D9.11; no longer D9.C
- net PIN22: now also D10.11; no longer D10.C
- net PIN23: now also D11.11; no longer D11.C
- net PIN24: now also D12.11; no longer D12.C
- net PIN27: now also D13.11; no longer D13.C
- net PIN28: now also D14.11; no longer D14.C
- net PIN29: now also D16.11; no longer D16.C
- net PIN30: now also D17.11; no longer D17.C
- net VSS: now also D10.22, D11.22, D12.22, D13.22, D14.22, D16.22, D17.22, D3.22, D4.22, D5.22, D6.22, D7.22, D8.22, D9.22; no longer D10.A, D11.A, D12.A, D13.A, D14.A, D16.A, D17.A, D3.A, D4.A, D5.A, D6.A, D7.A, D8.A, D9.A

Commit message: F?
Parts:
- removed Q4: IRF540, transistor-power:IRF540
- added OSC: (no value), crystal:CRYSTALTC26H
- DR1, DR2, DR3: value LM5114BMFX/S7003094SOT26-GATEDRIVER -> (none)
- Q1: device crystal:CRYSTALTC26H -> transistor-power:IRF540; MF 32.768KHz -> (none)
- Q2: value IRF540 -> Dave Ziegl
- Q3: value IRF540 -> R1.0 Aug/2017
- TERM1, TERM2: value 282837-3 -> (none)
- renumbered J1 to ZIF1, U1 to DR1, U2 to DR2, U3 to DR3, U4 to TERM2, U5 to TERM1, X2 to INPUTS-4, X3 to INPUTS-3, X4 to INPUTS-2, X5 to OUTPUTS-2, X7 to OUTPUTS-1, X8 to INPUTS-1, X9 to OUTPUTS-3
Connections:
- net N$46: now also Q3.D; no longer Q4.D
- net N$48: now also Q1.G; no longer Q2.G
- net N$50: now also Q2.G; no longer Q3.G
- net N$61: now also Q3.G; no longer Q4.G
- net N$65: now also Q2.D; no longer Q3.D
- net N$74: now also Q1.D; no longer Q2.D
- net SOSCI: now also OSC.1; no longer Q1.1
- net SOSCO: now also OSC.2; no longer Q1.2
- net VSS: now also Q1.S; no longer Q4.S
Other:
- note added: "Espresso Controller Aug 2017 By Dave Zieglgansberger"
- moved on the sheet: Q2, Q3

Commit message: DONE!
Parts:
- removed D16, D17: (no value), 0603ZenerDiode:CZRU52C3V3CZRU-M
- removed R61, R62, R63, R67, R68, R69, R70, R71, R72, R73, R74, R75, R76, R77, R78, R79, R80, R81, R82, R83, R84, R85, R86, R88, R89, R90, R91, R92, R93, R94, R95, R96: (no value), resistor:R-US_R0603
- added R100, R101, R102, R103, R104, R105, R106, R107, R108, R110, R111, R112, R113, R114, R115, R116, R117, R118, R119, R120, R121, R122, R123, R124, R125, R126, R127, R128, R129, R3, R52, R53: (no value), resistor:R-US_R0603
- added SOC1, SOC2: (no value), ic-package:DIL20
- D1, D2: device ic-package:DIL20 -> 0603ZenerDiode:CZRU52C3V3CZRU-M
- renumbered D15 to SOC3, IC1 to SOC7, IC2 to SOC6, IC3 to SOC5, IC4 to SOC4, R87 to R109
Connections:
- net N$100: now also R20.2; no longer R26.2
- net N$101: now also R19.2; no longer R25.2
- net N$102: now also SOC2.6; no longer D2.6
- net N$103: now also R19.1, SOC2.7; no longer D2.7, R25.1
- net N$104: now also SOC2.4; no longer D2.4
- net N$105: now also R17.1, SOC2.3; no longer D2.3, R23.1
- net N$106: now also R17.2; no longer R23.2
- net N$107: now also SOC2.2; no longer D2.2
- net N$108: now also SOC2.1; no longer D2.1
- net N$11: now also R36.2; no longer R48.2
- net N$110: now also SOC1.10; no longer D1.10
- net N$111: now also R7.2; no longer R13.2
- net N$112: now also R7.1, SOC1.9; no longer D1.9, R13.1
- net N$113: now also SOC1.8; no longer D1.8
- net N$114: now also R18.1, SOC2.5; no longer D2.5, R24.1
- net N$115: now also R18.2; no longer R24.2
- net N$116: now also R5.2; no longer R7.2
- net N$117: now also R5.1, SOC1.5; no longer D1.5, R7.1
- net N$118: now also SOC1.4; no longer D1.4
- net N$119: now also R4.2; no longer R6.2
- net N$120: now also R4.1, SOC1.3; no longer D1.3, R6.1
- net N$121: now also SOC1.2; no longer D1.2
- net N$122: now also R3.2; no longer R4.2
- net N$123: now also R3.1, SOC1.1; no longer D1.1, R4.1
- net N$13: now also R107.2; no longer R89.2
- net N$19: now also R36.1; no longer R48.1
- net N$21: now also R37.1; no longer R51.1
- net N$23: now also R35.2; no longer R43.2
- net N$25: now also R34.2; no longer R42.2
- net N$28: now also R33.2; no longer R41.2
- net N$3: now also R101.2; no longer R95.2
- net N$30: now also R32.2; no longer R40.2
- net N$32: now also R31.2; no longer R39.2
- net N$33: now also R54.1; no longer R57.1
- net N$34: now also R53.1; no longer R58.1
- net N$35: now also R52.1; no longer R55.1
- net N$36: now also R100.1; no longer R96.1
- net N$37: now also R102.1; no longer R94.1
- net N$38: now also R104.1; no longer R92.1
- net N$39: now also R106.1; no longer R90.1
- net N$40: now also R108.1; no longer R88.1
- net N$41: now also R51.1; no longer R56.1
- net N$42: now also R110.1; no longer R86.1
- net N$43: now also R111.2; no longer R85.2
- net N$44: now also SOC1.6; no longer D1.6
- net N$45: now also R6.2; no longer R10.2
- net N$47: now also R113.2; no longer R83.2
- net N$48: now also R51.2, R52.2; no longer R55.2, R56.2
- net N$49: now also R115.2; no longer R81.2
- net N$5: now also R37.2; no longer R51.2
- net N$50: now also R53.2, R54.2; no longer R57.2, R58.2
- net N$51: now also R117.2; no longer R79.2
- net N$52: now also R56.1; no longer R59.1
- net N$53: now also R119.2; no longer R77.2
- net N$54: now also R6.1, SOC1.7; no longer D1.7, R10.1
- net N$55: now also R118.1; no longer R78.1
- net N$56: now also R116.1; no longer R80.1
- net N$57: now also R114.1; no longer R82.1
- net N$58: now also R112.1; no longer R84.1
- net N$59: now also R55.1; no longer R60.1
- net N$6: now also R103.2; no longer R93.2
- net N$60: now also R121.2; no longer R75.2
- net N$61: now also R55.2, R56.2; no longer R59.2, R60.2
- net N$62: now also R123.2; no longer R73.2
- net N$64: now also R125.2; no longer R71.2
- net N$66: now also R127.2; no longer R69.2
- net N$68: now also R129.2; no longer R67.2
- net N$69: now also R128.1; no longer R68.1
- net N$70: now also R126.1; no longer R70.1
- net N$71: now also R124.1; no longer R72.1
- net N$72: now also R122.1; no longer R74.1
- net N$73: now also R120.1; no longer R76.1
- net N$77: now also R57.2; no longer R61.2
- net N$78: now also R58.2; no longer R62.2
- net N$79: now also R59.2; no longer R63.2
- net N$8: now also R105.2; no longer R91.2
- net N$80: now also R58.1; no longer R62.1
- net N$81: now also R59.1; no longer R63.1
- net N$84: now also R35.1; no longer R43.1
- net N$87: now also R34.1; no longer R42.1
- net N$90: now also R33.1; no longer R41.1
- net N$93: now also R32.1; no longer R40.1
- net N$95: now also R31.1; no longer R39.1
- net N$96: now also SOC2.10; no longer D2.10
- net N$98: now also R20.1, SOC2.9; no longer D2.9, R26.1
- net N$99: now also SOC2.8; no longer D2.8
- net OUT: now also R129.1, R60.2; no longer R54.2, R67.1
- net PIN11: now also D1.11, SOC1.18; no longer D1.18, D3.11
- net PIN12: now also D2.11, R10.1, R11.2, SOC1.16; no longer D1.16, D4.11, R11.1, R12.2
- net PIN13: now also D3.11, R12.1, R13.2, SOC1.14; no longer D1.14, D5.11, R14.1, R15.2
- net PIN14: now also D4.11, R14.1, R15.2, SOC1.12; no longer D1.12, D6.11, R17.1, R18.2
- net PIN17: now also D5.11, R21.1, R22.2, SOC2.20; no longer D2.20, D7.11, R20.1, R21.2
- net PIN18: now also D6.11, R23.1, R24.2, SOC2.18; no longer D2.18, D8.11, R19.1, R22.2
- net PIN21: now also D7.11, R25.1, R26.2, SOC2.16; no longer D2.16, D9.11, R27.1, R28.2
- net PIN22: now also D8.11, R27.1, R28.2, SOC2.14; no longer D10.11, D2.14, R29.1, R30.2
- net PIN23: now also D9.11, R29.1, R30.2, SOC2.12; no longer D11.11, D2.12, R31.1, R32.2
- net PIN24: now also D10.11, R38.1, R39.2; no longer D12.11, R33.1, R34.2
- net PIN27: now also D11.11, R40.1, R41.2; no longer D13.11, R35.1, R36.2
- net PIN28: now also D12.11, R42.1, R43.2; no longer D14.11, R37.1, R38.2
- net PIN29: now also D13.11; no longer D16.11
- net PIN30: now also D14.11; no longer D17.11
- net PIN31: now also R49.1; no longer R50.1
- net PIN32: now also R48.1; no longer R49.1
- net PIN33: now also R101.1; no longer R95.1
- net PIN34: now also R103.1; no longer R93.1
- net PIN36: now also R105.1; no longer R91.1
- net PIN37: now also R107.1; no longer R89.1
- net PIN40: now also R111.1; no longer R85.1
- net PIN45: now also R113.1; no longer R83.1
- net PIN46: now also R115.1; no longer R81.1
- net PIN49: now also R117.1; no longer R79.1
- net PIN50: now also R119.1; no longer R77.1
- net PIN51: now also R121.1; no longer R75.1
- net PIN52: now also R123.1; no longer R73.1
- net PIN53: now also R125.1; no longer R71.1
- net PIN54: now also R57.1, R60.1; no longer R54.1, R61.1
- net PIN59: now also R127.1; no longer R69.1
- net PIN8: now also R50.1, SOC1.20; no longer D1.20, R5.1
- net VDD: now also R10.2, R12.2, R21.2, R23.2, R25.2, R38.2, R40.2, R42.2, R48.2; no longer R11.2, R17.2, R19.2, R20.2, R31.2, R33.2, R35.2, R37.2, R5.2
- net VSS: now also D1.22, D2.22, R100.2, R102.2, R104.2, R106.2, R108.2, R11.1, R110.2, R112.2, R114.2, R116.2, R118.2, R120.2, R122.2, R124.2, R126.2, R128.2, R13.1, R24.1, R26.1, R39.1, R41.1, R43.1, SOC1.11, SOC1.13, SOC1.15, SOC1.17, SOC1.19, SOC2.11, SOC2.13, SOC2.15, SOC2.17, SOC2.19; no longer D1.11, D1.13, D1.15, D1.17, D1.19, D16.22, D17.22, D2.11, D2.13, D2.15, D2.17, D2.19, R12.1, R18.1, R21.1, R32.1, R34.1, R36.1, R38.1, R68.2, R70.2, R72.2, R74.2, R76.2, R78.2, R80.2, R82.2, R84.2, R86.2, R88.2, R90.2, R92.2, R94.2, R96.2
Other:
- note added: "LCD Header is Female 20 Pin header, on bach side of board, Pin 19 is connected through Brightness Pot, to POWER-1, Pin 20 is connected directly to POWER-2. Connect +5V to POWER-1 and GND to POWER-2 for Display with LED Backlighting, or EL Driver (or 120VAC) to POWER-1 and 2."
- note added: "R100,102,104,106,108,110,112,114,116,118,120,122, 124,126, and 128 are used for current limiting and brightness control for Indicating LED's on Outputs."
- note added: "R101,103,105,107,109,111,113,115,117,119,121,123,125, 127, and 129 are used for current limiting and thus affect the turn-on Resistance of the SSR's on the Outputs (if SSR is used) Size to keep current draw below Pin Max current capability, and to not overdrive SSR Diode"
- note added: "R8,10,12,14,21,23,25,27,29,38,40,42,44,46,48,49, and 50 are used as Pull-Up Resistors, when configured as Digital Inputs (Using Opto Isolator, Pin cofigured as High Input = 0, Low Input = 1)"
- note added: "Remove JP1 for Programming Operations"
- note added: "Resistors R3 to R7, R16 to R20, and R31 to R37, are Current limiting Resistors used when Input is a Digital, Analoge Inputs use a 0 Ohm Resistor here."
- note added: "VDD IS LIMITED TO 3.3 VOLTS!!!!!!"
- note added: "ZIF1 is used to attach Touch Screen, If used do not populate R34,35,36,37,44,45,46,47, R48,49, C22,C23,C24,C25, D13, or D14."
- note added: "Zener Diodes D1 to D14 used for OverVoltage and Reverse Polarity protection , when configured for Analog Input."
- moved on the sheet: D10, D11, D12, D13, D14, D3, D4, D5, D6, D7, D8, D9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
