File: PCB/PIC64-Final/64Pin-Final.brd (EAGLE design)
At the start: 100 x 80 mm, 179 parts, among them IC1 , IC2 , IC3 , IC4 , J1 84952-4, Q1 , Q2 IRF540, Q3 IRF540, Q4 IRF540, U1 LM5114BMFX/S7003094SOT26-GATE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, U2 LM5114BMFX/S7003094SOT26-GATE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, U3 LM5114BMFX/S7003094SOT26-GATE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, U4 282837-3, U5 282837-3, X2 , X3 , X4 , X5 , X7 , X8 , X9 

Commit message: AtOrd
Parts:
- removed D16, D17: (no value), zetex:SOD323
- removed Q4: IRF540, transistor-power:TO220BV
- removed R61, R62, R63: (no value), resistor:R0603
- added BRIGHTNESS: (no value), rcl:RTRIM3296W
- added OSC: (no value), crystal:TC26H
- added R3, R53: (no value), resistor:R0603
- added SOC1, SOC2: (no value), ic-package:DIL20
- D1, D2: device ic-package:DIL20 -> 0603ZenerDiode:CZRU-M
- D14: device zetex:SOD323 -> 0603ZenerDiode:CZRU-M
- DR1, DR2, DR3: value LM5114BMFX/S7003094SOT26-GATEDRIVER -> (none)
- Q1: device crystal:TC26H -> transistor-power:TO220BV
- Q2, Q3: value IRF540 -> (none)
- R52: device rcl:RTRIM3296W -> resistor:R0603
- TERM1, TERM2: value 282837-3 -> (none)
- moved R50 75.1 mm to (90.0, 55.8), flipped to the bottom, turned to 0 degrees
- moved R51 68.1 mm to (71.0, 32.5), turned to 0 degrees
- moved R52 43.0 mm to (71.0, 30.2)
- moved Q1 35.4 mm to (79.8, 35.5), flipped to the top, turned to 0 degrees
- moved R20 29.3 mm to (44.0, 71.5)
- moved D2 26.4 mm to (78.9, 58.0), flipped to the bottom, turned to 0 degrees
- moved R35 24.1 mm to (19.1, 71.6), turned to 0 degrees
- moved R19 22.9 mm to (49.5, 71.5)
- moved R18 22.5 mm to (55.0, 71.5), flipped to the top, turned to 0 degrees
- moved R34 22.5 mm to (24.1, 71.6)
- moved R33 21.8 mm to (29.2, 71.6), turned to 0 degrees
- moved R25 20.8 mm to (55.0, 51.4)
- moved R42 20.8 mm to (26.9, 51.0), turned to 270 degrees
- moved R37 20.3 mm to (7.64, 57.5), turned to 90 degrees
- moved R32 20.3 mm to (34.3, 71.6)
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- renumbered D15 to SOC3, IC1 to SOC7, IC2 to SOC6, IC3 to SOC5, IC4 to SOC4, J1 to ZIF1, R67 to R129, R68 to R128, R69 to R127, R70 to R126, R71 to R125, R72 to R124, R73 to R123, R74 to R122, R75 to R121, R76 to R120, R77 to R119, R78 to R118, R79 to R117, R80 to R116, R81 to R115, R82 to R114, R83 to R113, R84 to R112, R85 to R111, R86 to R110, R87 to R109, R88 to R108, R89 to R107, R90 to R106, R91 to R105, R92 to R104, R93 to R103, R94 to R102, R95 to R101, R96 to R100, U1 to DR1, U2 to DR2, U3 to DR3, U4 to TERM2, U5 to TERM1, X2 to INPUTS-4, X3 to INPUTS-3, X4 to INPUTS-2, X5 to OUTPUTS-2, X7 to OUTPUTS-1, X8 to INPUTS-1, X9 to OUTPUTS-3
Connections:
- net N$100: now also R20.2; no longer R26.2
- net N$101: now also R19.2; no longer R25.2
- net N$102: now also SOC2.6; no longer D2.6
- net N$103: now also R19.1, SOC2.7; no longer D2.7, R25.1
- net N$104: now also SOC2.4; no longer D2.4
- net N$105: now also R17.1, SOC2.3; no longer D2.3, R23.1
- net N$106: now also R17.2; no longer R23.2
- net N$107: now also SOC2.2; no longer D2.2
- net N$108: now also SOC2.1; no longer D2.1
- net N$11: now also R36.2; no longer R48.2
- net N$110: now also SOC1.10; no longer D1.10
- net N$111: now also R7.2; no longer R13.2
- net N$112: now also R7.1, SOC1.9; no longer D1.9, R13.1
- net N$113: now also SOC1.8; no longer D1.8
- net N$114: now also R18.1, SOC2.5; no longer D2.5, R24.1
- net N$115: now also R18.2; no longer R24.2
- net N$116: now also R5.2; no longer R7.2
- net N$117: now also R5.1, SOC1.5; no longer D1.5, R7.1
- net N$118: now also SOC1.4; no longer D1.4
- net N$119: now also R4.2; no longer R6.2
- net N$120: now also R4.1, SOC1.3; no longer D1.3, R6.1
- net N$121: now also SOC1.2; no longer D1.2
- net N$122: now also R3.2; no longer R4.2
- net N$123: now also R3.1, SOC1.1; no longer D1.1, R4.1
- net N$19: now also R36.1; no longer R48.1
- net N$21: now also R37.1; no longer R51.1
- net N$23: now also R35.2; no longer R43.2
- net N$25: now also R34.2; no longer R42.2
- net N$28: now also R33.2; no longer R41.2
- net N$30: now also R32.2; no longer R40.2
- net N$32: now also R31.2; no longer R39.2
- net N$33: now also R54.1; no longer R57.1
- net N$34: now also R53.1; no longer R58.1
- net N$35: now also R52.1; no longer R55.1
- net N$41: now also R51.1; no longer R56.1
- net N$44: now also SOC1.6; no longer D1.6
- net N$45: now also R6.2; no longer R10.2
- net N$46: now also Q3.D; no longer Q4.D
- net N$48: now also Q1.G, R51.2, R52.2; no longer Q2.G, R55.2, R56.2
- net N$5: now also R37.2; no longer R51.2
- net N$50: now also Q2.G, R53.2, R54.2; no longer Q3.G, R57.2, R58.2
- net N$52: now also R56.1; no longer R59.1
- net N$54: now also R6.1, SOC1.7; no longer D1.7, R10.1
- net N$59: now also R55.1; no longer R60.1
- net N$61: now also Q3.G, R55.2, R56.2; no longer Q4.G, R59.2, R60.2
- net N$65: now also Q2.D; no longer Q3.D
- net N$74: now also Q1.D; no longer Q2.D
- net N$75: now also BRIGHTNESS.1; no longer R52.1
- net N$76: now also BRIGHTNESS.2, BRIGHTNESS.3; no longer R52.2, R52.3
- net N$77: now also R57.2; no longer R61.2
- net N$78: now also R58.2; no longer R62.2
- net N$79: now also R59.2; no longer R63.2
- net N$80: now also R58.1; no longer R62.1
- net N$81: now also R59.1; no longer R63.1
- net N$84: now also R35.1; no longer R43.1
- net N$87: now also R34.1; no longer R42.1
- net N$90: now also R33.1; no longer R41.1
- net N$93: now also R32.1; no longer R40.1
- net N$95: now also R31.1; no longer R39.1
- net N$96: now also SOC2.10; no longer D2.10
- net N$98: now also R20.1, SOC2.9; no longer D2.9, R26.1
- net N$99: now also SOC2.8; no longer D2.8
- net OUT: now also R60.2; no longer R54.2
- net PIN11: now also D1.1, SOC1.18; no longer D1.18, D3.1
- net PIN12: now also D2.1, R10.1, R11.2, SOC1.16; no longer D1.16, D4.1, R11.1, R12.2
- net PIN13: now also D3.1, R12.1, R13.2, SOC1.14; no longer D1.14, D5.1, R14.1, R15.2
- net PIN14: now also D4.1, R14.1, R15.2, SOC1.12; no longer D1.12, D6.1, R17.1, R18.2
- net PIN17: now also D5.1, R21.1, R22.2, SOC2.20; no longer D2.20, D7.1, R20.1, R21.2
- net PIN18: now also D6.1, R23.1, R24.2, SOC2.18; no longer D2.18, D8.1, R19.1, R22.2
- net PIN21: now also D7.1, R25.1, R26.2, SOC2.16; no longer D2.16, D9.1, R27.1, R28.2
- net PIN22: now also D8.1, R27.1, R28.2, SOC2.14; no longer D10.1, D2.14, R29.1, R30.2
- net PIN23: now also D9.1, R29.1, R30.2, SOC2.12; no longer D11.1, D2.12, R31.1, R32.2
- net PIN24: now also D10.1, R38.1, R39.2; no longer D12.1, R33.1, R34.2
- net PIN27: now also D11.1, R40.1, R41.2; no longer D13.1, R35.1, R36.2
- net PIN28: now also D12.1, R42.1, R43.2; no longer D14.1, R37.1, R38.2
- net PIN29: now also D13.1; no longer D16.1
- net PIN30: now also D14.1; no longer D17.1
- net PIN31: now also R49.1; no longer R50.1
- net PIN32: now also R48.1; no longer R49.1
- net PIN54: now also R57.1, R60.1; no longer R54.1, R61.1
- net PIN8: now also R50.1, SOC1.20; no longer D1.20, R5.1
- net SOSCI: now also OSC.1; no longer Q1.1
- net SOSCO: now also OSC.2; no longer Q1.2
- net VDD: now also R10.2, R12.2, R21.2, R23.2, R25.2, R38.2, R40.2, R42.2, R48.2; no longer R11.2, R17.2, R19.2, R20.2, R31.2, R33.2, R35.2, R37.2, R5.2
- net VSS: now also D1.2, D2.2, Q1.S, R11.1, R13.1, R24.1, R26.1, R39.1, R41.1, R43.1, SOC1.11, SOC1.13, SOC1.15, SOC1.17, SOC1.19, SOC2.11, SOC2.13, SOC2.15, SOC2.17, SOC2.19; no longer D1.11, D1.13, D1.15, D1.17, D1.19, D16.2, D17.2, D2.11, D2.13, D2.15, D2.17, D2.19, Q4.S, R12.1, R18.1, R21.1, R32.1, R34.1, R36.1, R38.1
Routing:
- net VSS: track 610.6 -> 604.0 mm
Other:
- board text added: "1"
- board text added: "Dave Zieglgansberger Aug 2017, Rev 1.0"
