File: PCB/PIC64-Final/64Pin-Final.sch (EAGLE design)
At the start: 175 parts, among them Q1 , Q2 Dave Ziegl, Q3 R1.0 Aug/2017

Commit message: AtOrd
Parts:
- Q2: value Dave Ziegl -> (none)
- Q3: value R1.0 Aug/2017 -> (none)
Other:
- note added: "LCD Header is Female 20 Pin header, on back side of board, Pin 19 is connected through Brightness Pot, to POWER-1, Pin 20 is connected directly to POWER-2. Connect +5V to POWER-1 and GND to POWER-2 for Display with LED Backlighting, or EL Driver (or 120VAC) to POWER-1 and 2."
- note removed: "LCD Header is Female 20 Pin header, on bach side of board, Pin 19 is connected through Brightness Pot, to POWER-1, Pin 20 is connected directly to POWER-2. Connect +5V to POWER-1 and GND to POWER-2 for Display with LED Backlighting, or EL Driver (or 120VAC) to POWER-1 and 2."
Changed lines of the file:
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@@
 <setting verticaltext="up"/>
 </settings>
-<grid distance="0.05" unitdist="inch" unit="inch" style="lines" multiple="1" display="no" altdistance="0.01" altunitdist="inch" altunit="inch"/>
+<grid distance="0.1" unitdist="inch" unit="inch" style="lines" multiple="1" display="no" altdistance="0.01" altunitdist="inch" altunit="inch"/>
 <layers>
 <layer number="1" name="Top" color="4" fill="1" visible="no" active="no"/>
@@
 <part name="R52" library="resistor" deviceset="R-US_" device="R0603" value=" "/>
 <part name="R51" library="resistor" deviceset="R-US_" device="R0603" value=" "/>
-<part name="Q2" library="transistor-power" deviceset="IRF540" device="" value="Dave Ziegl"/>
+<part name="Q2" library="transistor-power" deviceset="IRF540" device="" value=" "/>
 <part name="Q1" library="transistor-power" deviceset="IRF540" device="" value=" "/>
-<part name="Q3" library="transistor-power" deviceset="IRF540" device="" value="R1.0 Aug/2017"/>
+<part name="Q3" library="transistor-power" deviceset="IRF540" device="" value=" "/>
 <part name="DR2" library="SOT26" deviceset="LM5114BMFX/S7003094" device="SOT26-GATEDRIVER" value=" "/>
 <part name="DR3" library="SOT26" deviceset="LM5114BMFX/S7003094" device="SOT26-GATEDRIVER" value=" "/>
@@
 as Digital Inputs (Using Opto Isolator, Pin cofigured as
 High Input = 0, Low Input = 1)</text>
-<text x="187.96" y="-199.39" size="1.778" layer="91">LCD Header is Female 20 Pin header, on bach side of board,
+<text x="187.96" y="-199.39" size="1.778" layer="91">LCD Header is Female 20 Pin header, on back side of board,
 Pin 19 is connected through Brightness Pot, to POWER-1,
 Pin 20 is connected directly to POWER-2.
