File: PCB/MPPT/MPPT.brd (EAGLE design)
At the start: 3 parts, among them IC1 ACS711KEXLT-15AB-T, IC2 ACS711KEXLT-15AB-T

Commit message: Start of Board Design
Parts:
- added C1, C2, C3, C4: 100nF, resistor:C0603
- added IC3, IC4: ACS711KEXLT-15AB-T, SamacSys_Parts:EX-PACKAGE
- added R1, R3, R5, R7: 100K, resistor:R0603
- added R2, R4, R6, R8: 20K, resistor:R0603
- moved IC1 31.4 mm to (30.5, 58.4), turned to 270 degrees
- moved IC2 25.7 mm to (43.2, 58.4), turned to 270 degrees
- moved U$1 1.44 mm to (50.8, 73.7)
Connections:
- new net N$1: C1.2, R1.1, R2.1
- new net N$2: C2.1, IC2.2, R4.1, U$1.PAD3
- new net N$3: IC2.1, R3.1, U$1.PAD4
- new net N$4: C2.2, R3.2, R4.2
- new net N$5: C3.2, R5.1, R6.2
- new net N$6: C4.2, R7.2, R8.1
- new net N$7: IC4.1, R7.1, U$1.PAD10
- new net N$8: C4.1, IC4.2, R8.2, U$1.PAD9
- new net N$B_1+: IC3.1, R5.2, U$1.PAD8
- new net N$B_1-: C3.1, IC3.2, R6.1, U$1.PAD7
- new net N$PV_1+: IC1.1, R1.2, U$1.PAD2
- new net N$PV_1-: C1.1, IC1.2, R2.2, U$1.PAD1
- new net VDD: IC1.10, IC2.10, IC3.10, IC4.10
- new net VSS: IC1.3, IC2.3, IC3.3, IC4.3

Commit message: progress
Parts:
- added BUCK1_IN+, BUCK1_IN-, BUCK1_OUT+, BUCK1_OUT-, BUCK2_IN+, BUCK2_IN-, BUCK2_OUT+, BUCK2_OUT-: (no value), wirepad:3,81/1,4
- renumbered IC1 to PV_1_I_SENSE, IC2 to BATT_1_I_SENSE
Connections:
- removed net N$5 (its old number): C3.2, R5.1, R6.2
- removed net N$B_1+: IC3.1, R5.2, U$1.PAD8
- removed net N$B_1-: C3.1, IC3.2, R6.1, U$1.PAD7
- removed net N$PV_1+: PV_1_I_SENSE.1, R1.2, U$1.PAD2
- removed net N$PV_1-: C1.1, PV_1_I_SENSE.2, R2.2, U$1.PAD1
- new net N$10: C3.2, R5.2, R6.2
- new net N$11: IC4.2, R7.2, U$1.PAD10
- new net N$12: C4.2, R7.1, R8.2
- new net N$4: BATT_1_I_SENSE.1, BUCK1_OUT+.1
- new net N$9: BUCK2_IN+.1, IC3.2
- net N$1: now also PV_1_I_SENSE.1, U$1.PAD1; no longer C1.2, R1.1, R2.1
- net N$2: now also BUCK1_IN+.1, PV_1_I_SENSE.2, R1.2; no longer BATT_1_I_SENSE.2, C2.1, R4.1, U$1.PAD3
- net N$3: now also C1.2, R1.1, R2.2; no longer BATT_1_I_SENSE.1, R3.1, U$1.PAD4
- net N$6: now also BATT_1_I_SENSE.2, R3.1, U$1.PAD4; no longer C4.2, R7.2, R8.1
- net N$7: now also BUCK2_OUT+.1; no longer R7.1, U$1.PAD10
- net N$8: now also IC3.1, R5.1, U$1.PAD7; no longer C4.1, IC4.2, R8.2, U$1.PAD9
- net VSS: now also BATT_1_I_SENSE.4, BUCK1_IN-.1, BUCK1_OUT-.1, BUCK2_IN-.1, BUCK2_OUT-.1, C1.1, C2.1, C3.1, C4.1, R2.1, R4.1, R6.1, R8.1, U$1.PAD2, U$1.PAD3, U$1.PAD8, U$1.PAD9; no longer IC4.3

Commit message: sc
Parts:
- moved BUCK2_OUT+ 147.3 mm to (88.9, 61.0), turned to 90 degrees
- moved BUCK2_OUT- 138.2 mm to (83.8, 61.0), turned to 90 degrees
- moved BUCK2_IN- 129.0 mm to (78.7, 61.0), turned to 90 degrees
- moved BUCK2_IN+ 119.9 mm to (73.7, 61.0), turned to 90 degrees
- moved BUCK1_OUT+ 91.8 mm to (25.4, 61.0), turned to 90 degrees
- moved BUCK1_OUT- 83.2 mm to (20.3, 61.0), turned to 90 degrees
- moved BUCK1_IN+ 74.7 mm to (15.2, 61.0), turned to 90 degrees
- moved BUCK1_IN- 66.5 mm to (10.2, 61.0), turned to 90 degrees
- moved R6 12.7 mm to (57.1, 50.8)
- moved C3 12.7 mm to (57.1, 47.0)
- moved C1 10.2 mm to (25.4, 49.5)
- moved R2 10.2 mm to (25.4, 53.3)
- moved R5 7.18 mm to (57.1, 58.4)
- moved IC4 5.68 mm to (69.8, 53.3)
- moved IC3 5.08 mm to (62.2, 53.3)
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Connections:
- removed net N$2: BUCK1_IN+.1, PV_1_I_SENSE.2, R1.2
- new net N$13: BUCK1_IN+.1, PV_1_I_SENSE.2
- net N$1: now also R1.1
- net N$3: now also R1.2, R2.1; no longer R1.1, R2.2
- net VSS: now also IC4.3, R2.2; no longer BATT_1_I_SENSE.4, R2.1

Commit message: BP
Parts:
- added R10, R11, R12, R13, R14, R15, R16, R17, R18, R19, R20, R21, R22, R23, R24, R9: 20K, resistor:R0603
- added U1: PIC16F18855-X/SS, 16F18855_SSOP:SSOP28_MC
- added U2, U3: LM324PWR, LM324PWR:PW14
Connections:
- new net N$14: R15.1, R16.2, U2.9
- new net N$15: R10.1, U2.1
- new net N$16: R11.1, R12.2, U2.6
- new net N$17: R12.1, U2.7
- new net N$18: R13.1, R14.2, U2.13
- new net N$19: R10.2, R9.1, U2.2
- new net N$2: PV_1_I_SENSE.9, U2.5
- new net N$20: R13.2, U2.14
- new net N$21: R15.2, U2.8
- new net N$22: BATT_1_I_SENSE.9, U2.12
- new net N$24: R18.1, U3.1
- new net N$25: R20.1, U3.7
- new net N$26: R19.1, R20.2, U3.6
- new net N$27: R21.2, U3.14
- new net N$28: R21.1, R22.2, U3.13
- new net N$29: R23.2, U3.8
- new net N$30: R23.1, R24.2, U3.9
- new net N$31: R17.1, R18.2, U3.2
- new net N$32: IC3.9, U3.5
- new net N$33: IC4.9, U3.12
- net N$10: now also U3.3
- net N$12: now also U3.10
- net N$3: now also U2.3
- net N$5: now also U2.10
- net VDD: now also U1.20, U2.4, U3.4
- net VSS: now also R11.2, R14.1, R16.1, R17.2, R19.2, R22.1, R24.1, R9.2, U1.19, U1.8, U2.11, U3.11

Commit message: CO
Parts:
- added BUCK: TINY_BUCK, Tiny_Buck:TINY_BUCK
- added LCD: (no value), con-lsta:FE08
- added R25, R26: 1K, resistor:R0603
- renumbered U1 to CONTROLLER, U2 to BUFFER1, U3 to BUFFER2
Connections:
- new net IN-: BUCK.IN-
- new net N$23: CONTROLLER.2, LCD.1
- new net N$34: CONTROLLER.3, LCD.2
- new net N$35: CONTROLLER.4, LCD.3
- new net N$36: CONTROLLER.5, LCD.4
- new net N$37: CONTROLLER.6, LCD.5
- new net N$38: LCD.7, R25.1, R26.2
- new net N$39: BUCK.IN+
- new net OUT+: BUCK.OUT+
- new net OUT-: BUCK.OUT-
- net VDD: now also LCD.6, R25.2
- net VSS: now also LCD.8, R26.1

Commit message: gfcr
Parts:
- removed BUCK: TINY_BUCK, Tiny_Buck:TINY_BUCK
- added 3.3V_BUCK: TINY_BUCK, Tiny_Buck:TINY_BUCK
- added C5, C6, C7: 100nF, resistor:C0603
- added PROGRAM: Pin 1, con-lstb:MA08-1
- added SV2: (no value), con-lstb:MA04-1
- moved R26 174.5 mm to (97.8, 25.4), turned to 270 degrees
- moved R25 166.7 mm to (97.8, 20.3), turned to 270 degrees
- moved R24 159.2 mm to (78.7, 38.1), turned to 270 degrees
- moved R22 154.0 mm to (78.7, 41.9), turned to 90 degrees
- moved R23 152.9 mm to (74.9, 38.1), turned to 180 degrees
- moved LCD 149.2 mm to (92.7, 15.2), turned to 90 degrees
- moved R21 148.7 mm to (74.9, 43.2), turned to 180 degrees
- moved R20 132.9 mm to (59.7, 39.4)
- moved R18 129.3 mm to (82.5, 26.7), turned to 180 degrees
- moved R19 121.6 mm to (45.7, 39.4)
- moved BUFFER2 120.2 mm to (67.3, 40.6)
- moved R17 119.8 mm to (53.3, 43.2), turned to 180 degrees
- moved R16 97.9 mm to (44.5, 35.6), turned to 180 degrees
- moved R14 95.5 mm to (45.7, 41.9), turned to 180 degrees
- moved R15 95.5 mm to (41.9, 39.4), turned to 180 degrees
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Connections:
- removed net IN-: BUCK.IN-
- removed net N$39: BUCK.IN+
- removed net OUT+: BUCK.OUT+
- removed net OUT-: BUCK.OUT-
- net N$15: now also CONTROLLER.18
- net N$17: now also CONTROLLER.17
- net N$20: now also CONTROLLER.15
- net N$21: now also CONTROLLER.16
- net N$24: now also CONTROLLER.14
- net N$25: now also CONTROLLER.13
- net N$27: now also CONTROLLER.11
- net N$29: now also CONTROLLER.12
- net N$6: now also 3.3V_BUCK.IN+
- net VDD: now also 3.3V_BUCK.OUT+, C5.2, C6.2, C7.2
- net VSS: now also 3.3V_BUCK.IN-, 3.3V_BUCK.OUT-, C5.1, C6.1, C7.1

Commit message: sog
Parts:
- moved R18 30.0 mm to (58.4, 44.5)
- moved IC4 24.7 mm to (87.6, 70.5)
- moved R7 16.5 mm to (82.5, 71.1), turned to 90 degrees
- moved C4 16.1 mm to (78.7, 66.0)
- moved R8 16.1 mm to (78.7, 69.8)
- moved IC3 9.86 mm to (64.8, 62.9), turned to 90 degrees
- moved R19 8.26 mm to (54.0, 39.4)
- moved C2 3.81 mm to (47.0, 61.0)
- moved R4 3.81 mm to (43.2, 61.0)
- moved C5 3.70 mm to (42.5, 19.7)
- moved C7 3.70 mm to (51.4, 19.7)
- moved C6 3.17 mm to (47.0, 19.7)
- moved R16 2.29 mm to (45.7, 37.5)
- moved R10 1.91 mm to (26.7, 43.8)
- moved R13 1.91 mm to (41.9, 43.8)
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Routing:
- net N$15: track 0.00 -> 76.4 mm
- net N$20: track 0.00 -> 47.8 mm
- net N$17: track 0.00 -> 46.4 mm
- net N$21: track 0.00 -> 33.1 mm
- net N$3: track 0.00 -> 30.4 mm, vias 0 -> 2
- net N$2: track 0.00 -> 23.1 mm, vias 0 -> 2
- net N$4: track 0.00 -> 22.8 mm, vias 0 -> 1
- net N$13: track 0.00 -> 19.9 mm
- net N$11: track 0.00 -> 18.9 mm
- net N$8: track 0.00 -> 18.8 mm
- net VDD: track 0.00 -> 18.7 mm, vias 0 -> 2
- net N$6: track 0.00 -> 18.0 mm
- net N$1: track 0.00 -> 16.5 mm
- net N$7: track 0.00 -> 15.7 mm
- net N$19: track 0.00 -> 9.18 mm
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- added copper zone on layer 1, net VSS

Commit message: cly
Parts:
- moved R2 4.02 mm to (36.8, 57.1)
- moved C1 3.86 mm to (31.1, 57.1)
- moved R1 2.29 mm to (31.1, 63.5)
- moved R3 1.91 mm to (42.5, 64.8)
- moved R4 1.27 mm to (44.5, 61.0)
- moved C2 1.27 mm to (48.3, 61.0)
Routing:
- net N$1: track 16.5 -> 17.8 mm
- net N$6: track 18.0 -> 19.1 mm
- net N$5: track 8.09 -> 9.20 mm
