File: PCB/MPPT/MPPT.brd (EAGLE design)
At the start: 53 parts, among them IC3 ACS711KEXLT-15AB-T, IC4 ACS711KEXLT-15AB-T

Commit message: qc
Parts:
- removed PROGRAM: Pin 1, con-lstb:MA08-1
- removed SV2: (no value), con-lstb:MA04-1
- added R27: 10K, rcl:R1206
- added R28: 10K, resistor:R0603
- added U$2, U$3, U$4, U$5: (no value), holes:4,5
- added X1, X2: 22-23-2021, con-molex:22-23-2021
- added X3: 22-23-2041, con-molex:22-23-2041
- moved R25 18.9 mm to (80.0, 14.0), turned to 180 degrees
- moved R26 18.1 mm to (83.8, 14.0), turned to 180 degrees
- moved LCD 17.3 mm to (76.2, 10.2), turned to 0 degrees
- moved 3.3V_BUCK 9.55 mm to (15.9, 17.1)
- moved R19 2.29 mm to (55.2, 37.5), turned to 180 degrees
- moved R7 2.25 mm to (82.9, 68.9)
- moved R22 2.01 mm to (79.4, 43.8), turned to 180 degrees
- moved R17 2.01 mm to (55.2, 43.8)
- moved R20 1.90 mm to (59.7, 37.5), turned to 180 degrees
- moved IC4 1.80 mm to (86.4, 69.2)
- moved R18 1.42 mm to (59.7, 43.8)
- moved C4 1.27 mm to (78.7, 64.8)
- moved R8 1.27 mm to (78.7, 68.6)
- moved R24 0.90 mm to (79.4, 37.5), turned to 180 degrees
- moved R21 0.90 mm to (75.6, 43.8)
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Connections:
- new net N$39: CONTROLLER.22, R28.2, X3.2
- new net N$42: CONTROLLER.21, R27.2, X3.4
- net VDD: now also R27.1, R28.1
- net VSS: now also X3.1, X3.3
Routing:
- net VDD: track 18.7 -> 279.2 mm, vias 2 -> 6
- net N$42: track 0.00 -> 131.0 mm
- net N$39: track 0.00 -> 130.3 mm
- net N$6: track 19.1 -> 81.4 mm
- net N$33: track 0.00 -> 43.4 mm
- net N$32: track 0.00 -> 40.6 mm, vias 0 -> 2
- net N$12: track 6.94 -> 44.2 mm, vias 0 -> 2
- net N$27: track 0.00 -> 36.2 mm
- net N$5: track 9.20 -> 40.9 mm, vias 0 -> 2
- net N$10: track 7.83 -> 38.8 mm
- net N$24: track 0.00 -> 28.2 mm
- net N$29: track 0.00 -> 26.4 mm, vias 0 -> 2
- net N$25: track 0.00 -> 25.2 mm
- net N$22: track 0.00 -> 20.4 mm, vias 0 -> 2
- net N$37: track 0.00 -> 11.4 mm
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
Commit message: cy
Parts:
- added PROGRAMMER: (no value), con-lstb:MA06-1
- added R29: 10K, resistor:R0603
- added U$7: (no value), DAVE:DAVE
- renumbered LCD to __LCD
Connections:
- new net N$40: CONTROLLER.1, PROGRAMMER.1, R29.1
- new net N$44: CONTROLLER.28, PROGRAMMER.4
- new net N$45: CONTROLLER.27, PROGRAMMER.5
- net VDD: now also PROGRAMMER.2, R29.2
- net VSS: now also PROGRAMMER.3
Routing:
- net N$45: track 0.00 -> 46.6 mm
- net N$44: track 0.00 -> 43.4 mm
- net N$40: track 0.00 -> 43.3 mm, vias 0 -> 2
- net VDD: track 279.2 -> 297.8 mm
Changed lines of the file:
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@@
 <element name="R23" library="resistor" package="R0603" value="20K" x="75.565" y="37.465" rot="R180"/>
 <element name="R24" library="resistor" package="R0603" value="20K" x="79.375" y="37.465" rot="R180"/>
-<element name="LCD" library="con-lsta" package="FE08" value=" " x="76.2" y="10.16">
+<element name="__LCD" library="con-lsta" package="FE08" value=" " x="76.2" y="10.16">
 <attribute name="MF" value="" x="76.2" y="10.16" size="1.778" layer="27" display="off"/>
 <attribute name="MPN" value="" x="76.2" y="10.16" size="1.778" layer="27" display="off"/>
@@
 <element name="U$4" library="holes" package="4,5" value="" x="6.985" y="6.985"/>
 <element name="U$5" library="holes" package="4,5" value="" x="93.345" y="73.025"/>
+<element name="U$7" library="DAVE" package="DAVE" value="" x="11.43" y="27.94" rot="R90"/>
+<element name="PROGRAMMER" library="con-lstb" package="MA06-1" value=" " x="26.035" y="5.08" rot="R180">
+<attribute name="OC_NEWARK" value="unknown" x="26.035" y="5.08" size="1.778" layer="27" rot="R180" display="off"/>
+<attribute name="MPN" value="" x="26.035" y="5.08" size="1.778" layer="27" rot="R180" display="off"/>
+<attribute name="MF" value="" x="26.035" y="5.08" size="1.778" layer="27" rot="R180" display="off"/>
+<attribute name="OC_FARNELL" value="unknown" x="26.035" y="5.08" size="1.778" layer="27" rot="R180" display="off"/>
+</element>
+<element name="R29" library="resistor" package="R0603" value="10K" x="31.115" y="8.345" rot="R180"/>
 </elements>
 <signals>
@@
 <contactref element="R19" pad="2"/>
 <contactref element="R24" pad="1"/>
-<contactref element="LCD" pad="8"/>
+<contactref element="__LCD" pad="8"/>
 <contactref element="R26" pad="1"/>
 <contactref element="CONTROLLER" pad="8"/>
@@
 <via x="15.24" y="68.2625" extent="1-16" drill="0.8" shape="square"/>
 <via x="17.78" y="57.785" extent="1-16" drill="0.8" shape="square"/>
-<via x="46.99" y="34.925" extent="1-16" drill="0.8" shape="square"/>
-<via x="19.685" y="32.385" extent="1-16" drill="0.8" shape="square"/>
-<via x="33.655" y="32.385" extent="1-16" drill="0.8" shape="square"/>
+<via x="45.72" y="34.925" extent="1-16" drill="0.8" shape="square"/>
+<via x="17.78" y="29.21" extent="1-16" drill="0.8" shape="square"/>
+<via x="36.195" y="29.21" extent="1-16" drill="0.8" shape="square"/>
 <contactref element="C1" pad="1"/>
 <contactref element="X3" pad="1"/>
@@
 <via x="68.2625" y="29.5275" extent="1-16" drill="0.6" shape="square"/>
 <via x="4.445" y="43.815" extent="1-16" drill="0.5" shape="square"/>
+<contactref element="PROGRAMMER" pad="3"/>
 </signal>
 <signal name="VDD">
@@
 <contactref element="BUFFER2" pad="4"/>
 <contactref element="CONTROLLER" pad="20"/>
-<contactref element="LCD" pad="6"/>
+<contactref element="__LCD" pad="6"/>
 <contactref element="R25" pad="2"/>
 <contactref element="3.3V_BUCK" pad="OUT+"/>
@@
 <wire x1="71.12" y1="75.565" x2="80.01" y2="75.565" width="0.3048" layer="16"/>
 <wire x1="80.01" y1="75.565" x2="86.36" y2="69.215" width="0.3048" layer="16"/>
+<contactref element="R29" pad="2"/>
+<contactref element="PROGRAMMER" pad="2"/>
+<wire x1="30.265" y1="8.345" x2="29.845" y2="5.08" width="0.3048" layer="1"/>
+<wire x1="36.075" y1="19.045" x2="29.845" y2="5.08" width="0.3048" layer="16"/>
 </signal>
 <signal name="N$3">
@@
 <wire x1="41.06" y1="43.815" x2="41.06" y2="45.505" width="0.3048" layer="1"/>
 <wire x1="41.06" y1="45.505" x2="42.545" y2="46.99" width="0.3048" layer="1"/>
-<wire x1="42.545" y1="46.99" x2="47.625" y2="46.99" width="0.3048" layer="1"/>
-<wire x1="47.625" y1="46.99" x2="50.165" y2="44.45" width="0.3048" layer="1"/>
-<wire x1="50.165" y1="44.45" x2="50.165" y2="28.575" width="0.3048" layer="1"/>
-<wire x1="50.165" y1="28.575" x2="56.515" y2="22.225" width="0.3048" layer="1"/>
+<wire x1="42.545" y1="46.99" x2="46.99" y2="46.99" width="0.3048" layer="1"/>
+<wire x1="46.99" y1="46.99" x2="48.26" y2="45.72" width="0.3048" layer="1"/>
+<wire x1="48.26" y1="45.72" x2="48.26" y2="30.48" width="0.3048" layer="1"/>
+<wire x1="48.26" y1="30.48" x2="56.515" y2="22.225" width="0.3048" layer="1"/>
 <wire x1="56.515" y1="22.225" x2="62.200509375" y2="22.225" width="0.3048" layer="1"/>
 <wire x1="62.200509375" y1="22.225" x2="62.4205" y2="22.005009375" width="0.3048" layer="1"/>
@@
 <signal name="N$23">
 <contactref element="CONTROLLER" pad="2"/>
-<contactref element="LCD" pad="1"/>
+<contactref element="__LCD" pad="1"/>
 <wire x1="69.6595" y1="14.205" x2="68.205" y2="14.205" width="0.4064" layer="1"/>
 <wire x1="68.205" y1="14.205" x2="67" y2="13" width="0.4064" layer="1"/>
@@
 <signal name="N$34">
 <contactref element="CONTROLLER" pad="3"/>
-<contactref element="LCD" pad="2"/>
+<contactref element="__LCD" pad="2"/>
 <wire x1="69.6595" y1="14.8549875" x2="71.1450125" y2="14.8549875" width="0.4064" layer="1"/>
 <wire x1="71.1450125" y1="14.8549875" x2="72" y2="14" width="0.4064" layer="1"/>
@@
 <signal name="N$35">
 <contactref element="CONTROLLER" pad="4"/>
-<contactref element="LCD" pad="3"/>
+<contactref element="__LCD" pad="3"/>
 <wire x1="69.6595" y1="15.504996875" x2="71.495003125" y2="15.504996875" width="0.4064" layer="1"/>
 <wire x1="71.495003125" y1="15.504996875" x2="73" y2="14" width="0.4064" layer="1"/>
@@
 <signal name="N$36">
 <contactref element="CONTROLLER" pad="5"/>
-<contactref element="LCD" pad="4"/>
+<contactref element="__LCD" pad="4"/>
 <wire x1="69.6595" y1="16.155009375" x2="71.844990625" y2="16.155009375" width="0.4064" layer="1"/>
 <wire x1="71.844990625" y1="16.155009375" x2="75" y2="13" width="0.4064" layer="1"/>
@@
 <signal name="N$37">
 <contactref element="CONTROLLER" pad="6"/>
-<contactref element="LCD" pad="5"/>
+<contactref element="__LCD" pad="5"/>
 <wire x1="69.6595" y1="16.804996875" x2="72.195003125" y2="16.804996875" width="0.4064" layer="1"/>
 <wire x1="72.195003125" y1="16.804996875" x2="77" y2="12" width="0.4064" layer="1"/>
@@
 <contactref element="R25" pad="1"/>
 <contactref element="R26" pad="2"/>
-<contactref element="LCD" pad="7"/>
+<contactref element="__LCD" pad="7"/>
 <wire x1="82.55" y1="10.16" x2="82.55" y2="10.45" width="0.4064" layer="1"/>
 <wire x1="82.55" y1="10.45" x2="81" y2="12" width="0.4064" layer="1"/>
@@
 <wire x1="21.9075" y1="65.0875" x2="21.9075" y2="76.2" width="0.4064" layer="1"/>
 </signal>
+<signal name="N$40">
+<contactref element="PROGRAMMER" pad="1"/>
+<contactref element="CONTROLLER" pad="1"/>
+<contactref element="R29" pad="1"/>
+<wire x1="69.6595" y1="13.554990625" x2="69.215" y2="12.7" width="0.3048" layer="1"/>
+<via x="69.215" y="12.7" extent="1-16" drill="0.5" shape="square"/>
+<wire x1="69.215" y1="12.7" x2="60.325" y2="12.7" width="0.3048" layer="16"/>
+<via x="60.325" y="12.7" extent="1-16" drill="0.5" shape="square"/>
+<wire x1="60.325" y1="12.7" x2="55.88" y2="8.255" width="0.3048" layer="1"/>
+<wire x1="55.88" y1="8.255" x2="31.965" y2="8.345" width="0.3048" layer="1"/>
+<wire x1="31.965" y1="8.345" x2="32.385" y2="5.08" width="0.3048" layer="1"/>
+</signal>
+<signal name="N$44">
+<contactref element="PROGRAMMER" pad="4"/>
+<contactref element="CONTROLLER" pad="28"/>
+<wire x1="62.4205" y1="13.554990625" x2="59.274990625" y2="13.554990625" width="0.3048" layer="1"/>
+<wire x1="59.274990625" y1="13.554990625" x2="55.245" y2="9.525" width="0.3048" layer="1"/>
+<wire x1="55.245" y1="9.525" x2="25.4" y2="9.525" width="0.3048" layer="1"/>
+<wire x1="25.4" y1="9.525" x2="24.765" y2="8.89" width="0.3048" layer="1"/>
+<wire x1="24.765" y1="8.89" x2="24.765" y2="5.08" width="0.3048" layer="1"/>
+</signal>
+<signal name="N$45">
+<contactref element="PROGRAMMER" pad="5"/>
+<contactref element="CONTROLLER" pad="27"/>
+<wire x1="62.4205" y1="14.205" x2="58.655" y2="14.205" width="0.3048" layer="1"/>
+<wire x1="58.655" y1="14.205" x2="55.245" y2="10.795" width="0.3048" layer="1"/>
+<wire x1="55.245" y1="10.795" x2="23.495" y2="10.795" width="0.3048" layer="1"/>
+<wire x1="23.495" y1="10.795" x2="22.225" y2="9.525" width="0.3048" layer="1"/>
+<wire x1="22.225" y1="9.525" x2="22.225" y2="5.08" width="0.3048" layer="1"/>
+</signal>
 </signals>
 </board>
 </drawing>
+<compatibility>
+<note version="6.3" minversion="6.2.2" severity="warning">
+Since Version 6.2.2 text objects can contain more than one line,
+which will not be processed correctly with this version.
+</note>
+</compatibility>
 </eagle>

Commit message: cu
Routing:
- net VDD: track 297.8 -> 292.0 mm
- net N$5: track 40.9 -> 39.2 mm
Changed lines of the file:
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@@
 <setting verticaltext="up"/>
 </settings>
-<grid distance="0.635" unitdist="mm" unit="mm" style="lines" multiple="1" display="yes" altdistance="0.025" altunitdist="inch" altunit="mm"/>
+<grid distance="0.635" unitdist="mm" unit="mm" style="lines" multiple="1" display="no" altdistance="0.025" altunitdist="inch" altunit="mm"/>
 <layers>
 <layer number="1" name="Top" color="4" fill="1" visible="yes" active="yes"/>
@@
 <via x="4.445" y="43.815" extent="1-16" drill="0.5" shape="square"/>
 <contactref element="PROGRAMMER" pad="3"/>
+<via x="36.195" y="62.23" extent="1-16" drill="0.8" shape="square"/>
+<via x="10.795" y="52.705" extent="1-16" drill="0.8" shape="square"/>
+<via x="32.385" y="54.61" extent="1-16" drill="0.6" shape="square"/>
 </signal>
 <signal name="VDD">
@@
 <via x="29.5275" y="40.9575" extent="1-16" drill="0.6" shape="square"/>
 <wire x1="29.5275" y1="40.9575" x2="29.5275" y2="50.4825" width="0.3048" layer="16"/>
-<wire x1="29.5275" y1="50.4825" x2="32.385" y2="53.34" width="0.3048" layer="16"/>
-<via x="32.385" y="53.34" extent="1-16" drill="0.6" shape="square"/>
-<wire x1="32.385" y1="53.34" x2="29.54" y2="53.34" width="0.3048" layer="1"/>
+<wire x1="29.5275" y1="50.4825" x2="31.115" y2="53.34" width="0.3048" layer="16"/>
+<via x="31.115" y="53.34" extent="1-16" drill="0.6" shape="square"/>
+<wire x1="31.115" y1="53.34" x2="29.54" y2="53.34" width="0.3048" layer="1"/>
 <wire x1="29.54" y1="53.34" x2="29.39" y2="53.19" width="0.3048" layer="1"/>
 <wire x1="43.36" y1="53.19" x2="42.06" y2="53.19" width="0.3048" layer="1"/>
 <wire x1="42.06" y1="53.19" x2="41.91" y2="53.34" width="0.3048" layer="1"/>
 <via x="41.91" y="53.34" extent="1-16" drill="0.6" shape="square"/>
-<wire x1="41.91" y1="53.34" x2="35.56" y2="53.34" width="0.3048" layer="16"/>
-<wire x1="35.56" y1="53.34" x2="34.925" y2="53.975" width="0.3048" layer="16"/>
-<wire x1="34.925" y1="53.975" x2="34.925" y2="55.88" width="0.3048" layer="16"/>
-<wire x1="34.925" y1="55.88" x2="34.29" y2="56.515" width="0.3048" layer="16"/>
-<wire x1="34.29" y1="56.515" x2="33.02" y2="56.515" width="0.3048" layer="16"/>
-<wire x1="33.02" y1="56.515" x2="32.385" y2="55.88" width="0.3048" layer="16"/>
-<wire x1="32.385" y1="55.88" x2="32.385" y2="53.34" width="0.3048" layer="16"/>
-<wire x1="43.36" y1="53.19" x2="48.745" y2="53.19" width="0.3048" layer="1"/>
-<wire x1="48.745" y1="53.19" x2="50.165" y2="54.61" width="0.3048" layer="1"/>
-<wire x1="50.165" y1="54.61" x2="50.165" y2="73.66" width="0.3048" layer="1"/>
+<wire x1="41.91" y1="53.34" x2="31.115" y2="53.34" width="0.3048" layer="16"/>
+<wire x1="50.165" y1="53.34" x2="50.165" y2="73.66" width="0.3048" layer="1"/>
 <wire x1="50.165" y1="73.66" x2="51.435" y2="74.93" width="0.3048" layer="1"/>
 <wire x1="51.435" y1="74.93" x2="59.055" y2="74.93" width="0.3048" layer="1"/>
@@
 <wire x1="64.4906" y1="40.64" x2="52.07" y2="40.64" width="0.3048" layer="1"/>
 <wire x1="52.07" y1="40.64" x2="51.435" y2="41.275" width="0.3048" layer="1"/>
-<wire x1="51.435" y1="41.275" x2="51.435" y2="53.34" width="0.3048" layer="1"/>
-<wire x1="51.435" y1="53.34" x2="50.165" y2="54.61" width="0.3048" layer="1"/>
+<wire x1="51.435" y1="41.275" x2="51.435" y2="53.19" width="0.3048" layer="1"/>
 <wire x1="42.545" y1="18.835" x2="36.285" y2="18.835" width="0.6096" layer="1"/>
 <wire x1="36.285" y1="18.835" x2="36.075" y2="19.045" width="0.6096" layer="1"/>
@@
 <wire x1="79" y1="8" x2="79" y2="9.15" width="0.4064" layer="1"/>
 <wire x1="79" y1="9.15" x2="80.01" y2="10.16" width="0.4064" layer="1"/>
-<wire x1="32.385" y1="53.34" x2="31.115" y2="54.61" width="0.4064" layer="16"/>
-<wire x1="31.115" y1="54.61" x2="1.27" y2="54.61" width="0.4064" layer="16"/>
+<wire x1="31.115" y1="53.34" x2="29.845" y2="54.61" width="0.4064" layer="16"/>
+<wire x1="29.845" y1="54.61" x2="1.27" y2="54.61" width="0.4064" layer="16"/>
 <via x="1.27" y="54.61" extent="1-16" drill="0.6" shape="square"/>
 <wire x1="1.27" y1="54.61" x2="1.69" y2="55.03" width="0.4064" layer="1"/>
@@
 <wire x1="30.265" y1="8.345" x2="29.845" y2="5.08" width="0.3048" layer="1"/>
 <wire x1="36.075" y1="19.045" x2="29.845" y2="5.08" width="0.3048" layer="16"/>
+<wire x1="43.36" y1="53.19" x2="51.435" y2="53.19" width="0.3048" layer="1"/>
+<wire x1="51.435" y1="53.19" x2="51.435" y2="53.34" width="0.3048" layer="1"/>
+<wire x1="50.165" y1="53.34" x2="51.435" y2="53.34" width="0.3048" layer="1"/>
 </signal>
 <signal name="N$3">
@@
 <wire x1="33.64" y1="41.29" x2="33.655" y2="41.275" width="0.3048" layer="1"/>
 <via x="33.655" y="41.275" extent="1-16" drill="0.6" shape="square"/>
-<wire x1="33.655" y1="41.275" x2="33.655" y2="55.245" width="0.3048" layer="16"/>
-<via x="33.655" y="55.245" extent="1-16" drill="0.6" shape="square"/>
+<wire x1="33.655" y1="41.275" x2="33.655" y2="52.07" width="0.3048" layer="16"/>
+<via x="33.655" y="52.07" extent="1-16" drill="0.6" shape="square"/>
 <contactref element="C1" pad="2"/>
 <wire x1="31.115" y1="58" x2="33.655" y2="58" width="0.3048" layer="1"/>
 <wire x1="33.655" y1="58" x2="36.83" y2="58" width="0.3048" layer="1"/>
-<wire x1="33.655" y1="55.245" x2="33.655" y2="58" width="0.3048" layer="1"/>
+<wire x1="33.655" y1="52.07" x2="33.655" y2="58" width="0.3048" layer="1"/>
 <wire x1="31.115" y1="58" x2="31.115" y2="62.23" width="0.3048" layer="1"/>
 <wire x1="31.115" y1="62.23" x2="31.965" y2="63.5" width="0.3048" layer="1"/>
@@
 <contactref element="C2" pad="2"/>
 <contactref element="BUFFER1" pad="10"/>
-<wire x1="43.395" y1="64.77" x2="42.545" y2="64.77" width="0.3048" layer="1"/>
-<wire x1="42.545" y1="64.77" x2="43.18" y2="64.135" width="0.3048" layer="1"/>
 <wire x1="48.26" y1="61.81" x2="44.45" y2="61.81" width="0.3048" layer="1"/>
 <wire x1="43.395" y1="64.77" x2="43.815" y2="64.77" width="0.3048" layer="1"/>

Commit message: NFpRW
Parts:
- added D1, D2: 1N4004, diode:DO41-10
- added PWM_1, PWM_2: WIREPAD2,54/1,1, wirepad:2,54/1,1
- added R30: 470R, resistor:R0603
- added R31: 470R, resistor:R1206
- added U$8, U$9: (no value), holes:3,3
- moved U$7 19.5 mm to (8.40, 8.64), turned to 0 degrees
- moved R29 19.4 mm to (50.5, 8.24)
- moved PROGRAMMER 19.0 mm to (45.0, 4.98)
- moved U$4 5.35 mm to (3.15, 3.25)
- moved U$2 4.31 mm to (3.15, 75.0)
- moved U$3 3.74 mm to (93.1, 3.25)
- moved X1 2.00 mm to (69.0, 51.0)
- moved X2 2.00 mm to (84.0, 51.0)
- moved U$5 1.99 mm to (93.1, 75.0)
Connections:
- new net N$41: CONTROLLER.10, D2.A, D2.C, R31.2
- new net N$43: CONTROLLER.9, D1.A
- new net N$46: PWM_2.1, R30.1
- new net N$47: D1.C, R30.2
- new net N$48: PWM_1.1, R31.1
Routing:
- net N$41: track 0.00 -> 50.0 mm
- net N$40: track 43.3 -> 23.9 mm
- net N$45: track 46.6 -> 27.3 mm
- net N$44: track 43.4 -> 24.3 mm
- net N$48: track 0.00 -> 11.3 mm
- net N$43: track 0.00 -> 10.1 mm
- net N$46: track 0.00 -> 6.88 mm
- net N$47: track 0.00 -> 2.96 mm
- net N$29: track 26.4 -> 28.4 mm
- net VDD: track 292.0 -> 293.8 mm
- net N$33: track 43.4 -> 44.5 mm
- net N$12: track 44.2 -> 45.2 mm
- net N$27: track 36.2 -> 35.7 mm

Commit message: NM
Routing:
- net VDD: track 293.8 -> 306.7 mm
Changed lines of the file:
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@@
 <contactref element="R29" pad="2"/>
 <contactref element="PROGRAMMER" pad="2"/>
-<wire x1="36.075" y1="19.045" x2="48.845" y2="4.98" width="0.4064" layer="16"/>
 <wire x1="43.36" y1="53.19" x2="51.435" y2="53.19" width="0.3048" layer="1"/>
 <wire x1="51.435" y1="53.19" x2="51.435" y2="53.34" width="0.3048" layer="1"/>
@@
 <wire x1="49.665" y1="8.245" x2="48.845" y2="7.425" width="0.4064" layer="1"/>
 <wire x1="48.845" y1="7.425" x2="48.845" y2="4.98" width="0.4064" layer="1"/>
+<wire x1="36.075" y1="19.045" x2="36.075" y2="3.93" width="0.4064" layer="16"/>
+<wire x1="36.075" y1="3.93" x2="38.735" y2="1.27" width="0.4064" layer="16"/>
+<wire x1="38.735" y1="1.27" x2="47.3075" y2="1.27" width="0.4064" layer="16"/>
+<wire x1="47.3075" y1="1.27" x2="48.895" y2="2.8575" width="0.4064" layer="16"/>
+<wire x1="48.895" y1="2.8575" x2="48.895" y2="4.93" width="0.4064" layer="16"/>
+<wire x1="48.895" y1="4.93" x2="48.845" y2="4.98" width="0.4064" layer="16"/>
 </signal>
 <signal name="N$3">

Commit message: NS
Connections:
- new net N$49: D2.C, R31.2
- net N$41: no longer D2.C, R31.2
Routing:
- net N$41: track 50.0 -> 20.3 mm
Changed lines of the file:
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@@
 <signal name="N$41">
 <contactref element="D2" pad="A"/>
-<contactref element="D2" pad="C"/>
 <contactref element="CONTROLLER" pad="10"/>
-<contactref element="R31" pad="2"/>
-<wire x1="15.392" y1="26.3525" x2="45.085" y2="26.3525" width="0.4064" layer="1"/>
 <wire x1="69.6595" y1="19.404990625" x2="66.637509375" y2="19.404990625" width="0.4064" layer="1"/>
 <wire x1="66.637509375" y1="19.404990625" x2="65.7225" y2="20.32" width="0.4064" layer="1"/>
@@
 <wire x1="65.7225" y1="25.4" x2="64.77" y2="26.3525" width="0.4064" layer="1"/>
 <wire x1="64.77" y1="26.3525" x2="55.245" y2="26.3525" width="0.4064" layer="1"/>
-<wire x1="45.085" y1="26.3525" x2="55.245" y2="26.3525" width="0" layer="19" extent="1-1"/>
 </signal>
 <signal name="N$43">
@@
 <wire x1="8.89" y1="34.39" x2="9" y2="34.5" width="0.4064" layer="1"/>
 </signal>
+<signal name="N$49">
+<contactref element="R31" pad="2"/>
+<contactref element="D2" pad="C"/>
+<wire x1="15.392" y1="26.3525" x2="45.085" y2="26.3525" width="0" layer="19" extent="1-1"/>
+</signal>
 </signals>

Commit message: ND
Routing:
- net N$49: track 0.00 -> 29.7 mm
Changed lines of the file:
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@@
 <setting verticaltext="up"/>
 </settings>
-<grid distance="0.3175" unitdist="mm" unit="mm" style="lines" multiple="1" display="no" altdistance="0.025" altunitdist="inch" altunit="mm"/>
+<grid distance="0.3175" unitdist="mm" unit="mm" style="lines" multiple="1" display="yes" altdistance="0.025" altunitdist="inch" altunit="mm"/>
 <layers>
 <layer number="1" name="Top" color="4" fill="1" visible="yes" active="yes"/>
@@
 <contactref element="R31" pad="2"/>
 <contactref element="D2" pad="C"/>
-<wire x1="15.392" y1="26.3525" x2="45.085" y2="26.3525" width="0" layer="19" extent="1-1"/>
+<wire x1="15.392" y1="26.3525" x2="45.085" y2="26.3525" width="0.4064" layer="1"/>
 </signal>
 </signals>
