File: PCB/MPPT/MPPT.sch (EAGLE design)
At the start: 2 parts, among them IC1 ACS711KEXLT-15AB-T, IC2 ACS711KEXLT-15AB-T

Commit message: nothing
Parts:
- added U$1: CONN-KF2EDG-10(5.08)E-BAYPLUGGABLECONNECTORS, Stuff_I_Use:CONN-KF2EDG-10(5.08)E-BAYPLUGGABLECONNECTORS
Other:
- moved on the sheet: IC1, IC2
Changed lines of the file:
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@@
 <part name="IC1" library="SamacSys_Parts" deviceset="ACS711KEXLT-15AB-T" device=""/>
 <part name="IC2" library="SamacSys_Parts" deviceset="ACS711KEXLT-15AB-T" device=""/>
+<part name="U$1" library="Stuff_I_Use" deviceset="CONN-KF2EDG-10(5.08)" device="E-BAYPLUGGABLECONNECTORS"/>
 </parts>
 <sheets>
@@
 </plain>
 <instances>
-<instance part="IC1" gate="G$1" x="35.56" y="142.24"/>
-<instance part="IC2" gate="G$1" x="35.56" y="99.06"/>
+<instance part="IC1" gate="G$1" x="104.14" y="157.48" rot="R270"/>
+<instance part="IC2" gate="G$1" x="147.32" y="157.48" rot="R270"/>
+<instance part="U$1" gate="G$1" x="121.92" y="185.42"/>
 </instances>
 <busses>

Commit message: Start of Board Design
Parts:
- added C1, C2, C3, C4: 100nF, resistor:C-USC0603
- added IC3, IC4: ACS711KEXLT-15AB-T, SamacSys_Parts:ACS711KEXLT-15AB-T
- added R1, R3, R5, R7: 100K, resistor:R-US_R0603
- added R2, R4, R6, R8: 20K, resistor:R-US_R0603
Connections:
- new net N$1: C1.2, R1.1, R2.1
- new net N$2: C2.1, IC2.IP-, R4.1, U$1.P$3
- new net N$3: IC2.IP+, R3.1, U$1.P$4
- new net N$4: C2.2, R3.2, R4.2
- new net N$5: C3.2, R5.1, R6.2
- new net N$6: C4.2, R7.2, R8.1
- new net N$7: IC4.IP+, R7.1, U$1.P$10
- new net N$8: C4.1, IC4.IP-, R8.2, U$1.P$9
- new net N$B_1+: IC3.IP+, R5.2, U$1.P$8
- new net N$B_1-: C3.1, IC3.IP-, R6.1, U$1.P$7
- new net N$PV_1+: IC1.IP+, R1.2, U$1.P$2
- new net N$PV_1-: C1.1, IC1.IP-, R2.2, U$1.P$1
- new net VDD: IC1.VCC, IC2.VCC, IC3.VCC, IC4.VCC
- new net VSS: IC1.GND, IC2.GND, IC3.GND, IC4.GND
Other:
- moved on the sheet: IC1, IC2

Commit message: progress
Parts:
- removed IC1, IC2: ACS711KEXLT-15AB-T, SamacSys_Parts:ACS711KEXLT-15AB-T
- added BATT_1_I_SENSE, PV_1_I_SENSE: ACS711KEXLT-15AB-T, SamacSys_Parts:ACS711KEXLT-15AB-T
- added BUCK1_IN+, BUCK1_IN-, BUCK1_OUT+, BUCK1_OUT-, BUCK2_IN+, BUCK2_IN-, BUCK2_OUT+, BUCK2_OUT-: (no value), wirepad:3,81/1,4
Connections:
- removed net N$5 (its old number): C3.2, R5.1, R6.2
- removed net N$B_1+: IC3.IP+, R5.2, U$1.P$8
- removed net N$B_1-: C3.1, IC3.IP-, R6.1, U$1.P$7
- removed net N$PV_1+: IC1.IP+, R1.2, U$1.P$2
- removed net N$PV_1-: C1.1, IC1.IP-, R2.2, U$1.P$1
- new net N$10: C3.2, R5.2, R6.2
- new net N$11: IC4.IP-, R7.2, U$1.P$10
- new net N$12: C4.2, R7.1, R8.2
- new net N$4: BATT_1_I_SENSE.IP+, BUCK1_OUT+.P
- new net N$9: BUCK2_IN+.P, IC3.IP-
- net N$1: now also PV_1_I_SENSE.IP+, U$1.P$1; no longer C1.2, R1.1, R2.1
- net N$2: now also BUCK1_IN+.P, PV_1_I_SENSE.IP-, R1.2; no longer C2.1, IC2.IP-, R4.1, U$1.P$3
- net N$3: now also C1.2, R1.1, R2.2; no longer IC2.IP+, R3.1, U$1.P$4
- net N$6: now also BATT_1_I_SENSE.IP-, R3.1, U$1.P$4; no longer C4.2, R7.2, R8.1
- net N$7: now also BUCK2_OUT+.P; no longer R7.1, U$1.P$10
- net N$8: now also IC3.IP+, R5.1, U$1.P$7; no longer C4.1, IC4.IP-, R8.2, U$1.P$9
- net VDD: now also BATT_1_I_SENSE.VCC, PV_1_I_SENSE.VCC; no longer IC1.VCC, IC2.VCC
- net VSS: now also BATT_1_I_SENSE.!FAULT, BATT_1_I_SENSE.GND, BUCK1_IN-.P, BUCK1_OUT-.P, BUCK2_IN-.P, BUCK2_OUT-.P, C1.1, C2.1, C3.1, C4.1, PV_1_I_SENSE.GND, R2.1, R4.1, R6.1, R8.1, U$1.P$2, U$1.P$3, U$1.P$8, U$1.P$9; no longer IC1.GND, IC2.GND, IC4.GND
Other:
- moved on the sheet: C1, C2, C3, C4, IC3, IC4, R1, R2, R3, R4, R5, R6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

Commit message: sc
Connections:
- removed net N$2: BUCK1_IN+.P, PV_1_I_SENSE.IP-, R1.2
- new net N$13: BUCK1_IN+.P, PV_1_I_SENSE.IP-
- net N$1: now also R1.1
- net N$3: now also R1.2, R2.1; no longer R1.1, R2.2
- net VSS: now also IC4.GND, R2.2; no longer BATT_1_I_SENSE.!FAULT, R2.1
Other:
- moved on the sheet: BUCK1_IN+, BUCK1_IN-, C1, PV_1_I_SENSE, R1, R2

Commit message: BP
Parts:
- added R10, R11, R12, R13, R14, R15, R16, R17, R18, R19, R20, R21, R22, R23, R24, R9: 20K, resistor:R-US_R0603
- added U1: PIC16F18855-X/SS, 16F18855_SSOP:PIC16F18855-X/SS
- added U2, U3: LM324PWR, LM324PWR:LM324PWR
Connections:
- new net N$14: R15.1, R16.2, U2.3IN-
- new net N$15: R10.1, U2.1OUT
- new net N$16: R11.1, R12.2, U2.2IN-
- new net N$17: R12.1, U2.2OUT
- new net N$18: R13.1, R14.2, U2.4IN-
- new net N$19: R10.2, R9.1, U2.1IN-
- new net N$2: PV_1_I_SENSE.VOUT, U2.2IN+
- new net N$20: R13.2, U2.4OUT
- new net N$21: R15.2, U2.3OUT
- new net N$22: BATT_1_I_SENSE.VOUT, U2.4IN+
- new net N$24: R18.1, U3.1OUT
- new net N$25: R20.1, U3.2OUT
- new net N$26: R19.1, R20.2, U3.2IN-
- new net N$27: R21.2, U3.4OUT
- new net N$28: R21.1, R22.2, U3.4IN-
- new net N$29: R23.2, U3.3OUT
- new net N$30: R23.1, R24.2, U3.3IN-
- new net N$31: R17.1, R18.2, U3.1IN-
- new net N$32: IC3.VOUT, U3.2IN+
- new net N$33: IC4.VOUT, U3.4IN+
- net N$10: now also U3.1IN+
- net N$12: now also U3.3IN+
- net N$3: now also U2.1IN+
- net N$5: now also U2.3IN+
- net VDD: now also U1.VDD, U2.VCC, U3.VCC
- net VSS: now also R11.2, R14.1, R16.1, R17.2, R19.2, R22.1, R24.1, R9.2, U1.VSS, U1.VSS_2, U2.GND, U3.GND

Commit message: CO
Parts:
- removed U1: PIC16F18855-X/SS, 16F18855_SSOP:PIC16F18855-X/SS
- added BUCK: TINY_BUCK, Tiny_Buck:TINY_BUCK
- added CONTROLLER: PIC16F18855-X/SS, 16F18855_SSOP:PIC16F18855-X/SS
- added LCD: (no value), con-lsta:FE08-1
- added R25, R26: 1K, resistor:R-US_R0603
- renumbered U2 to BUFFER1, U3 to BUFFER2
Connections:
- new net N$23: CONTROLLER.RA0, LCD.1
- new net N$34: CONTROLLER.RA1, LCD.2
- new net N$35: CONTROLLER.RA2, LCD.3
- new net N$36: CONTROLLER.RA3, LCD.4
- new net N$37: CONTROLLER.RA4, LCD.5
- new net N$38: LCD.7, R25.1, R26.2
- new net N$39: BUCK.IN+
- net VDD: now also BUFFER1.VDD, BUFFER2.VDD, CONTROLLER.VDD, LCD.6, R25.2; no longer BUFFER1.VCC, BUFFER2.VCC, U1.VDD
- net VSS: now also BUFFER1.VSS, BUFFER2.VSS, CONTROLLER.VSS, CONTROLLER.VSS_2, LCD.8, R26.1; no longer BUFFER1.GND, BUFFER2.GND, U1.VSS, U1.VSS_2
Other:
- note added: "These resistors are either/or, not both"

Commit message: gfcr
Parts:
- removed BUCK: TINY_BUCK, Tiny_Buck:TINY_BUCK
- added 3.3V_BUCK: TINY_BUCK, Tiny_Buck:TINY_BUCK
- added C5, C6, C7: 100nF, resistor:C-USC0603
- added PROGRAM: Pin 1, con-lstb:MA08-1
- added SV2: (no value), con-lstb:MA04-1
Connections:
- removed net N$39: BUCK.IN+
- net N$15: now also CONTROLLER.RC7
- net N$17: now also CONTROLLER.RC6
- net N$20: now also CONTROLLER.RC4
- net N$21: now also CONTROLLER.RC5
- net N$24: now also CONTROLLER.RC3
- net N$25: now also CONTROLLER.RC2
- net N$27: now also CONTROLLER.RC0
- net N$29: now also CONTROLLER.RC1
- net N$6: now also 3.3V_BUCK.IN+
- net VDD: now also 3.3V_BUCK.OUT+, C5.2, C6.2, C7.2
- net VSS: now also 3.3V_BUCK.IN-, 3.3V_BUCK.OUT-, C5.1, C6.1, C7.1
Changed lines of the file:
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@@
 <setting verticaltext="up"/>
 </settings>
-<grid distance="0.1" unitdist="mm" unit="mm" style="lines" multiple="1" display="yes" altdistance="0.01" altunitdist="inch" altunit="inch"/>
+<grid distance="0.1" unitdist="inch" unit="mm" style="lines" multiple="1" display="yes" altdistance="0.01" altunitdist="inch" altunit="inch"/>
 <layers>
 <layer number="1" name="Top" color="4" fill="1" visible="no" active="no"/>
@@
 <part name="R26" library="resistor" deviceset="R-US_" device="R0603" value="1K"/>
 <part name="VSS11" library="supply1" deviceset="VSS" device=""/>
-<part name="BUCK" library="Tiny_Buck" deviceset="TINY_BUCK" device=""/>
+<part name="3.3V_BUCK" library="Tiny_Buck" deviceset="TINY_BUCK" device=""/>
+<part name="C5" library="resistor" deviceset="C-US" device="C0603" value="100nF"/>
+<part name="C6" library="resistor" deviceset="C-US" device="C0603" value="100nF"/>
+<part name="C7" library="resistor" deviceset="C-US" device="C0603" value="100nF"/>
+<part name="PROGRAM" library="con-lstb" deviceset="MA08-1" device="" value="Pin 1"/>
+<part name="SV2" library="con-lstb" deviceset="MA04-1" device="" value=" "/>
 </parts>
 <sheets>
 <sheet>
 <plain>
-<frame x1="0" y1="0" x2="266.7" y2="203.2" columns="8" rows="5" layer="91"/>
 <text x="220.98" y="30.48" size="1.778" layer="91">These resistors are either/or, not both</text>
 </plain>
@@
 <instance part="R26" gate="G$1" x="218.44" y="35.56" rot="R270"/>
 <instance part="VSS11" gate="G$1" x="124.46" y="27.94"/>
-<instance part="BUCK" gate="G$1" x="23.4" y="21"/>
+<instance part="3.3V_BUCK" gate="G$1" x="33.02" y="25.4"/>
+<instance part="C5" gate="G$1" x="60.96" y="35.56"/>
+<instance part="C6" gate="G$1" x="71.12" y="35.56"/>
+<instance part="C7" gate="G$1" x="81.28" y="35.56"/>
+<instance part="PROGRAM" gate="1" x="66.04" y="2.54" rot="R90"/>
+<instance part="SV2" gate="1" x="15.24" y="2.54" rot="R90"/>
 </instances>
 <busses>
@@
 <wire x1="109.22" y1="45.72" x2="124.46" y2="45.72" width="0.1524" layer="91"/>
 <wire x1="124.46" y1="45.72" x2="124.46" y2="33.02" width="0.1524" layer="91"/>
+<junction x="88.9" y="38.1"/>
+<wire x1="88.9" y1="38.1" x2="81.28" y2="38.1" width="0.1524" layer="91"/>
+<pinref part="3.3V_BUCK" gate="G$1" pin="OUT-"/>
+<wire x1="81.28" y1="38.1" x2="71.12" y2="38.1" width="0.1524" layer="91"/>
+<wire x1="71.12" y1="38.1" x2="60.96" y2="38.1" width="0.1524" layer="91"/>
+<wire x1="60.96" y1="38.1" x2="60.96" y2="40.64" width="0.1524" layer="91"/>
+<wire x1="60.96" y1="40.64" x2="60.96" y2="45.72" width="0.1524" layer="91"/>
+<wire x1="60.96" y1="45.72" x2="27.94" y2="45.72" width="0.1524" layer="91"/>
+<pinref part="3.3V_BUCK" gate="G$1" pin="IN-"/>
+<wire x1="27.94" y1="45.72" x2="27.94" y2="40.64" width="0.1524" layer="91"/>
+<junction x="60.96" y="40.64"/>
+<pinref part="C5" gate="G$1" pin="1"/>
+<junction x="60.96" y="38.1"/>
+<pinref part="C6" gate="G$1" pin="1"/>
+<junction x="71.12" y="38.1"/>
+<pinref part="C7" gate="G$1" pin="1"/>
+<junction x="81.28" y="38.1"/>
 </segment>
 </net>
@@
 <pinref part="VDD7" gate="G$1" pin="VDD"/>
 <wire x1="88.9" y1="35.56" x2="116.84" y2="35.56" width="0.1524" layer="91"/>
+<pinref part="3.3V_BUCK" gate="G$1" pin="OUT+"/>
+<pinref part="C5" gate="G$1" pin="2"/>
+<wire x1="60.96" y1="27.94" x2="60.96" y2="30.48" width="0.1524" layer="91"/>
+<pinref part="C7" gate="G$1" pin="2"/>
+<wire x1="60.96" y1="30.48" x2="71.12" y2="30.48" width="0.1524" layer="91"/>
+<wire x1="71.12" y1="30.48" x2="81.28" y2="30.48" width="0.1524" layer="91"/>
+<wire x1="81.28" y1="30.48" x2="83.82" y2="30.48" width="0.1524" layer="91"/>
+<wire x1="83.82" y1="30.48" x2="83.82" y2="35.56" width="0.1524" layer="91"/>
+<wire x1="83.82" y1="35.56" x2="88.9" y2="35.56" width="0.1524" layer="91"/>
+<junction x="60.96" y="30.48"/>
+<pinref part="C6" gate="G$1" pin="2"/>
+<junction x="71.12" y="30.48"/>
+<junction x="81.28" y="30.48"/>
+<junction x="88.9" y="35.56"/>
 </segment>
 <segment>
@@
 <wire x1="93.98" y1="142.24" x2="93.98" y2="129.54" width="0.1524" layer="91"/>
 <wire x1="93.98" y1="129.54" x2="5.08" y2="129.54" width="0.1524" layer="91"/>
-<wire x1="5.08" y1="129.54" x2="5.08" y2="22.86" width="0.1524" layer="91"/>
-<wire x1="5.08" y1="22.86" x2="15.3" y2="22.8" width="0.1524" layer="91"/>
+<wire x1="5.08" y1="129.54" x2="5.08" y2="27.94" width="0.1524" layer="91"/>
+<pinref part="3.3V_BUCK" gate="G$1" pin="IN+"/>
+<wire x1="5.08" y1="27.94" x2="27.94" y2="27.94" width="0.1524" layer="91"/>
 </segment>
 </net>
@@
 <pinref part="BUFFER1" gate="A" pin="1OUT"/>
 <pinref part="R10" gate="G$1" pin="1"/>
+<junction x="35.56" y="91.44"/>
+<wire x1="35.56" y1="91.44" x2="35.56" y2="99.06" width="0.1524" layer="91"/>
+<wire x1="35.56" y1="99.06" x2="55.88" y2="99.06" width="0.1524" layer="91"/>
+<wire x1="55.88" y1="99.06" x2="55.88" y2="48.26" width="0.1524" layer="91"/>
+<wire x1="55.88" y1="48.26" x2="68.58" y2="48.26" width="0.1524" layer="91"/>
+<wire x1="68.58" y1="48.26" x2="68.58" y2="40.64" width="0.1524" layer="91"/>
+<pinref part="CONTROLLER" gate="A" pin="RC7"/>
+<wire x1="68.58" y1="40.64" x2="88.9" y2="40.64" width="0.1524" layer="91"/>
 </segment>
 </net>
@@
 <pinref part="BUFFER1" gate="A" pin="2OUT"/>
 <pinref part="R12" gate="G$1" pin="1"/>
+<junction x="35.56" y="76.2"/>
+<wire x1="35.56" y1="76.2" x2="35.56" y2="50.8" width="0.1524" layer="91"/>
+<wire x1="35.56" y1="50.8" x2="71.12" y2="50.8" width="0.1524" layer="91"/>
+<wire x1="71.12" y1="50.8" x2="71.12" y2="43.18" width="0.1524" layer="91"/>
+<pinref part="CONTROLLER" gate="A" pin="RC6"/>
+<wire x1="71.12" y1="43.18" x2="88.9" y2="43.18" width="0.1524" layer="91"/>
 </segment>
 </net>
@@
 <pinref part="BUFFER1" gate="A" pin="4OUT"/>
 <pinref part="R13" gate="G$1" pin="2"/>
+<junction x="91.44" y="91.44"/>
+<wire x1="91.44" y1="91.44" x2="91.44" y2="96.52" width="0.1524" layer="91"/>
+<wire x1="91.44" y1="96.52" x2="114.3" y2="96.52" width="0.1524" layer="91"/>
+<wire x1="114.3" y1="96.52" x2="114.3" y2="63.5" width="0.1524" layer="91"/>
+<wire x1="114.3" y1="63.5" x2="76.2" y2="63.5" width="0.1524" layer="91"/>
+<wire x1="76.2" y1="63.5" x2="76.2" y2="48.26" width="0.1524" layer="91"/>
+<pinref part="CONTROLLER" gate="A" pin="RC4"/>
+<wire x1="76.2" y1="48.26" x2="88.9" y2="48.26" width="0.1524" layer="91"/>
 </segment>
 </net>
@@
 <pinref part="BUFFER1" gate="A" pin="3OUT"/>
 <pinref part="R15" gate="G$1" pin="2"/>
+<junction x="91.44" y="76.2"/>
+<wire x1="91.44" y1="76.2" x2="91.44" y2="66.04" width="0.1524" layer="91"/>
+<wire x1="91.44" y1="66.04" x2="73.66" y2="66.04" width="0.1524" layer="91"/>
+<wire x1="73.66" y1="66.04" x2="73.66" y2="45.72" width="0.1524" layer="91"/>
+<pinref part="CONTROLLER" gate="A" pin="RC5"/>
+<wire x1="73.66" y1="45.72" x2="88.9" y2="45.72" width="0.1524" layer="91"/>
 </segment>
 </net>
@@
 <pinref part="BUFFER2" gate="A" pin="1OUT"/>
 <pinref part="R18" gate="G$1" pin="1"/>
+<junction x="175.26" y="91.44"/>
+<wire x1="175.26" y1="91.44" x2="175.26" y2="99.06" width="0.1524" layer="91"/>
+<wire x1="175.26" y1="99.06" x2="147.32" y2="99.06" width="0.1524" layer="91"/>
+<wire x1="147.32" y1="99.06" x2="147.32" y2="48.26" width="0.1524" layer="91"/>
+<pinref part="CONTROLLER" gate="A" pin="RC3"/>
+<wire x1="147.32" y1="48.26" x2="144.78" y2="48.26" width="0.1524" layer="91"/>
 </segment>
 </net>
@@
 <pinref part="BUFFER2" gate="A" pin="2OUT"/>
 <pinref part="R20" gate="G$1" pin="1"/>
+<junction x="175.26" y="76.2"/>
+<wire x1="175.26" y1="76.2" x2="175.26" y2="60.96" width="0.1524" layer="91"/>
+<wire x1="175.26" y1="60.96" x2="149.86" y2="60.96" width="0.1524" layer="91"/>
+<wire x1="149.86" y1="60.96" x2="149.86" y2="45.72" width="0.1524" layer="91"/>
+<pinref part="CONTROLLER" gate="A" pin="RC2"/>
+<wire x1="149.86" y1="45.72" x2="144.78" y2="45.72" width="0.1524" layer="91"/>
 </segment>
 </net>
@@
 <pinref part="BUFFER2" gate="A" pin="4OUT"/>
 <pinref part="R21" gate="G$1" pin="2"/>
+<junction x="231.14" y="91.44"/>
+<wire x1="231.14" y1="91.44" x2="231.14" y2="99.06" width="0.1524" layer="91"/>
+<wire x1="231.14" y1="99.06" x2="259.08" y2="99.06" width="0.1524" layer="91"/>
+<wire x1="259.08" y1="99.06" x2="259.08" y2="55.88" width="0.1524" layer="91"/>
+<wire x1="259.08" y1="55.88" x2="154.94" y2="55.88" width="0.1524" layer="91"/>
+<wire x1="154.94" y1="55.88" x2="154.94" y2="40.64" width="0.1524" layer="91"/>
+<pinref part="CONTROLLER" gate="A" pin="RC0"/>
+<wire x1="154.94" y1="40.64" x2="144.78" y2="40.64" width="0.1524" layer="91"/>
 </segment>
 </net>
@@
 <pinref part="BUFFER2" gate="A" pin="3OUT"/>
 <pinref part="R23" gate="G$1" pin="2"/>
+<junction x="231.14" y="76.2"/>
+<wire x1="231.14" y1="76.2" x2="231.14" y2="58.42" width="0.1524" layer="91"/>
+<wire x1="231.14" y1="58.42" x2="152.4" y2="58.42" width="0.1524" layer="91"/>
+<wire x1="152.4" y1="58.42" x2="152.4" y2="43.18" width="0.1524" layer="91"/>
+<pinref part="CONTROLLER" gate="A" pin="RC1"/>
+<wire x1="152.4" y1="43.18" x2="144.78" y2="43.18" width="0.1524" layer="91"/>
 </segment>
 </net>
@@
 </segment>
 </net>
-<net name="N$39" class="0">
-<segment>
-<pinref part="BUCK" gate="G$1" pin="IN+"/>
-<wire x1="18.2" y1="22.9" x2="15.3" y2="22.8" width="0.1524" layer="91"/>
-</segment>
-</net>
