File: PCB/MPPT/MPPT.sch (EAGLE design)
At the start: 53 parts, among them IC3 ACS711KEXLT-15AB-T, IC4 ACS711KEXLT-15AB-T

Commit message: cly
Changed lines of the file:
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@@
 <?xml version="1.0" encoding="utf-8"?>
 <!DOCTYPE eagle SYSTEM "eagle.dtd">
-<eagle version="7.2.0">
+<eagle version="9.0.1">
 <drawing>
 <settings>
 <setting alwaysvectorfont="no"/>
+<setting keepoldvectorfont="yes"/>
 <setting verticaltext="up"/>
 </settings>
@@
 <part name="R7" library="resistor" deviceset="R-US_" device="R0603" value="100K"/>
 <part name="R8" library="resistor" deviceset="R-US_" device="R0603" value="20K"/>
-<part name="C1" library="resistor" deviceset="C-US" device="C0603" value="100nF"/>
 <part name="C2" library="resistor" deviceset="C-US" device="C0603" value="100nF"/>
 <part name="C3" library="resistor" deviceset="C-US" device="C0603" value="100nF"/>
@@
 <part name="PROGRAM" library="con-lstb" deviceset="MA08-1" device="" value="Pin 1"/>
 <part name="SV2" library="con-lstb" deviceset="MA04-1" device="" value=" "/>
+<part name="C1" library="resistor" deviceset="C-US" device="C0603" value="100nF"/>
 </parts>
 <sheets>
@@
 <instance part="R7" gate="G$1" x="157.48" y="177.8"/>
 <instance part="R8" gate="G$1" x="147.32" y="177.8"/>
-<instance part="C1" gate="G$1" x="78.74" y="165.1" rot="R90"/>
 <instance part="C2" gate="G$1" x="104.14" y="177.8"/>
 <instance part="C3" gate="G$1" x="124.46" y="175.26"/>
@@
 <instance part="PROGRAM" gate="1" x="66.04" y="2.54" rot="R90"/>
 <instance part="SV2" gate="1" x="15.24" y="2.54" rot="R90"/>
+<instance part="C1" gate="G$1" x="78.74" y="165.1" rot="R90"/>
 </instances>
 <busses>
@@
 <segment>
 <pinref part="R2" gate="G$1" pin="2"/>
-<pinref part="C1" gate="G$1" pin="1"/>
 <wire x1="76.2" y1="177.8" x2="76.2" y2="165.1" width="0.1524" layer="91"/>
-<junction x="76.2" y="165.1"/>
 <pinref part="VSS5" gate="G$1" pin="VSS"/>
+<pinref part="PV_1_I_SENSE" gate="G$1" pin="GND"/>
 <wire x1="76.2" y1="165.1" x2="76.2" y2="157.48" width="0.1524" layer="91"/>
-<pinref part="PV_1_I_SENSE" gate="G$1" pin="GND"/>
 <wire x1="76.2" y1="157.48" x2="78.74" y2="157.48" width="0.1524" layer="91"/>
 <wire x1="78.74" y1="157.48" x2="78.74" y2="144.78" width="0.1524" layer="91"/>
 <junction x="76.2" y="157.48"/>
+<pinref part="C1" gate="G$1" pin="1"/>
+<junction x="76.2" y="165.1"/>
 </segment>
 <segment>
@@
 <net name="N$3" class="0">
 <segment>
-<pinref part="C1" gate="G$1" pin="2"/>
-<pinref part="C1" gate="G$1" pin="2"/>
 <wire x1="83.82" y1="165.1" x2="86.36" y2="165.1" width="0.1524" layer="91"/>
 <pinref part="R1" gate="G$1" pin="2"/>
@@
 <wire x1="86.36" y1="165.1" x2="86.36" y2="177.8" width="0.1524" layer="91"/>
 <junction x="86.36" y="177.8"/>
-<junction x="83.82" y="165.1"/>
 <wire x1="86.36" y1="177.8" x2="86.36" y2="187.96" width="0.1524" layer="91"/>
 <wire x1="86.36" y1="187.96" x2="10.16" y2="187.96" width="0.1524" layer="91"/>
@@
 <pinref part="BUFFER1" gate="A" pin="1IN+"/>
 <wire x1="10.16" y1="86.36" x2="35.56" y2="86.36" width="0.1524" layer="91"/>
+<pinref part="C1" gate="G$1" pin="2"/>
 </segment>
 </net>

Commit message: qc
Parts:
- removed PROGRAM: Pin 1, con-lstb:MA08-1
- removed SV2: (no value), con-lstb:MA04-1
- added R27: 10K, rcl:R-US_R1206
- added R28: 10K, resistor:R-US_R0603
- added X1, X2: 22-23-2021, con-molex:22-23-2021
- added X3: 22-23-2041, con-molex:22-23-2041
Connections:
- new net N$39: CONTROLLER.RB1, R28.2, X3-2.S
- new net N$42: CONTROLLER.RB0, R27.2, X3-4.S
- net VDD: now also R27.1, R28.1
- net VSS: now also X3-1.S, X3-3.S
Other:
- moved on the sheet: C6, C7
Changed lines of the file:
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@@
 <?xml version="1.0" encoding="utf-8"?>
 <!DOCTYPE eagle SYSTEM "eagle.dtd">
-<eagle version="9.0.1">
+<eagle version="7.2.0">
 <drawing>
 <settings>
 <setting alwaysvectorfont="no"/>
-<setting keepoldvectorfont="yes"/>
 <setting verticaltext="up"/>
 </settings>
-<grid distance="0.1" unitdist="inch" unit="inch" style="lines" multiple="1" display="no" altdistance="0.01" altunitdist="inch" altunit="inch"/>
+<grid distance="0.1" unitdist="inch" unit="mm" style="lines" multiple="1" display="yes" altdistance="0.01" altunitdist="inch" altunit="inch"/>
 <layers>
 <layer number="1" name="Top" color="4" fill="1" visible="no" active="no"/>
@@
 <part name="C6" library="resistor" deviceset="C-US" device="C0603" value="100nF"/>
 <part name="C7" library="resistor" deviceset="C-US" device="C0603" value="100nF"/>
-<part name="PROGRAM" library="con-lstb" deviceset="MA08-1" device="" value="Pin 1"/>
-<part name="SV2" library="con-lstb" deviceset="MA04-1" device="" value=" "/>
 <part name="C1" library="resistor" deviceset="C-US" device="C0603" value="100nF"/>
+<part name="X1" library="con-molex" deviceset="22-23-2021" device=""/>
+<part name="X2" library="con-molex" deviceset="22-23-2021" device=""/>
+<part name="X3" library="con-molex" deviceset="22-23-2041" device=""/>
+<part name="R28" library="resistor" deviceset="R-US_" device="R0603" value="10K"/>
+<part name="VDD9" library="supply1" deviceset="VDD" device=""/>
+<part name="VSS12" library="supply1" deviceset="VSS" device=""/>
+<part name="R27" library="rcl" deviceset="R-US_" device="R1206" value="10K"/>
 </parts>
 <sheets>
@@
 <instance part="3.3V_BUCK" gate="G$1" x="33.02" y="25.4"/>
 <instance part="C5" gate="G$1" x="60.96" y="35.56"/>
-<instance part="C6" gate="G$1" x="71.12" y="35.56"/>
-<instance part="C7" gate="G$1" x="81.28" y="35.56"/>
-<instance part="PROGRAM" gate="1" x="66.04" y="2.54" rot="R90"/>
-<instance part="SV2" gate="1" x="15.24" y="2.54" rot="R90"/>
+<instance part="C6" gate="G$1" x="68.58" y="35.56"/>
+<instance part="C7" gate="G$1" x="78.74" y="35.56"/>
 <instance part="C1" gate="G$1" x="78.74" y="165.1" rot="R90"/>
+<instance part="X1" gate="-1" x="193.04" y="40.64"/>
+<instance part="X1" gate="-2" x="193.04" y="38.1"/>
+<instance part="X2" gate="-1" x="193.04" y="17.78"/>
+<instance part="X2" gate="-2" x="193.04" y="15.24"/>
+<instance part="X3" gate="-1" x="-2.54" y="182.88" rot="R90"/>
+<instance part="X3" gate="-2" x="0" y="182.88" rot="R90"/>
+<instance part="X3" gate="-3" x="2.54" y="182.88" rot="R90"/>
+<instance part="X3" gate="-4" x="5.08" y="182.88" rot="R90"/>
+<instance part="R28" gate="G$1" x="0" y="175.26" rot="R90"/>
+<instance part="VDD9" gate="G$1" x="7.62" y="149.86"/>
+<instance part="VSS12" gate="G$1" x="-2.54" y="147.32"/>
+<instance part="R27" gate="G$1" x="5.08" y="160.02" rot="R90"/>
 </instances>
 <busses>
@@
 <wire x1="124.46" y1="45.72" x2="124.46" y2="33.02" width="0.1524" layer="91"/>
 <junction x="88.9" y="38.1"/>
-<wire x1="88.9" y1="38.1" x2="81.28" y2="38.1" width="0.1524" layer="91"/>
+<wire x1="88.9" y1="38.1" x2="78.74" y2="38.1" width="0.1524" layer="91"/>
 <pinref part="3.3V_BUCK" gate="G$1" pin="OUT-"/>
-<wire x1="81.28" y1="38.1" x2="71.12" y2="38.1" width="0.1524" layer="91"/>
-<wire x1="71.12" y1="38.1" x2="60.96" y2="38.1" width="0.1524" layer="91"/>
+<wire x1="78.74" y1="38.1" x2="68.58" y2="38.1" width="0.1524" layer="91"/>
+<wire x1="68.58" y1="38.1" x2="60.96" y2="38.1" width="0.1524" layer="91"/>
 <wire x1="60.96" y1="38.1" x2="60.96" y2="40.64" width="0.1524" layer="91"/>
 <wire x1="60.96" y1="40.64" x2="60.96" y2="45.72" width="0.1524" layer="91"/>
@@
 <junction x="60.96" y="38.1"/>
 <pinref part="C6" gate="G$1" pin="1"/>
-<junction x="71.12" y="38.1"/>
+<junction x="68.58" y="38.1"/>
 <pinref part="C7" gate="G$1" pin="1"/>
-<junction x="81.28" y="38.1"/>
+<junction x="78.74" y="38.1"/>
+</segment>
+<segment>
+<pinref part="X3" gate="-1" pin="S"/>
+<pinref part="VSS12" gate="G$1" pin="VSS"/>
+<wire x1="-2.54" y1="180.34" x2="-2.54" y2="167.64" width="0.1524" layer="91"/>
+<junction x="-2.54" y="167.64"/>
+<wire x1="-2.54" y1="167.64" x2="-2.54" y2="149.86" width="0.1524" layer="91"/>
+<pinref part="X3" gate="-3" pin="S"/>
+<wire x1="2.54" y1="180.34" x2="2.54" y2="167.64" width="0.1524" layer="91"/>
+<wire x1="2.54" y1="167.64" x2="-2.54" y2="167.64" width="0.1524" layer="91"/>
 </segment>
 </net>
@@
 <wire x1="60.96" y1="27.94" x2="60.96" y2="30.48" width="0.1524" layer="91"/>
 <pinref part="C7" gate="G$1" pin="2"/>
-<wire x1="60.96" y1="30.48" x2="71.12" y2="30.48" width="0.1524" layer="91"/>
-<wire x1="71.12" y1="30.48" x2="81.28" y2="30.48" width="0.1524" layer="91"/>
-<wire x1="81.28" y1="30.48" x2="83.82" y2="30.48" width="0.1524" layer="91"/>
-<wire x1="83.82" y1="30.48" x2="83.82" y2="35.56" width="0.1524" layer="91"/>
-<wire x1="83.82" y1="35.56" x2="88.9" y2="35.56" width="0.1524" layer="91"/>
+<wire x1="60.96" y1="30.48" x2="68.58" y2="30.48" width="0.1524" layer="91"/>
+<wire x1="68.58" y1="30.48" x2="78.74" y2="30.48" width="0.1524" layer="91"/>
+<wire x1="78.74" y1="30.48" x2="86.36" y2="35.56" width="0.1524" layer="91"/>
+<wire x1="86.36" y1="35.56" x2="88.9" y2="35.56" width="0.1524" layer="91"/>
 <junction x="60.96" y="30.48"/>
 <pinref part="C6" gate="G$1" pin="2"/>
-<junction x="71.12" y="30.48"/>
-<junction x="81.28" y="30.48"/>
+<junction x="68.58" y="30.48"/>
+<junction x="78.74" y="30.48"/>
 <junction x="88.9" y="35.56"/>
 </segment>
@@
 <wire x1="187.96" y1="20.32" x2="218.44" y2="20.32" width="0.1524" layer="91"/>
 <junction x="182.88" y="30.48"/>
+</segment>
+<segment>
+<pinref part="VDD9" gate="G$1" pin="VDD"/>
+<wire x1="7.62" y1="142.24" x2="7.62" y2="147.32" width="0.1524" layer="91"/>
+<wire x1="5.08" y1="142.24" x2="7.62" y2="142.24" width="0.1524" layer="91"/>
+<pinref part="R27" gate="G$1" pin="1"/>
+<wire x1="5.08" y1="142.24" x2="5.08" y2="154.94" width="0.1524" layer="91"/>
+<junction x="5.08" y="154.94"/>
+<wire x1="5.08" y1="154.94" x2="0" y2="154.94" width="0.1524" layer="91"/>
+<pinref part="R28" gate="G$1" pin="1"/>
+<wire x1="0" y1="154.94" x2="0" y2="170.18" width="0.1524" layer="91"/>
 </segment>
 </net>
@@
 </segment>
 </net>
+<net name="N$39" class="0">
+<segment>
+<wire x1="-5.08" y1="177.8" x2="-5.08" y2="20.32" width="0.1524" layer="91"/>
+<wire x1="-5.08" y1="20.32" x2="73.66" y2="20.32" width="0.1524" layer="91"/>
+<wire x1="73.66" y1="20.32" x2="88.9" y2="30.48" width="0.1524" layer="91"/>
+<pinref part="CONTROLLER" gate="A" pin="RB1"/>
+<pinref part="X3" gate="-2" pin="S"/>
+<pinref part="R28" gate="G$1" pin="2"/>
+<junction x="0" y="180.34"/>
+<wire x1="-5.08" y1="177.8" x2="0" y2="180.34" width="0.1524" layer="91"/>
+</segment>
+</net>
+<net name="N$42" class="0">
+<segment>
+<pinref part="R27" gate="G$1" pin="2"/>
+<pinref part="X3" gate="-4" pin="S"/>
+<wire x1="5.08" y1="165.1" x2="5.08" y2="180.34" width="0.1524" layer="91"/>
+<junction x="5.08" y="165.1"/>
+<wire x1="2.54" y1="165.1" x2="2.54" y2="22.86" width="0.1524" layer="91"/>
+<wire x1="2.54" y1="22.86" x2="71.12" y2="22.86" width="0.1524" layer="91"/>
+<wire x1="71.12" y1="22.86" x2="86.36" y2="33.02" width="0.1524" layer="91"/>
+<pinref part="CONTROLLER" gate="A" pin="RB0"/>
+<wire x1="86.36" y1="33.02" x2="88.9" y2="33.02" width="0.1524" layer="91"/>
+<wire x1="5.08" y1="165.1" x2="2.54" y2="165.1" width="0.1524" layer="91"/>
+</segment>
+</net>

Commit message: cy
Parts:
- added PROGRAMMER: (no value), con-lstb:MA06-1
- added R29: 10K, resistor:R-US_R0603
- renumbered LCD to __LCD
Connections:
- new net N$40: CONTROLLER.VPP/*MCLR/RS3, PROGRAMMER.1, R29.1
- new net N$44: CONTROLLER.RB7, PROGRAMMER.4
- new net N$45: CONTROLLER.RB6, PROGRAMMER.5
- net VDD: now also PROGRAMMER.2, R29.2
- net VSS: now also PROGRAMMER.3
Changed lines of the file:
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@@
 <setting verticaltext="up"/>
 </settings>
-<grid distance="0.1" unitdist="inch" unit="mm" style="lines" multiple="1" display="yes" altdistance="0.01" altunitdist="inch" altunit="inch"/>
+<grid distance="0.1" unitdist="inch" unit="inch" style="lines" multiple="1" display="no" altdistance="0.01" altunitdist="inch" altunit="inch"/>
 <layers>
 <layer number="1" name="Top" color="4" fill="1" visible="no" active="no"/>
@@
 <part name="VSS10" library="supply1" deviceset="VSS" device=""/>
 <part name="VDD7" library="supply1" deviceset="VDD" device=""/>
-<part name="LCD" library="con-lsta" deviceset="FE08-1" device="" value=" "/>
+<part name="__LCD" library="con-lsta" deviceset="FE08-1" device="" value=" "/>
 <part name="VDD8" library="supply1" deviceset="VDD" device=""/>
 <part name="R25" library="resistor" deviceset="R-US_" device="R0603" value="1K"/>
@@
 <part name="VSS12" library="supply1" deviceset="VSS" device=""/>
 <part name="R27" library="rcl" deviceset="R-US_" device="R1206" value="10K"/>
+<part name="PROGRAMMER" library="con-lstb" deviceset="MA06-1" device="" value=" "/>
+<part name="R29" library="resistor" deviceset="R-US_" device="R0603" value="10K"/>
 </parts>
 <sheets>
@@
 <instance part="VSS10" gate="G$1" x="203.2" y="33.02"/>
 <instance part="VDD7" gate="G$1" x="116.84" y="38.1"/>
-<instance part="LCD" gate="G$1" x="175.26" y="25.4"/>
+<instance part="__LCD" gate="G$1" x="175.26" y="25.4"/>
 <instance part="VDD8" gate="G$1" x="165.1" y="33.02"/>
 <instance part="R25" gate="G$1" x="218.44" y="25.4" rot="R270"/>
@@
 <instance part="VSS12" gate="G$1" x="-2.54" y="147.32"/>
 <instance part="R27" gate="G$1" x="5.08" y="160.02" rot="R90"/>
+<instance part="PROGRAMMER" gate="1" x="66.04" y="7.62"/>
+<instance part="R29" gate="G$1" x="88.9" y="5.08" rot="R90"/>
 </instances>
 <busses>
@@
 </segment>
 <segment>
-<pinref part="LCD" gate="G$1" pin="8"/>
+<pinref part="__LCD" gate="G$1" pin="8"/>
 <pinref part="VSS10" gate="G$1" pin="VSS"/>
 <wire x1="182.88" y1="35.56" x2="203.2" y2="35.56" width="0.1524" layer="91"/>
@@
 <pinref part="C7" gate="G$1" pin="1"/>
 <junction x="78.74" y="38.1"/>
+<pinref part="PROGRAMMER" gate="1" pin="3"/>
+<wire x1="73.66" y1="5.08" x2="81.28" y2="5.08" width="0.1524" layer="91"/>
+<wire x1="81.28" y1="5.08" x2="81.28" y2="12.7" width="0.1524" layer="91"/>
+<wire x1="81.28" y1="12.7" x2="109.22" y2="12.7" width="0.1524" layer="91"/>
+<wire x1="109.22" y1="12.7" x2="109.22" y2="33.02" width="0.1524" layer="91"/>
+<wire x1="109.22" y1="33.02" x2="124.46" y2="33.02" width="0.1524" layer="91"/>
 </segment>
 <segment>
@@
 <junction x="78.74" y="30.48"/>
 <junction x="88.9" y="35.56"/>
+<pinref part="PROGRAMMER" gate="1" pin="2"/>
+<wire x1="73.66" y1="2.54" x2="83.82" y2="2.54" width="0.1524" layer="91"/>
+<wire x1="83.82" y1="2.54" x2="83.82" y2="10.16" width="0.1524" layer="91"/>
+<pinref part="R29" gate="G$1" pin="2"/>
+<wire x1="83.82" y1="10.16" x2="88.9" y2="10.16" width="0.1524" layer="91"/>
+<wire x1="88.9" y1="10.16" x2="93.98" y2="10.16" width="0.1524" layer="91"/>
+<wire x1="93.98" y1="10.16" x2="93.98" y2="2.54" width="0.1524" layer="91"/>
+<wire x1="93.98" y1="2.54" x2="116.84" y2="2.54" width="0.1524" layer="91"/>
+<wire x1="116.84" y1="2.54" x2="116.84" y2="35.56" width="0.1524" layer="91"/>
+<junction x="88.9" y="10.16"/>
+<junction x="116.84" y="35.56"/>
 </segment>
 <segment>
 <pinref part="VDD8" gate="G$1" pin="VDD"/>
-<pinref part="LCD" gate="G$1" pin="6"/>
+<pinref part="__LCD" gate="G$1" pin="6"/>
 <wire x1="165.1" y1="30.48" x2="182.88" y2="30.48" width="0.1524" layer="91"/>
 <wire x1="182.88" y1="30.48" x2="187.96" y2="30.48" width="0.1524" layer="91"/>
@@
 <segment>
 <pinref part="CONTROLLER" gate="A" pin="RA0"/>
-<pinref part="LCD" gate="G$1" pin="1"/>
+<pinref part="__LCD" gate="G$1" pin="1"/>
 <wire x1="144.78" y1="17.78" x2="182.88" y2="17.78" width="0.1524" layer="91"/>
 </segment>
@@
 <segment>
 <pinref part="CONTROLLER" gate="A" pin="RA1"/>
-<pinref part="LCD" gate="G$1" pin="2"/>
+<pinref part="__LCD" gate="G$1" pin="2"/>
 <wire x1="144.78" y1="20.32" x2="182.88" y2="20.32" width="0.1524" layer="91"/>
 </segment>
@@
 <segment>
 <pinref part="CONTROLLER" gate="A" pin="RA2"/>
-<pinref part="LCD" gate="G$1" pin="3"/>
+<pinref part="__LCD" gate="G$1" pin="3"/>
 <wire x1="144.78" y1="22.86" x2="182.88" y2="22.86" width="0.1524" layer="91"/>
 </segment>
@@
 <segment>
 <pinref part="CONTROLLER" gate="A" pin="RA3"/>
-<pinref part="LCD" gate="G$1" pin="4"/>
+<pinref part="__LCD" gate="G$1" pin="4"/>
 <wire x1="144.78" y1="25.4" x2="182.88" y2="25.4" width="0.1524" layer="91"/>
 </segment>
@@
 <segment>
 <pinref part="CONTROLLER" gate="A" pin="RA4"/>
-<pinref part="LCD" gate="G$1" pin="5"/>
+<pinref part="__LCD" gate="G$1" pin="5"/>
 <wire x1="144.78" y1="27.94" x2="182.88" y2="27.94" width="0.1524" layer="91"/>
 </segment>
@@
 <pinref part="R25" gate="G$1" pin="1"/>
 <pinref part="R26" gate="G$1" pin="2"/>
-<pinref part="LCD" gate="G$1" pin="7"/>
+<pinref part="__LCD" gate="G$1" pin="7"/>
 <wire x1="182.88" y1="33.02" x2="190.5" y2="33.02" width="0.1524" layer="91"/>
 <wire x1="190.5" y1="33.02" x2="190.5" y2="30.48" width="0.1524" layer="91"/>
@@
 </segment>
 </net>
+<net name="N$40" class="0">
+<segment>
+<pinref part="PROGRAMMER" gate="1" pin="1"/>
+<pinref part="CONTROLLER" gate="A" pin="VPP/*MCLR/RS3"/>
+<wire x1="73.66" y1="0" x2="88.9" y2="0" width="0.1524" layer="91"/>
+<wire x1="88.9" y1="0" x2="144.78" y2="0" width="0.1524" layer="91"/>
+<wire x1="144.78" y1="0" x2="144.78" y2="15.24" width="0.1524" layer="91"/>
+<pinref part="R29" gate="G$1" pin="1"/>
+<junction x="88.9" y="0"/>
+</segment>
+</net>
+<net name="N$44" class="0">
+<segment>
+<pinref part="PROGRAMMER" gate="1" pin="4"/>
+<wire x1="73.66" y1="7.62" x2="78.74" y2="7.62" width="0.1524" layer="91"/>
+<wire x1="78.74" y1="7.62" x2="78.74" y2="15.24" width="0.1524" layer="91"/>
+<pinref part="CONTROLLER" gate="A" pin="RB7"/>
+<wire x1="78.74" y1="15.24" x2="88.9" y2="15.24" width="0.1524" layer="91"/>
+</segment>
+</net>
+<net name="N$45" class="0">
+<segment>
+<pinref part="PROGRAMMER" gate="1" pin="5"/>
+<wire x1="73.66" y1="10.16" x2="76.2" y2="10.16" width="0.1524" layer="91"/>
+<wire x1="76.2" y1="10.16" x2="76.2" y2="17.78" width="0.1524" layer="91"/>
+<pinref part="CONTROLLER" gate="A" pin="RB6"/>
+<wire x1="76.2" y1="17.78" x2="88.9" y2="17.78" width="0.1524" layer="91"/>
+</segment>
+</net>

Commit message: NFpRW
Parts:
- added D1, D2: 1N4004, diode:1N4004
- added PWM_1, PWM_2: WIREPAD2,54/1,1, wirepad:WIREPAD2,54/1,1
- added R30: 470R, resistor:R-US_R0603
- added R31: 470R, resistor:R-US_R1206
Connections:
- new net N$41: CONTROLLER.RA6, D2.A, D2.C, R31.2
- new net N$43: CONTROLLER.RA7, D1.A
- new net N$46: PWM_2.P, R30.1
- new net N$47: D1.C, R30.2
- new net N$48: PWM_1.P, R31.1
Changed lines of the file:
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@@
 <part name="PROGRAMMER" library="con-lstb" deviceset="MA06-1" device="" value=" "/>
 <part name="R29" library="resistor" deviceset="R-US_" device="R0603" value="10K"/>
+<part name="PWM_1" library="wirepad" deviceset="WIREPAD" device="2,54/1,1"/>
+<part name="PWM_2" library="wirepad" deviceset="WIREPAD" device="2,54/1,1"/>
+<part name="D1" library="diode" deviceset="1N4004" device=""/>
+<part name="D2" library="diode" deviceset="1N4004" device=""/>
+<part name="R30" library="resistor" deviceset="R-US_" device="R0603" value="470R"/>
+<part name="R31" library="resistor" deviceset="R-US_" device="R1206" value="470R"/>
 </parts>
 <sheets>
@@
 <instance part="PROGRAMMER" gate="1" x="66.04" y="7.62"/>
 <instance part="R29" gate="G$1" x="88.9" y="5.08" rot="R90"/>
+<instance part="PWM_1" gate="G$1" x="205.74" y="50.8" rot="R180"/>
+<instance part="PWM_2" gate="G$1" x="259.08" y="48.26" rot="R180"/>
+<instance part="D1" gate="1" x="213.36" y="48.26"/>
+<instance part="D2" gate="1" x="160.02" y="50.8"/>
+<instance part="R30" gate="G$1" x="228.6" y="48.26" rot="R180"/>
+<instance part="R31" gate="G$1" x="177.8" y="50.8" rot="R180"/>
 </instances>
 <busses>
@@
 </segment>
 </net>
+<net name="N$41" class="0">
+<segment>
+<wire x1="157.48" y1="50.8" x2="162.56" y2="50.8" width="0.1524" layer="91"/>
+<pinref part="D2" gate="1" pin="A"/>
+<pinref part="D2" gate="1" pin="C"/>
+<pinref part="CONTROLLER" gate="A" pin="RA6"/>
+<wire x1="144.78" y1="38.1" x2="157.48" y2="38.1" width="0.1524" layer="91"/>
+<wire x1="157.48" y1="38.1" x2="157.48" y2="50.8" width="0.1524" layer="91"/>
+<pinref part="R31" gate="G$1" pin="2"/>
+<wire x1="162.56" y1="50.8" x2="172.72" y2="50.8" width="0.1524" layer="91"/>
+</segment>
+</net>
+<net name="N$43" class="0">
+<segment>
+<pinref part="CONTROLLER" gate="A" pin="RA7"/>
+<wire x1="144.78" y1="35.56" x2="160.02" y2="35.56" width="0.1524" layer="91"/>
+<wire x1="160.02" y1="35.56" x2="160.02" y2="48.26" width="0.1524" layer="91"/>
+<wire x1="160.02" y1="48.26" x2="210.82" y2="48.26" width="0.1524" layer="91"/>
+<pinref part="D1" gate="1" pin="A"/>
+</segment>
+</net>
+<net name="N$46" class="0">
+<segment>
+<pinref part="PWM_2" gate="G$1" pin="P"/>
+<pinref part="R30" gate="G$1" pin="1"/>
+<wire x1="233.68" y1="48.26" x2="256.54" y2="48.26" width="0.1524" layer="91"/>
+</segment>
+</net>
+<net name="N$47" class="0">
+<segment>
+<pinref part="R30" gate="G$1" pin="2"/>
+<wire x1="215.9" y1="48.26" x2="223.52" y2="48.26" width="0.1524" layer="91"/>
+<pinref part="D1" gate="1" pin="C"/>
+</segment>
+</net>
+<net name="N$48" class="0">
+<segment>
+<pinref part="R31" gate="G$1" pin="1"/>
+<pinref part="PWM_1" gate="G$1" pin="P"/>
+<wire x1="182.88" y1="50.8" x2="203.2" y2="50.8" width="0.1524" layer="91"/>
+</segment>
+</net>
