File: PCB/MPPT2/MPPT2.sch (EAGLE design)
At the start: 53 parts, among them IC3 ACS711KEXLT-15AB-T, IC4 ACS711KEXLT-15AB-T

Commit message: NS
Parts:
- removed BATT_1_I_SENSE, IC3, IC4, PV_1_I_SENSE: ACS711KEXLT-15AB-T, SamacSys_Parts:ACS711KEXLT-15AB-T
- removed PROGRAM: Pin 1, con-lstb:MA08-1
- removed SV2: (no value), con-lstb:MA04-1
- added B1_I, B2_I, PV1_I, PV2_I: ACS711KEXLT-15AB-T, SamacSys_Parts:ACS711KEXLT-15AB-T
- added C10, C11, C8, C9: 100nF, resistor:C-USC0603
- added D1, D2: 1N4004, diode:1N4004
- added PROGRAMMER: (no value), con-lstb:MA06-1
- added PWM_1, PWM_2: WIREPAD2,54/1,1, wirepad:WIREPAD2,54/1,1
- added R27: 10K, rcl:R-US_R1206
- added R28, R29: 10K, resistor:R-US_R0603
- added R30: 470R, resistor:R-US_R0603
- added R31: 470R, resistor:R-US_R1206
- added R32, R33, R34, R35: 1K, resistor:R-US_R0603
- added X1, X2: 22-23-2021, con-molex:22-23-2021
- added X3: 22-23-2041, con-molex:22-23-2041
- renumbered LCD to __LCD
Connections:
- new net N$10: B1_I.!FAULT, R33.1
- new net N$39: CONTROLLER.RB1, R28.2, X3-2.S
- new net N$40: CONTROLLER.VPP/*MCLR/RS3, PROGRAMMER.1, R29.1
- new net N$41: CONTROLLER.RA6, D2.A
- new net N$42: CONTROLLER.RB0, R27.2, X3-4.S
- new net N$43: CONTROLLER.RA7, D1.A
- new net N$44: CONTROLLER.RB7, PROGRAMMER.4
- new net N$45: CONTROLLER.RB6, PROGRAMMER.5
- new net N$46: PWM_2.P, R30.1
- new net N$47: D1.C, R30.2
- new net N$48: PWM_1.P, R31.1
- new net N$49: D2.C, R31.2
- new net N$50: PV1_I.IP+, R1.1, U$1.P$1
- new net N$51: PV2_I.!FAULT, R34.1
- new net N$56: B2_I.!FAULT, R35.1
- net N$1: now also BUCK1_IN+.P, PV1_I.IP-; no longer PV_1_I_SENSE.IP+, R1.1, U$1.P$1
- net N$11: now also B2_I.IP-; no longer IC4.IP-
- net N$13: now also B2_I.IP+, BUCK2_OUT+.P; no longer BUCK1_IN+.P, PV_1_I_SENSE.IP-
- net N$2: now also PV1_I.VOUT; no longer PV_1_I_SENSE.VOUT
- net N$22: now also B1_I.IP+, BUCK1_OUT+.P; no longer BATT_1_I_SENSE.VOUT, BUFFER1.4IN+
- net N$32: now also PV2_I.VOUT; no longer IC3.VOUT
- net N$33: now also B2_I.VOUT; no longer IC4.VOUT
- net N$4: now also PV1_I.!FAULT, R32.1; no longer BATT_1_I_SENSE.IP+, BUCK1_OUT+.P
- net N$6: now also B1_I.IP-; no longer BATT_1_I_SENSE.IP-
- net N$7: now also B1_I.VOUT, BUFFER1.4IN+; no longer BUCK2_OUT+.P, IC4.IP+
- net N$8: now also PV2_I.IP+; no longer IC3.IP+
- net N$9: now also PV2_I.IP-; no longer IC3.IP-
- net VDD: now also B1_I.VCC, B2_I.VCC, C10.2, C11.2, C8.2, C9.2, PROGRAMMER.2, PV1_I.VCC, PV2_I.VCC, R27.1, R28.1, R29.2, R32.2, R33.2, R34.2, R35.2; no longer BATT_1_I_SENSE.VCC, IC3.VCC, IC4.VCC, PV_1_I_SENSE.VCC
- net VSS: now also B1_I.GND, B2_I.GND, C10.1, C11.1, C8.1, C9.1, PROGRAMMER.3, PV1_I.GND, PV2_I.GND, X3-1.S, X3-3.S; no longer BATT_1_I_SENSE.GND, IC3.GND, IC4.GND, PV_1_I_SENSE.GND
Other:
- moved on the sheet: BUCK1_IN+, BUCK1_IN-, BUCK1_OUT+, BUCK1_OUT-, BUCK2_IN+, BUCK2_OUT+, BUCK2_OUT-, C1, C2, C6, C7, R1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
