File: PCB/MPPT2/MPPT2.brd (EAGLE design)
At the start: 67 parts, among them IC3 ACS711KEXLT-15AB-T, IC4 ACS711KEXLT-15AB-T, X1 22-23-2021, X2 22-23-2021, X3 22-23-2041

Commit message: NS
Parts:
- added C10, C11, C8, C9: 100nF, resistor:C0603
- added D1, D2: 1N4004, diode:DO41-10
- added R30: 470R, resistor:R0603
- added R31: 470R, resistor:R1206
- added R32, R33, R34, R35: 1K, resistor:R0603
- renumbered BATT_1_I_SENSE to B1_I, IC3 to PV2_I, IC4 to B2_I, PV_1_I_SENSE to PV1_I
Connections:
- new net N$10: B1_I.4, R33.1
- new net N$4: PV1_I.4, R32.1
- new net N$46: PWM_2.1, R30.1
- new net N$47: D1.C, R30.2
- new net N$48: PWM_1.1, R31.1
- new net N$49: D2.C, R31.2
- new net N$51: PV2_I.4, R34.1
- new net N$56: B2_I.4, R35.1
- net N$41: now also D2.A; no longer PWM_1.1
- net N$43: now also D1.A; no longer PWM_2.1
- net VDD: now also C10.2, C11.2, C8.2, C9.2, R32.2, R33.2, R34.2, R35.2
- net VSS: now also C10.1, C11.1, C8.1, C9.1
Routing:
- net N$41: track 87.9 -> 20.3 mm, vias 2 -> 0
- net N$52: track 38.8 -> 0.00 mm
- net N$22: track 22.8 -> 0.00 mm, vias 1 -> 0
- net N$7: track 20.4 -> 0.00 mm, vias 2 -> 0
- net N$1: track 19.9 -> 0.00 mm
- net N$50: track 17.8 -> 0.00 mm
- net N$43: track 22.8 -> 10.1 mm
- net N$13: track 11.8 -> 0.00 mm
- net N$48: track 0.00 -> 11.3 mm
- net N$5: track 39.2 -> 30.7 mm
- net N$6: track 81.4 -> 74.2 mm
- net N$46: track 0.00 -> 6.88 mm
- net N$4: track 0.00 -> 3.75 mm
- net VDD: track 293.8 -> 297.1 mm
- net N$47: track 0.00 -> 2.96 mm
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
Commit message: ND
Parts:
- C5: value 100nF -> 10uF
- moved C8 8.45 mm to (19.1, 53.7), turned to 90 degrees
- moved R34 7.24 mm to (68.6, 64.1), turned to 90 degrees
- moved C10 6.79 mm to (64.8, 57.5)
- moved C9 6.79 mm to (45.4, 55.2), turned to 270 degrees
- moved C11 6.73 mm to (96.8, 65.7), turned to 90 degrees
- moved C3 4.13 mm to (54.3, 54.6)
- moved R6 3.81 mm to (58.4, 54.6)
- moved U$7 2.01 mm to (10.3, 9.28)
- moved R32 1.59 mm to (23.2, 53.7), turned to 90 degrees
- moved R35 1.42 mm to (94.0, 65.7), turned to 90 degrees
- moved R33 0.71 mm to (38.1, 50.2)
Routing:
- net VDD: track 297.1 -> 346.5 mm, vias 6 -> 10
- net N$52: track 0.00 -> 35.7 mm
- net N$49: track 0.00 -> 29.7 mm
- net N$22: track 0.00 -> 22.6 mm, vias 0 -> 1
- net N$1: track 0.00 -> 21.1 mm
- net N$50: track 0.00 -> 18.5 mm
- net N$7: track 0.00 -> 18.2 mm, vias 0 -> 2
- net N$56: track 0.00 -> 13.2 mm, vias 0 -> 2
- net N$13: track 0.00 -> 12.2 mm
- net N$6: track 74.2 -> 81.8 mm
- net N$5: track 30.7 -> 37.4 mm
- net N$10: track 0.00 -> 3.67 mm
- net N$8: track 18.2 -> 15.7 mm
- net N$51: track 0.00 -> 2.46 mm
- net N$37: track 11.4 -> 13.6 mm
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
Commit message: wtf
Parts:
- added C12, C13: 100nF, resistor:C0603
- added D3, D4: CZRU52C3V3, 0603ZenerDiode:CZRU
- added R36, R37: 165R, resistor:R0603
Connections:
- net N$39: now also C12.2, D3.1, R36.1
- net N$42: now also C13.2, D4.1, R37.1
- net VSS: now also C12.1, C13.1, D3.2, D4.2, R36.2, R37.2
Routing:
- net N$39: track 130.3 -> 135.7 mm
- net N$42: track 131.0 -> 135.4 mm
Changed lines of the file:
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@@
 <setting verticaltext="up"/>
 </settings>
-<grid distance="0.3175" unitdist="mm" unit="mm" style="lines" multiple="1" display="yes" altdistance="0.025" altunitdist="inch" altunit="mm"/>
+<grid distance="0.635" unitdist="mm" unit="mm" style="lines" multiple="1" display="yes" altdistance="0.025" altunitdist="inch" altunit="mm"/>
 <layers>
 <layer number="1" name="Top" color="4" fill="1" visible="yes" active="yes"/>
@@
 <element name="C10" library="resistor" package="C0603" value="100nF" x="64.77" y="57.4675"/>
 <element name="C11" library="resistor" package="C0603" value="100nF" x="96.8375" y="65.7225" rot="R90"/>
+<element name="D4" library="0603ZenerDiode" package="CZRU" value="CZRU52C3V3" x="20.32" y="71.12" rot="R180">
+<attribute name="VENDOR" value="Comchip" x="20.32" y="71.12" size="1.778" layer="27" rot="R180" display="off"/>
+<attribute name="MANUFACTURER_PART_NUMBER" value="" x="20.32" y="71.12" size="1.778" layer="27" rot="R180" display="off"/>
+</element>
+<element name="D3" library="0603ZenerDiode" package="CZRU" value="CZRU52C3V3" x="15.24" y="71.12" rot="R180">
+<attribute name="VENDOR" value="Comchip" x="15.24" y="71.12" size="1.778" layer="27" rot="R180" display="off"/>
+<attribute name="MANUFACTURER_PART_NUMBER" value="" x="15.24" y="71.12" size="1.778" layer="27" rot="R180" display="off"/>
+</element>
+<element name="R36" library="resistor" package="R0603" value="165R" x="10.16" y="68.58" rot="R90"/>
+<element name="R37" library="resistor" package="R0603" value="165R" x="20.32" y="67.31" rot="R180"/>
+<element name="C12" library="resistor" package="C0603" value="100nF" x="5.08" y="64.77" rot="R270"/>
+<element name="C13" library="resistor" package="C0603" value="100nF" x="25.4" y="64.77" rot="R180"/>
 </elements>
 <signals>
@@
 <via x="83.82" y="64.4525" extent="1-16" drill="0.8" shape="square"/>
 <via x="83.82" y="56.515" extent="1-16" drill="0.8" shape="square"/>
-<via x="15.24" y="68.2625" extent="1-16" drill="0.8" shape="square"/>
+<via x="0.9525" y="60.6425" extent="1-16" drill="0.8" shape="square"/>
 <via x="17.78" y="58.42" extent="1-16" drill="0.8" shape="square"/>
 <via x="45.72" y="34.925" extent="1-16" drill="0.8" shape="square"/>
@@
 <contactref element="C2" pad="1"/>
 <contactref element="C10" pad="1"/>
+<contactref element="D4" pad="2"/>
+<contactref element="D3" pad="2"/>
+<contactref element="R36" pad="2"/>
+<contactref element="R37" pad="2"/>
+<contactref element="C12" pad="1"/>
+<contactref element="C13" pad="1"/>
 </signal>
 <signal name="VDD">
@@
 <contactref element="X3" pad="2"/>
 <contactref element="R28" pad="2"/>
-<wire x1="9.2075" y1="65.405" x2="4.445" y2="60.6425" width="0.4064" layer="1"/>
+<wire x1="9.2075" y1="65.405" x2="5.55625" y2="61.75375" width="0.4064" layer="1"/>
+<wire x1="5.55625" y1="61.75375" x2="4.445" y2="60.6425" width="0.4064" layer="1"/>
 <wire x1="4.445" y1="60.6425" x2="4.445" y2="58.205" width="0.4064" layer="1"/>
 <wire x1="4.445" y1="58.205" x2="3.39" y2="57.15" width="0.4064" layer="1"/>
@@
 <wire x1="5.08" y1="14.605" x2="3.39" y2="16.295" width="0.4064" layer="1"/>
 <wire x1="3.39" y1="16.295" x2="3.39" y2="57.15" width="0.4064" layer="1"/>
-<wire x1="9.2075" y1="65.405" x2="15.875" y2="65.405" width="0.4064" layer="1"/>
+<wire x1="9.2075" y1="65.405" x2="10.16" y2="65.405" width="0.4064" layer="1"/>
+<wire x1="10.16" y1="65.405" x2="15.875" y2="65.405" width="0.4064" layer="1"/>
 <wire x1="15.875" y1="65.405" x2="16.8275" y2="66.3575" width="0.4064" layer="1"/>
-<wire x1="16.8275" y1="66.3575" x2="16.8275" y2="76.2" width="0.4064" layer="1"/>
+<wire x1="16.8275" y1="66.3575" x2="16.8275" y2="71.12" width="0.4064" layer="1"/>
+<contactref element="D3" pad="1"/>
+<contactref element="R36" pad="1"/>
+<contactref element="C12" pad="2"/>
+<wire x1="16.8275" y1="71.12" x2="16.8275" y2="76.2" width="0.4064" layer="1"/>
+<wire x1="16.1163" y1="71.12" x2="16.8275" y2="71.12" width="0.4064" layer="1"/>
+<wire x1="10.16" y1="67.73" x2="10.16" y2="65.405" width="0.4064" layer="1"/>
+<wire x1="5.08" y1="63.92" x2="5.08" y2="62.23" width="0.4064" layer="1"/>
+<wire x1="5.08" y1="62.23" x2="5.55625" y2="61.75375" width="0.4064" layer="1"/>
 </signal>
 <signal name="N$42">
@@
 <wire x1="4.9145" y1="51.283" x2="4.9145" y2="51.435" width="0.4064" layer="1"/>
 <wire x1="9.2075" y1="64.135" x2="20.955" y2="64.135" width="0.4064" layer="1"/>
-<wire x1="20.955" y1="64.135" x2="21.9075" y2="65.0875" width="0.4064" layer="1"/>
-<wire x1="21.9075" y1="65.0875" x2="21.9075" y2="76.2" width="0.4064" layer="1"/>
+<wire x1="20.955" y1="64.135" x2="21.59" y2="64.77" width="0.4064" layer="1"/>
+<wire x1="21.59" y1="64.77" x2="21.9075" y2="65.0875" width="0.4064" layer="1"/>
+<wire x1="21.9075" y1="65.0875" x2="21.9075" y2="67.31" width="0.4064" layer="1"/>
+<contactref element="D4" pad="1"/>
+<contactref element="R37" pad="1"/>
+<contactref element="C13" pad="2"/>
+<wire x1="21.9075" y1="67.31" x2="21.9075" y2="71.12" width="0.4064" layer="1"/>
+<wire x1="21.9075" y1="71.12" x2="21.9075" y2="76.2" width="0.4064" layer="1"/>
+<wire x1="21.1963" y1="71.12" x2="21.9075" y2="71.12" width="0.4064" layer="1"/>
+<wire x1="21.17" y1="67.31" x2="21.9075" y2="67.31" width="0.4064" layer="1"/>
+<wire x1="24.55" y1="64.77" x2="21.59" y2="64.77" width="0.4064" layer="1"/>
 </signal>
 <signal name="N$40">
