File: PCB/MPPT3/MPPT3.brd (EAGLE design)
At the start: 85 parts, among them X1 22-23-2021, X2 22-23-2021, X3 22-23-2041

Commit message: wtf
Parts:
- R32, R33: device resistor:R0603 -> resistor:R1206
- R36, R37: value 20K -> 165R
- moved C8 11.4 mm to (29.2, 48.6)
- moved C10 8.52 mm to (61.0, 65.1), turned to 270 degrees
- moved C12 6.82 mm to (5.08, 64.8), turned to 270 degrees
- moved C13 6.11 mm to (25.4, 64.8), turned to 180 degrees
- moved D3 5.84 mm to (15.2, 71.1), turned to 180 degrees
- moved D2 4.02 mm to (48.9, 30.2), turned to 45 degrees
- moved C9 3.43 mm to (48.3, 53.3), turned to 180 degrees
- moved R32 2.88 mm to (22.9, 50.8), turned to 270 degrees
- moved R33 2.69 mm to (36.2, 52.1), turned to 135 degrees
- moved R36 2.03 mm to (10.2, 68.6), turned to 90 degrees
- moved C3 1.91 mm to (54.3, 52.7)
- moved R6 1.91 mm to (58.4, 52.7)
- moved R37 1.35 mm to (20.3, 67.3), turned to 180 degrees
- moved R5 1.27 mm to (58.4, 59.1)
- moved C11 1.00 mm to (97.8, 65.4)
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Connections:
- new net N$53: B1_I.10, B2_I.10, C10.2, C11.2, C8.2, C9.2, CONTROLLER.7, PV1_I.10, PV2_I.10, R32.2, R33.2, R34.2, R35.2
- net VDD: no longer B1_I.10, B2_I.10, C10.2, C11.2, C8.2, C9.2, PV1_I.10, PV2_I.10, R32.2, R33.2, R34.2, R35.2
Routing:
- net N$53: track 0.00 -> 178.4 mm, vias 0 -> 6
- net VDD: track 346.5 -> 223.0 mm, vias 10 -> 3
- net N$39: track 130.3 -> 135.7 mm
- net N$41: track 20.3 -> 25.3 mm
- net N$42: track 131.0 -> 135.4 mm
- net N$8: track 15.7 -> 18.2 mm
- net N$52: track 35.7 -> 33.6 mm
- net N$4: track 3.53 -> 4.10 mm
- net N$51: track 2.46 -> 3.00 mm

Commit message: OK
Changed lines of the file:
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@@
 <setting verticaltext="up"/>
 </settings>
-<grid distance="0.635" unitdist="mm" unit="mm" style="lines" multiple="1" display="no" altdistance="0.025" altunitdist="inch" altunit="mm"/>
+<grid distance="0.3175" unitdist="mm" unit="mm" style="lines" multiple="1" display="yes" altdistance="0.025" altunitdist="inch" altunit="mm"/>
 <layers>
 <layer number="1" name="Top" color="4" fill="1" visible="yes" active="yes"/>
@@
 <contactref element="C13" pad="1"/>
 <via x="40.005" y="50.165" extent="1-16" drill="0.8" shape="square"/>
-<wire x1="62.4205" y1="19.404990625" x2="69.6595" y2="18.10499375" width="0" layer="19" extent="1-1"/>
+<via x="71.755" y="30.7975" extent="1-16" drill="0.6" shape="square"/>
+<via x="66.3575" y="15.5575" extent="1-16" drill="0.5" shape="square"/>
 </signal>
 <signal name="VDD">

Commit message: nm
Parts:
- added S1: Reset, SparkFun-Switches:TACTILE_SWITCH_PTH_6.0MM
- added S2: UP, SparkFun-Switches:TACTILE_SWITCH_PTH_6.0MM
- added S3: DOWN, SparkFun-Switches:TACTILE_SWITCH_PTH_6.0MM
- added S4: ENTER, SparkFun-Switches:TACTILE_SWITCH_PTH_6.0MM
- moved U$7 0.32 mm to (10.6, 9.28)
Connections:
- removed net N$10: B1_I.4, R33.1
- removed net N$4: PV1_I.4, R32.1
- removed net N$51: PV2_I.4, R34.1
- net N$40: now also S1.1
- net N$56: now also B1_I.4, CONTROLLER.23, PV1_I.4, PV2_I.4, R32.1, R33.1, R34.1
- net VSS: now also S1.3
Routing:
- net N$40: track 23.9 -> 61.1 mm
- net N$4: track 4.10 -> 0.00 mm
- net N$10: track 4.01 -> 0.00 mm
- net N$51: track 3.00 -> 0.00 mm

Commit message: F
Parts:
- removed S2: UP, SparkFun-Switches:TACTILE_SWITCH_PTH_6.0MM
- removed S3: DOWN, SparkFun-Switches:TACTILE_SWITCH_PTH_6.0MM
- removed S4: ENTER, SparkFun-Switches:TACTILE_SWITCH_PTH_6.0MM
- added R38, R39, R40: 10K, resistor:R0603
- added _: ENTER, SparkFun-Switches:TACTILE_SWITCH_PTH_6.0MM
- added __: DOWN, SparkFun-Switches:TACTILE_SWITCH_PTH_6.0MM
- added ___: UP, SparkFun-Switches:TACTILE_SWITCH_PTH_6.0MM
- R5: device resistor:R0603 -> resistor:R1206
- moved S1 21.5 mm to (4.45, 20.6), turned to 0 degrees
- moved U$7 0.45 mm to (10.3, 9.59)
Connections:
- new net N$10: R39.2, __.3
- new net N$4: R38.2, ___.3
- new net N$51: R40.2, _.3
- net VDD: now also _.1, __.1, ___.1
- net VSS: now also CONTROLLER.24, R38.1, R39.1, R40.1
Routing:
- net N$56: track 13.3 -> 180.7 mm, vias 2 -> 10
- net VDD: track 223.0 -> 254.6 mm
- net N$40: track 61.1 -> 88.8 mm
- net N$4: track 0.00 -> 15.6 mm
- net N$10: track 0.00 -> 14.1 mm
- net N$51: track 0.00 -> 2.52 mm
- net VSS: track 0.00 -> 1.28 mm, vias 20 -> 21
- net N$8: track 18.2 -> 17.0 mm
- net N$52: track 33.6 -> 33.0 mm
