File: PCB/MPPT3/MPPT3.sch (EAGLE design)
At the start: 78 parts, among them X1 22-23-2021, X2 22-23-2021, X3 22-23-2041

Commit message: wtf
Parts:
- R32, R33: device resistor:R-US_R0603 -> resistor:R-US_R1206
- R36, R37: value 20K -> 165R
Connections:
- new net N$53: B1_I.VCC, B2_I.VCC, C10.2, C11.2, C8.2, C9.2, CONTROLLER.RA5, PV1_I.VCC, PV2_I.VCC, R32.2, R33.2, R34.2, R35.2
- net VDD: no longer B1_I.VCC, B2_I.VCC, C10.2, C11.2, C8.2, C9.2, PV1_I.VCC, PV2_I.VCC, R32.2, R33.2, R34.2, R35.2
Other:
- moved on the sheet: D2, PWM_1, R31, R32, R33, R34, R35

Commit message: nm
Parts:
- added S1: Reset, SparkFun-Switches:MOMENTARY-SWITCH-SPST-PTH-6.0MM
- added S2: UP, SparkFun-Switches:MOMENTARY-SWITCH-SPST-PTH-6.0MM
- added S3: DOWN, SparkFun-Switches:MOMENTARY-SWITCH-SPST-PTH-6.0MM
- added S4: ENTER, SparkFun-Switches:MOMENTARY-SWITCH-SPST-PTH-6.0MM
Connections:
- removed net N$10: B1_I.!FAULT, R33.1
- removed net N$4: PV1_I.!FAULT, R32.1
- removed net N$51: PV2_I.!FAULT, R34.1
- net N$40: now also S1.1
- net N$56: now also B1_I.!FAULT, CONTROLLER.RB2, PV1_I.!FAULT, PV2_I.!FAULT, R32.1, R33.1, R34.1
- net VSS: now also S1.2

Commit message: F
Parts:
- removed S2: UP, SparkFun-Switches:MOMENTARY-SWITCH-SPST-PTH-6.0MM
- removed S3: DOWN, SparkFun-Switches:MOMENTARY-SWITCH-SPST-PTH-6.0MM
- removed S4: ENTER, SparkFun-Switches:MOMENTARY-SWITCH-SPST-PTH-6.0MM
- added R38, R39, R40: 10K, resistor:R-US_R0603
- added _: ENTER, SparkFun-Switches:MOMENTARY-SWITCH-SPST-PTH-6.0MM
- added __: DOWN, SparkFun-Switches:MOMENTARY-SWITCH-SPST-PTH-6.0MM
- added ___: UP, SparkFun-Switches:MOMENTARY-SWITCH-SPST-PTH-6.0MM
- R5: device resistor:R-US_R0603 -> resistor:R-US_R1206
Connections:
- new net N$10: R39.2, __.2
- new net N$4: R38.2, ___.2
- new net N$51: R40.2, _.2
- net VDD: now also _.1, __.1, ___.1
- net VSS: now also CONTROLLER.RB3, R38.1, R39.1, R40.1
Changed lines of the file:
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@@
 <setting verticaltext="up"/>
 </settings>
-<grid distance="0.1" unitdist="inch" unit="mm" style="lines" multiple="1" display="yes" altdistance="0.01" altunitdist="inch" altunit="inch"/>
+<grid distance="0.1" unitdist="inch" unit="inch" style="lines" multiple="1" display="no" altdistance="0.01" altunitdist="inch" altunit="inch"/>
 <layers>
 <layer number="1" name="Top" color="4" fill="1" visible="yes" active="no"/>
@@
 <part name="R3" library="resistor" deviceset="R-US_" device="R0603" value="100K"/>
 <part name="R4" library="resistor" deviceset="R-US_" device="R0603" value="20K"/>
-<part name="R5" library="resistor" deviceset="R-US_" device="R0603" value="100K"/>
+<part name="R5" library="resistor" deviceset="R-US_" device="R1206" value="100K"/>
 <part name="R6" library="resistor" deviceset="R-US_" device="R0603" value="20K"/>
 <part name="R7" library="resistor" deviceset="R-US_" device="R0603" value="100K"/>
@@
 <part name="S1" library="SparkFun-Switches" deviceset="MOMENTARY-SWITCH-SPST" device="-PTH-6.0MM" value="Reset"/>
 <part name="VSS14" library="supply1" deviceset="VSS" device=""/>
-<part name="S2" library="SparkFun-Switches" deviceset="MOMENTARY-SWITCH-SPST" device="-PTH-6.0MM" value="UP"/>
-<part name="S3" library="SparkFun-Switches" deviceset="MOMENTARY-SWITCH-SPST" device="-PTH-6.0MM" value="DOWN"/>
-<part name="S4" library="SparkFun-Switches" deviceset="MOMENTARY-SWITCH-SPST" device="-PTH-6.0MM" value="ENTER"/>
+<part name="___" library="SparkFun-Switches" deviceset="MOMENTARY-SWITCH-SPST" device="-PTH-6.0MM" value="UP"/>
+<part name="__" library="SparkFun-Switches" deviceset="MOMENTARY-SWITCH-SPST" device="-PTH-6.0MM" value="DOWN"/>
+<part name="_" library="SparkFun-Switches" deviceset="MOMENTARY-SWITCH-SPST" device="-PTH-6.0MM" value="ENTER"/>
+<part name="R38" library="resistor" deviceset="R-US_" device="R0603" value="10K"/>
+<part name="R39" library="resistor" deviceset="R-US_" device="R0603" value="10K"/>
+<part name="R40" library="resistor" deviceset="R-US_" device="R0603" value="10K"/>
+<part name="VSS15" library="supply1" deviceset="VSS" device=""/>
 </parts>
 <sheets>
@@
 <instance part="S1" gate="G$1" x="180.34" y="7.62"/>
 <instance part="VSS14" gate="G$1" x="213.36" y="5.08"/>
-<instance part="S2" gate="G$1" x="43.18" y="15.24"/>
-<instance part="S3" gate="G$1" x="43.18" y="7.62"/>
-<instance part="S4" gate="G$1" x="43.18" y="0"/>
+<instance part="___" gate="G$1" x="40.64" y="15.24"/>
+<instance part="__" gate="G$1" x="40.64" y="7.62"/>
+<instance part="_" gate="G$1" x="40.64" y="0"/>
+<instance part="R38" gate="G$1" x="50.8" y="15.24" rot="R180"/>
+<instance part="R39" gate="G$1" x="50.8" y="7.62" rot="R180"/>
+<instance part="R40" gate="G$1" x="50.8" y="0" rot="R180"/>
+<instance part="VSS15" gate="G$1" x="62.23" y="-2.54"/>
 </instances>
 <busses>
@@
 <wire x1="185.42" y1="7.62" x2="213.36" y2="7.62" width="0.1524" layer="91"/>
 </segment>
+<segment>
+<pinref part="CONTROLLER" gate="A" pin="RB3"/>
+<pinref part="R40" gate="G$1" pin="1"/>
+<wire x1="88.9" y1="25.4" x2="58.42" y2="25.4" width="0.1524" layer="91"/>
+<wire x1="58.42" y1="25.4" x2="55.88" y2="15.24" width="0.1524" layer="91"/>
+<pinref part="VSS15" gate="G$1" pin="VSS"/>
+<wire x1="55.88" y1="15.24" x2="55.88" y2="7.62" width="0.1524" layer="91"/>
+<wire x1="55.88" y1="7.62" x2="55.88" y2="0" width="0.1524" layer="91"/>
+<wire x1="55.88" y1="0" x2="62.23" y2="0" width="0.1524" layer="91"/>
+<junction x="55.88" y="0"/>
+<pinref part="R39" gate="G$1" pin="1"/>
+<junction x="55.88" y="7.62"/>
+<pinref part="R38" gate="G$1" pin="1"/>
+<junction x="55.88" y="15.24"/>
+</segment>
 </net>
 <net name="VDD" class="0">
@@
 <junction x="88.9" y="10.16"/>
 <junction x="116.84" y="35.56"/>
+<pinref part="_" gate="G$1" pin="1"/>
+<wire x1="60.96" y1="30.48" x2="40.64" y2="30.48" width="0.1524" layer="91"/>
+<wire x1="40.64" y1="30.48" x2="35.56" y2="15.24" width="0.1524" layer="91"/>
+<pinref part="___" gate="G$1" pin="1"/>
+<junction x="35.56" y="15.24"/>
+<wire x1="35.56" y1="15.24" x2="35.56" y2="7.62" width="0.1524" layer="91"/>
+<pinref part="__" gate="G$1" pin="1"/>
+<junction x="35.56" y="7.62"/>
+<wire x1="35.56" y1="7.62" x2="35.56" y2="0" width="0.1524" layer="91"/>
 </segment>
 <segment>
@@
 <wire x1="144.78" y1="7.62" x2="144.78" y2="15.24" width="0.1524" layer="91"/>
 <wire x1="175.26" y1="7.62" x2="144.78" y2="7.62" width="0.1524" layer="91"/>
+<junction x="144.78" y="7.62"/>
 </segment>
 </net>
@@
 </segment>
 </net>
+<net name="N$4" class="0">
+<segment>
+<pinref part="___" gate="G$1" pin="2"/>
+<pinref part="R38" gate="G$1" pin="2"/>
+</segment>
+</net>
+<net name="N$10" class="0">
+<segment>
+<pinref part="__" gate="G$1" pin="2"/>
+<pinref part="R39" gate="G$1" pin="2"/>
+</segment>
+</net>
+<net name="N$51" class="0">
+<segment>
+<pinref part="_" gate="G$1" pin="2"/>
+<pinref part="R40" gate="G$1" pin="2"/>
+</segment>
+</net>

Commit message: SendOutForFab
Parts:
- renumbered S1 to --
Changed lines of the file:
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@@
 <grid distance="0.1" unitdist="inch" unit="inch" style="lines" multiple="1" display="no" altdistance="0.01" altunitdist="inch" altunit="inch"/>
 <layers>
-<layer number="1" name="Top" color="4" fill="1" visible="yes" active="no"/>
-<layer number="16" name="Bottom" color="1" fill="1" visible="yes" active="no"/>
-<layer number="17" name="Pads" color="2" fill="1" visible="yes" active="no"/>
-<layer number="18" name="Vias" color="2" fill="1" visible="yes" active="no"/>
-<layer number="19" name="Unrouted" color="6" fill="1" visible="yes" active="no"/>
-<layer number="20" name="Dimension" color="15" fill="1" visible="yes" active="no"/>
-<layer number="21" name="tPlace" color="7" fill="1" visible="yes" active="no"/>
-<layer number="22" name="bPlace" color="7" fill="1" visible="yes" active="no"/>
-<layer number="23" name="tOrigins" color="15" fill="1" visible="yes" active="no"/>
-<layer number="24" name="bOrigins" color="15" fill="1" visible="yes" active="no"/>
-<layer number="25" name="tNames" color="7" fill="1" visible="yes" active="no"/>
-<layer number="26" name="bNames" color="7" fill="1" visible="yes" active="no"/>
-<layer number="27" name="tValues" color="7" fill="1" visible="yes" active="no"/>
-<layer number="28" name="bValues" color="7" fill="1" visible="yes" active="no"/>
+<layer number="1" name="Top" color="4" fill="1" visible="no" active="no"/>
+<layer number="16" name="Bottom" color="1" fill="1" visible="no" active="no"/>
+<layer number="17" name="Pads" color="2" fill="1" visible="no" active="no"/>
+<layer number="18" name="Vias" color="2" fill="1" visible="no" active="no"/>
+<layer number="19" name="Unrouted" color="6" fill="1" visible="no" active="no"/>
+<layer number="20" name="Dimension" color="15" fill="1" visible="no" active="no"/>
+<layer number="21" name="tPlace" color="7" fill="1" visible="no" active="no"/>
+<layer number="22" name="bPlace" color="7" fill="1" visible="no" active="no"/>
+<layer number="23" name="tOrigins" color="15" fill="1" visible="no" active="no"/>
+<layer number="24" name="bOrigins" color="15" fill="1" visible="no" active="no"/>
+<layer number="25" name="tNames" color="7" fill="1" visible="no" active="no"/>
+<layer number="26" name="bNames" color="7" fill="1" visible="no" active="no"/>
+<layer number="27" name="tValues" color="7" fill="1" visible="no" active="no"/>
+<layer number="28" name="bValues" color="7" fill="1" visible="no" active="no"/>
 <layer number="29" name="tStop" color="7" fill="3" visible="no" active="no"/>
 <layer number="30" name="bStop" color="7" fill="6" visible="no" active="no"/>
@@
 <layer number="35" name="tGlue" color="7" fill="4" visible="no" active="no"/>
 <layer number="36" name="bGlue" color="7" fill="5" visible="no" active="no"/>
-<layer number="37" name="tTest" color="7" fill="1" visible="yes" active="no"/>
-<layer number="38" name="bTest" color="7" fill="1" visible="yes" active="no"/>
+<layer number="37" name="tTest" color="7" fill="1" visible="no" active="no"/>
+<layer number="38" name="bTest" color="7" fill="1" visible="no" active="no"/>
 <layer number="39" name="tKeepout" color="4" fill="11" visible="no" active="no"/>
 <layer number="40" name="bKeepout" color="1" fill="11" visible="no" active="no"/>
@@
 <layer number="44" name="Drills" color="7" fill="1" visible="no" active="no"/>
 <layer number="45" name="Holes" color="7" fill="1" visible="no" active="no"/>
-<layer number="46" name="Milling" color="3" fill="1" visible="yes" active="no"/>
-<layer number="47" name="Measures" color="7" fill="1" visible="yes" active="no"/>
-<layer number="48" name="Document" color="7" fill="1" visible="yes" active="no"/>
-<layer number="49" name="Reference" color="7" fill="1" visible="yes" active="no"/>
-<layer number="50" name="dxf" color="7" fill="1" visible="yes" active="no"/>
-<layer number="51" name="tDocu" color="7" fill="1" visible="yes" active="no"/>
-<layer number="52" name="bDocu" color="7" fill="1" visible="yes" active="no"/>
-<layer number="53" name="tGND_GNDA" color="7" fill="9" visible="yes" active="no"/>
-<layer number="54" name="bGND_GNDA" color="1" fill="9" visible="yes" active="no"/>
-<layer number="56" name="wert" color="7" fill="1" visible="yes" active="no"/>
-<layer number="57" name="tCAD" color="7" fill="1" visible="yes" active="no"/>
-<layer number="59" name="tCarbon" color="7" fill="1" visible="yes" active="no"/>
-<layer number="60" name="bCarbon" color="7" fill="1" visible="yes" active="no"/>
+<layer number="46" name="Milling" color="3" fill="1" visible="no" active="no"/>
+<layer number="47" name="Measures" color="7" fill="1" visible="no" active="no"/>
+<layer number="48" name="Document" color="7" fill="1" visible="no" active="no"/>
+<layer number="49" name="Reference" color="7" fill="1" visible="no" active="no"/>
+<layer number="50" name="dxf" color="7" fill="1" visible="no" active="no"/>
+<layer number="51" name="tDocu" color="7" fill="1" visible="no" active="no"/>
+<layer number="52" name="bDocu" color="7" fill="1" visible="no" active="no"/>
+<layer number="53" name="tGND_GNDA" color="7" fill="9" visible="no" active="no"/>
+<layer number="54" name="bGND_GNDA" color="1" fill="9" visible="no" active="no"/>
+<layer number="56" name="wert" color="7" fill="1" visible="no" active="no"/>
+<layer number="57" name="tCAD" color="7" fill="1" visible="no" active="no"/>
+<layer number="59" name="tCarbon" color="7" fill="1" visible="no" active="no"/>
+<layer number="60" name="bCarbon" color="7" fill="1" visible="no" active="no"/>
 <layer number="90" name="Modules" color="5" fill="1" visible="yes" active="yes"/>
 <layer number="91" name="Nets" color="2" fill="1" visible="yes" active="yes"/>
@@
 <part name="R33" library="resistor" deviceset="R-US_" device="R1206" value="1K"/>
 <part name="R32" library="resistor" deviceset="R-US_" device="R1206" value="1K"/>
-<part name="S1" library="SparkFun-Switches" deviceset="MOMENTARY-SWITCH-SPST" device="-PTH-6.0MM" value="Reset"/>
+<part name="--" library="SparkFun-Switches" deviceset="MOMENTARY-SWITCH-SPST" device="-PTH-6.0MM" value="Reset"/>
 <part name="VSS14" library="supply1" deviceset="VSS" device=""/>
 <part name="___" library="SparkFun-Switches" deviceset="MOMENTARY-SWITCH-SPST" device="-PTH-6.0MM" value="UP"/>
@@
 <instance part="R33" gate="G$1" x="91.44" y="139.7" rot="R270"/>
 <instance part="R32" gate="G$1" x="50.8" y="139.7" rot="R270"/>
-<instance part="S1" gate="G$1" x="180.34" y="7.62"/>
+<instance part="--" gate="G$1" x="180.34" y="7.62"/>
 <instance part="VSS14" gate="G$1" x="213.36" y="5.08"/>
 <instance part="___" gate="G$1" x="40.64" y="15.24"/>
@@
 </segment>
 <segment>
-<pinref part="S1" gate="G$1" pin="2"/>
+<pinref part="--" gate="G$1" pin="2"/>
 <pinref part="VSS14" gate="G$1" pin="VSS"/>
 <wire x1="185.42" y1="7.62" x2="213.36" y2="7.62" width="0.1524" layer="91"/>
@@
 <pinref part="R29" gate="G$1" pin="1"/>
 <junction x="88.9" y="0"/>
-<pinref part="S1" gate="G$1" pin="1"/>
+<pinref part="--" gate="G$1" pin="1"/>
 <wire x1="144.78" y1="7.62" x2="144.78" y2="15.24" width="0.1524" layer="91"/>
 <wire x1="175.26" y1="7.62" x2="144.78" y2="7.62" width="0.1524" layer="91"/>
